File: kicad/oresat-c3-sch-uhf-band.kicad_sch (KiCad schematic)
At the start: 129 parts, among them Q3 NTR4101, Q4 PMV45EN, U16 AX5043, U18 LT5534, U19 BDCN-20-13+, U20 QPC1022, U21 TQP7M9105, U22 LT5534, U25 SN74LVC1G11IDCKRQ1, U26 TLV7041DBV, U27 LP2985AIM5-1.8_NOPB, U29 TQP3M9036, U32 SF2446E, U33 SF2446E, U40 MAX941EUA+, X1 TYKTBLSANF-16.000000

Commit message: Added Oresat symbol lib. Removed any L-band related components from pcb and schematic
Parts:
- renumbered C37 to C118, C37 to C119, C50 to C120, C50 to C121, C50 to C140, C50 to C141, C50 to C55, C50 to C57, C50 to C58, C50 to C59, C50 to C60, C50 to C61, C50 to C62, C50 to C63, C50 to C64, C50 to C66, C50 to C67, C50 to C68, C50 to C69, C50 to C70, C45 to C71, C48 to C72, C44 to C73, C46 to C75, C43 to C76, C42 to C77, C41 to C80, C40 to C81, C39 to C82, C41 to C83, C40 to C84, C38 to C85, C37 to C86, C12 to C87, C40 to C88, C50 to C89, C50 to C90, C50 to C91, C50 to C92, C50 to C94, C50 to C95, C50 to C96, C50 to C97, D11 to D15, D1 to D16, L2 to L12, L7 to L13, L9 to L14, L8 to L15, L7 to L16, L6 to L17, L5 to L18, L8 to L19, L8 to L20, L8 to L26, R10 to R106, R90 to R107, R10 to R108, R10 to R109, R10 to R110, R10 to R112, R10 to R113, R10 to R114, R10 to R12, R10 to R13, R10 to R14, R10 to R15, R10 to R16, R10 to R19, R6 to R20, R5 to R21, R4 to R22, R10 to R23, R10 to R24, R10 to R25, R10 to R65, R10 to R81, TP28 to TP105, TP28 to TP122, TP28 to TP36, TP28 to TP41, TP28 to TP43, TP28 to TP44, TP28 to TP45, TP28 to TP50, TP28 to TP51, TP28 to TP52, TP28 to TP53, TP28 to TP54, TP28 to TP55, TP28 to TP56, TP28 to TP57, TP28 to TP60, TP28 to TP88, U16 to U23

Commit message: Removed UF band
Parts:
- removed AT1, AT2, AT3, AT4: 10dB, oresat-passives:PAT0816(0603), symbol oresat-passives:PAT0816-attenuator
- removed C118, C119, C120, C58, C67, C75, C84, C94, C96: 100p, Capacitor_SMD:C_0402_1005Metric, symbol Device:C_Small
- removed C121, C95, C97: 1u, Capacitor_SMD:C_0603_1608Metric, symbol Device:C_Small
- removed C140, C61: 10u, Capacitor_SMD:C_0603_1608Metric, symbol Device:C_Small
- removed C141, C57, C60, C68, C89, C90: 100n, Capacitor_SMD:C_0603_1608Metric, symbol Device:C_Small
- removed C55: 8.2p, Capacitor_SMD:C_0603_1608Metric, symbol Device:C_Small
- removed C59, C69, C71, C73: 1n, Capacitor_SMD:C_0402_1005Metric, symbol Device:C_Small
- removed C62, C63, C64: 100p, Capacitor_SMD:C_0603_1608Metric, symbol Device:C_Small
- removed C66: 22n, Capacitor_SMD:C_0603_1608Metric, symbol Device:C_Small
- removed C70: 10p, Capacitor_SMD:C_0603_1608Metric, symbol Device:C_Small
- removed C72, C92: 4.7u, Capacitor_SMD:C_0603_1608Metric, symbol Device:C_Small
- removed C76, C77: 82p, Capacitor_SMD:C_0402_1005Metric, symbol Device:C_Small
- removed C80, C81: 8.2p, Capacitor_SMD:C_0402_1005Metric, symbol Device:C_Small
- removed C82, C88: 22p, Capacitor_SMD:C_0402_1005Metric, symbol Device:C_Small
- removed C83: 27p, Capacitor_SMD:C_0402_1005Metric, symbol Device:C_Small
- removed C85, C87: 3p, Capacitor_SMD:C_0402_1005Metric, symbol Device:C_Small
- removed C86: 8.3p, Capacitor_SMD:C_0402_1005Metric, symbol Device:C_Small
- removed C91: 10n, Capacitor_SMD:C_0603_1608Metric, symbol Device:C_Small
- removed D15: GREEN, LED_SMD:LED_0603_1608Metric, symbol Device:LED_Small
- removed D16: 1N4151WS, Diode_SMD:D_SOD-323, symbol oresat-diodes:1N4151WS-HE3
- removed L12: 10n, Inductor_SMD:L_0603_1608Metric, symbol Device:L_Small
- removed L13: 4.1n, Inductor_SMD:L_0402_1005Metric, symbol Device:L_Small
- removed L14, L19: 91n, Inductor_SMD:L_0603_1608Metric, symbol Device:L_Small
- removed L15: 43n, Inductor_SMD:L_0603_1608Metric, symbol Device:L_Small
- removed L16: 43n, Inductor_SMD:L_0402_1005Metric, symbol Device:L_Small
- removed L17, L18: 18n, Inductor_SMD:L_0402_1005Metric, symbol Device:L_Small
- removed L20: 22n, Inductor_SMD:L_0805_2012Metric, symbol Device:L_Small
- removed L26: 68n, Inductor_SMD:L_0603_1608Metric, symbol Device:L_Small
- removed Q3: NTR4101, Package_TO_SOT_SMD:SOT-23-3, symbol Device:Q_PMOS_GSD
- removed Q4: PMV45EN, Package_TO_SOT_SMD:SOT-23-3, symbol Device:Q_NMOS_GSD
- removed R106: 33k, Resistor_SMD:R_0603_1608Metric, symbol Device:R_Small_US
- removed R107, R115, R23, R24, R81: 10k, Resistor_SMD:R_0603_1608Metric, symbol Device:R_Small_US
- removed R108, R25: 100k, Resistor_SMD:R_0603_1608Metric, symbol Device:R_Small_US
- removed R109, R110: 15k, Resistor_SMD:R_0603_1608Metric, symbol Device:R_Small_US
- removed R11, R17, R18, R4: 4.7k, Resistor_SMD:R_0603_1608Metric, symbol Device:R_Small_US
- removed R111: 150, Resistor_SMD:R_0603_1608Metric, symbol Device:R_Small_US
- removed R112, R114, R65: 47k, Resistor_SMD:R_0603_1608Metric, symbol Device:R_Small_US
- removed R113, R14, R15: 22k, Resistor_SMD:R_0603_1608Metric, symbol Device:R_Small_US
- removed R12, R19: 50, Resistor_SMD:R_0402_1005Metric, symbol Device:R_Small_US
- removed R13, R16: 3k, Resistor_SMD:R_0603_1608Metric, symbol Device:R_Small_US
- removed R20: 150, Resistor_SMD:R_0402_1005Metric, symbol Device:R_Small_US
- removed R21, R22: 0, Resistor_SMD:R_0402_1005Metric, symbol Device:R_Small_US
- removed TP105, TP122, TP36, TP41, TP43, TP44, TP45, TP50, TP51, TP52, TP53, TP54, TP55, TP56, TP57, TP60, TP88: Test-Point, oresat-misc:TestPoint_Pad_D1.0mm, symbol oresat-misc:Test-Point-1mm-round
- removed TP901, TP902, TP903, TP904, TP905, TP906, TP907, TP908, TP909: ~, oresat-misc:TestPoint_RF_Probe, symbol oresat-misc:Test-Point-RF-Probe-Stripline
- removed U18, U22: LT5534, Package_TO_SOT_SMD:SOT-363_SC-70-6, symbol oresat-ics:LT5534
- removed U19: BDCN-20-13+, oresat-ics:BDCN-20-13+, symbol oresat-ics:BDCN-20-13+
- removed U20: QPC1022, oresat-ics:QPC1022, symbol oresat-ics:QPC1022
- removed U21: TQP7M9105, oresat-ics:U-QORVO-TQP7M9105-VIAS, symbol oresat-ics:TQP7M9105
- removed U23: AX5043, oresat-ics:U-AX5043-QFN28-5X5-WITH-CENTER-PAD, symbol oresat-ics:AX5043
- removed U25: SN74LVC1G11IDCKRQ1, Package_TO_SOT_SMD:Texas_R-PDSO-G6, symbol oresat-ics:SN74LVC1G11IDCKRQ1
- removed U26: TLV7041DBV, Package_TO_SOT_SMD:SOT-23-5, symbol Comparator:TLV7041DBV
- removed U27: LP2985AIM5-1.8_NOPB, Package_TO_SOT_SMD:SOT-23-5, symbol oresat-ics:LP2985-N
- removed U29: TQP3M9036, oresat-ics:U-Qorvo-TQP3M9036-QFN-8-MO-220E, symbol oresat-ics:TQP3M9036
- removed U32, U33: SF2446E, oresat-ics:SM3030-6, symbol oresat-ics:SF2446E
- removed U40: MAX941EUA+, oresat-ics:LINEAR-MSOP-8-AND-MAXIM-UMAX-8-21-0036, symbol oresat-ics:MAX941EUA+
- removed X1: TYKTBLSANF-16.000000, oresat-ics:X_TCXO_SMD_Taitien_2.5x2.0mm, symbol oresat-ics:Taiten-TY-Series-TXCO
Connections:
- no-connect marks 1 -> 0
Other:
- note removed: "+10 dBm"
- note removed: "+13 dBm (single ended)"
- note removed: "+20 dB LNA"
- note removed: "+23 dB Power Amp"
- note removed: "+32.8 dBm"
- note removed: "+33 dBm"
- note removed: "-58.7 dBm"
- note removed: "-61.7 dBm"
- note removed: "-80.2 dBm"
- note removed: "-83.2 dBm"
- note removed: "0.43V level ~ 0-1 dB"
- note removed: "0402"
- note removed: "10dB"
- note removed: "16 MHz TCXO with 1.8V LDO"
- note removed: "16 MHz clipped sine wave output"
- note removed: "2.9V"
- note removed: "30dB"
- note removed: "5th order LPF"
- note removed: "AX5043 Pins 11, 12, 13, 21 intentionally left floating."
- note removed: "AX5043 Transceiver (UHF, 435 - 438 MHz)"
- note removed: "Bi-directional Coupler"
- note removed: "Clear nLatch only (don't latch accidentally)"
- note removed: "FORWARD Log RF Detector"
- note removed: "Measured TOT time: 880 ms"
- note removed: "Note: 0603 for power!"
- note removed: "Pins 9 & 10 are both inputs and are intentionally shorted"
- note removed: "RECEIVE"
- note removed: "REVERSE Log RF Detector"
- note removed: "RF Switch"
- note removed: "RX: -80 dBm in"
- note removed: "TRANSMIT"
- note removed: "TX: +32.6 dBm"
- note removed: "To backplane and UHF tape anntenna"
- note removed: "Tx Time Out Timer (TOT)"
