File: kicad/oresat-c3-sch-deployers.kicad_sch (KiCad schematic)
At the start: 28 parts, among them Q10 FDMQ86530L, Q11 DMP2240UDM-7, Q5 DMP2240UDM-7, Q7 DMP2240UDM-7, Q8 FDMQ86530L, Q9 DMP2240UDM-7

Commit message: Added Oresat symbol lib. Removed any L-band related components from pcb and schematic
Parts:
- renumbered D3 to D13, D3 to D14, R80 to R100, R80 to R101, R80 to R102, R68 to R117, R68 to R30, R80 to R91, R80 to R94, R80 to R95, R80 to R96, R80 to R97, R68 to R98, R80 to R99, TP64 to TP62, TP65 to TP63

Commit message: Removed antenna deployers, fixed
Parts:
- removed D13, D14: 1N4151WS, Diode_SMD:D_SOD-323, symbol oresat-diodes:1N4151WS-HE3
- removed Q10, Q8: FDMQ86530L, oresat-transistors:FDMQ86530L, symbol oresat-transistors:FDMQ86530L
- removed Q11, Q5, Q7, Q9: DMP2240UDM-7, Package_TO_SOT_SMD:SOT-23-6, symbol oresat-transistors:DMP2240UDM-7
- removed R100, R96: 1k, Resistor_SMD:R_0603_1608Metric, symbol Device:R_Small_US
- removed R101, R94: 47k, Resistor_SMD:R_0603_1608Metric, symbol Device:R_Small_US
- removed R102, R117, R30, R91, R95, R97, R98, R99: 10k, Resistor_SMD:R_0603_1608Metric, symbol Device:R_Small_US
- removed TP1, TP111, TP112, TP156, TP161, TP3, TP62, TP63: Test-Point, oresat-misc:TestPoint_Pad_D1.0mm, symbol oresat-misc:Test-Point-1mm-round
Connections:
- no-connect marks 8 -> 0
Other:
- note removed: "(6.0, 7.2, 8.4)V"
- note removed: "Helical Antenna Deployer"
- note removed: "Main Antenna Deployer (Turnstiles + Monopoles)"
- note removed: "Must not go above 1.8V for Octavo ADC"
