File: kicad/oresat-c3-sch-opd-and-i2c.kicad_sch (KiCad schematic)
At the start: 38 parts, among them Q1 NTR4101P, U12 RCLAMP0504FB, U13 MAX892LEUA+T, U24 RV-3028-C7, U30 FM24CL64B-DGTR, U37 LTC4300A-1

Commit message: Added Oresat symbol lib. Removed any L-band related components from pcb and schematic
Parts:
- renumbered D3 to D10, D2 to D12, R33 to R78, TP1 to TP141, TP1 to TP148, TP1 to TP149, TP109 to TP163, TP1 to TP164, TP1 to TP165, TP1 to TP166, TP1 to TP167, TP1 to TP168, TP1 to TP169, TP63 to TP61
