File: kicad/oresat-c3-sch-opd-and-i2c.kicad_sch (KiCad schematic)
At the start: 38 parts, among them Q1 NTR4101P, U12 RCLAMP0504FB, U13 MAX892LEUA+T, U24 RV-3028-C7, U30 FM24CL64B-DGTR, U37 LTC4300A-1

Commit message: Removed OPD and added LTC4300A to I2C1 bus
Parts:
- removed C129, C79: 1u, Capacitor_SMD:C_0603_1608Metric, symbol Device:C_Small
- removed R52: 23.7k, Resistor_SMD:R_0603_1608Metric, symbol Device:R_Small_US
- removed TP166, TP167, TP61: Test-Point, oresat-misc:TestPoint_Pad_D1.0mm, symbol oresat-misc:Test-Point-1mm-round
- removed U13: MAX892LEUA+T, oresat-ics:LINEAR-MSOP-8-AND-MAXIM-UMAX-8-21-0036, symbol oresat-ics:MAX892LEUA+T
- C131: value 100n -> 10n
- R92, R93: value 4.7k -> 10k
Connections:
- net OPD_PWR is gone; now on net 3.3V: C131.1, R78.2, R92.1, R93.1, TP163.1, U12.5 (VCC), U37.1 (ENABLE), U37.8 (VCC)
- net I2C2_SYS_SCL: no longer U37.3 (SCLIN)
- net I2C2_SYS_SDA: no longer U37.6 (SDAIN)
- net OPD_nENABLE renamed I2C1_SYS_SDA
- net I2C1_SYS_SDA: now also U37.6 (SDAIN)
- net OPD_nFAULT renamed I2C1_SYS_SCL
- net I2C1_SYS_SCL: now also U37.3 (SCLIN)
Other:
- note removed: "Limits OPD_PWR to 50 mA"
- note removed: "Should not go above 1.4V"
- moved on the sheet: R49, R51

Commit message: Finished Labelling CSKB - Removed old UART GNSS Pin, no longer needed - Labelled GPIOs on CSKB 	- Mapped all available GPIOs in BBB Sheet - Labelled UART lines on CSKB
Connections:
- net OPD_SCL renamed I2C1_SCL
- net OPD_SDA renamed I2C1_SDA
Changed lines of the file:
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@@
 		)
 	)
-	(global_label "OPD_SDA"
+	(global_label "I2C1_SDA"
 		(shape bidirectional)
 		(at 278.13 223.52 0)
@@
 		)
 		(property "Intersheetrefs" "${INTERSHEET_REFS}"
-			(at 290.5533 223.52 0)
+			(at 291.056 223.52 0)
 			(effects
 				(font
@@
 		)
 	)
-	(global_label "OPD_SCL"
+	(global_label "I2C1_SCL"
 		(shape output)
 		(at 278.13 219.71 0)
@@
 		)
 		(property "Intersheetrefs" "${INTERSHEET_REFS}"
-			(at 289.3815 219.71 0)
+			(at 289.8842 219.71 0)
 			(effects
 				(font

Commit message: - Grounded FRAM Write protect permanently - Erased old CAN transceivers for unused bus - Fixed CAN termination resistor value to 120 ohm - Redid Clock skew for CAN lines - Removed UART0 from CSKB - Added second I2C buffer for I2C2 bus - Re-routed and placed all I2C bus components 	- Still need to route I2C sys disable, will do later after GPIOs since its lower prio - Added ADCS Enable pin components and routed everything
Parts:
- removed TP160: Test-Point, oresat-misc:TestPoint_Pad_D1.0mm, symbol oresat-misc:Test-Point-1mm-round
- added C3: 10n, Capacitor_SMD:C_0603_1608Metric, symbol Device:C_Small
- added R1, R5, R7, R8: 10k, Resistor_SMD:R_0603_1608Metric, symbol Device:R_Small_US
- added TP5: ~, oresat-misc:TestPoint_Pad_D1.0mm, symbol oresat-misc:Test-Point-1mm-round
- added TP6: TestPoint-MinTH, oresat-misc:TestPoint-0.75mm-th, symbol oresat-misc:Test-Point-0.75mm-th
- added TP7, TP8: Test-Point, oresat-misc:TestPoint_Pad_D1.0mm, symbol oresat-misc:Test-Point-1mm-round
- added U3: LTC4300A-1, oresat-ics:LINEAR-MSOP-8-AND-MAXIM-UMAX-8-21-0036, symbol oresat-ics:LTC4300A-1
- added U4: RCLAMP0504FB, Package_TO_SOT_SMD:SOT-363_SC-70-6, symbol oresat-ics:RCLAMP0504FB
Connections:
- net 3.3V: now also C3.1, R1.1, R5.1, R7.1, R8.1, TP6.1, U3.1 (ENABLE), U3.8 (VCC), U4.5 (VCC)
- net GND: now also U30.7 (WP), C3.2, U3.4 (GND), U4.2 (GND)
- net I2C2_SYS_SCL: now also R1.2, U3.3 (SCLIN)
- net I2C2_SYS_SDA: now also R5.2, U3.6 (SDAIN)
- new net: TP5.1, U3.5 (READY)
- new net I2C2_SCL: R7.2, TP7.1, U3.2 (SCLOUT), U4.1 (I1)
- new net I2C2_SDA: R8.2, TP8.1, U3.7 (SDAOUT), U4.3 (I2)
- no-connect marks 2 -> 4
Other:
- note added: "External I2C Buffers"
- note removed: "OreSat Power Domain (OPD) Control"
- note removed: "To OPD. See Connectors sheet."
- moved on the sheet: C131, D12, R49, R51, R78, R92, R93, TP140, TP163, TP164, TP165, U12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

Commit message: added automotive grade capacitors to the BOM
Parts:
- C115: Description_1 (none) -> CAP CER 100UF 6.3V X5R 1210; Manufacturer_Name (none) -> Murata Electronics; Manufacturer_Part_Number (none) -> GRT32ER60J107ME13L
- C116, C117: Description_1 (none) -> CAP CER 0.1UF 16V X7R 0603; Manufacturer_Name (none) -> Murata Electronics; Manufacturer_Part_Number (none) -> GCJ188R71C104KA01D
- C131, C3: Description_1 (none) -> CAP CER 10NF 16V X7R 0603; Manufacturer_Name (none) -> Samsung Electro-Mechanics; Manufacturer_Part_Number (none) -> CL10B103KO8WPNC
- R1, R49, R5, R51, R66, R7, R78, R79, R8, R92, R93: Description_1 (none) -> RES 10K OHM 1% 1/8W 0603; Manufacturer_Name (none) -> Stackpole Electronics Inc; Manufacturer_Part_Number (none) -> RNCP0603FTD10K0

Commit message: added automotive grade resistors to BOM
Parts:
- R1, R49, R5, R51, R66, R7, R78, R79, R8, R92, R93: Description_1 RES 10K OHM 1% 1/8W 0603 -> RES 0603 10 KOHM 1% 0.125W AUTO; Manufacturer_Part_Number RNCP0603FTD10K0 -> RMCA0603FT10K0-HP
- R67: Description_1 (none) -> RES 0603 150 OHM 1% 0.125W AUTO; Manufacturer_Name (none) -> Stackpole Electronics Inc; Manufacturer_Part_Number (none) -> RMCA0603FT150R-HP
- R68, R80: Description_1 (none) -> RES 0603 4.7 KOHM 1% 0.125W AUTO; Manufacturer_Name (none) -> Stackpole Electronics Inc; Manufacturer_Part_Number (none) -> RMCA0603FT4K70-HP
Changed lines of the file:
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@@
 			)
 		)
-		(property "Description_1" "RES 10K OHM 1% 1/8W 0603"
+		(property "Description_1" "RES 0603 10 KOHM 1% 0.125W AUTO"
 			(at 365.76 212.09 0)
 			(effects
@@
 			)
 		)
-		(property "Manufacturer_Part_Number" "RNCP0603FTD10K0"
+		(property "Manufacturer_Part_Number" "RMCA0603FT10K0-HP"
 			(at 365.76 212.09 0)
 			(effects
@@
 			)
 		)
-		(property "Description_1" "RES 10K OHM 1% 1/8W 0603"
+		(property "Description_1" "RES 0603 10 KOHM 1% 0.125W AUTO"
 			(at 227.33 213.36 0)
 			(effects
@@
 			)
 		)
-		(property "Manufacturer_Part_Number" "RNCP0603FTD10K0"
+		(property "Manufacturer_Part_Number" "RMCA0603FT10K0-HP"
 			(at 227.33 213.36 0)
 			(effects
@@
 			)
 		)
-		(property "Description_1" "RES 10K OHM 1% 1/8W 0603"
+		(property "Description_1" "RES 0603 10 KOHM 1% 0.125W AUTO"
 			(at 207.01 52.07 0)
 			(effects
@@
 			)
 		)
-		(property "Manufacturer_Part_Number" "RNCP0603FTD10K0"
+		(property "Manufacturer_Part_Number" "RMCA0603FT10K0-HP"
 			(at 207.01 52.07 0)
 			(effects
@@
 			)
 		)
-		(property "Description_1" "RES 10K OHM 1% 1/8W 0603"
+		(property "Description_1" "RES 0603 10 KOHM 1% 0.125W AUTO"
 			(at 163.83 168.91 0)
 			(effects
@@
 			)
 		)
-		(property "Manufacturer_Part_Number" "RNCP0603FTD10K0"
+		(property "Manufacturer_Part_Number" "RMCA0603FT10K0-HP"
 			(at 163.83 168.91 0)
 			(effects
@@
 			)
 		)
-		(property "Description_1" ""
+		(property "Description_1" "RES 0603 150 OHM 1% 0.125W AUTO"
+			(at 184.15 69.85 0)
+			(effects
+				(font
+					(size 1.27 1.27)
+				)
+				(hide yes)
+			)
+		)
+		(property "Manufacturer_Name" "Stackpole Electronics Inc"
+			(at 184.15 69.85 0)
+			(effects
+				(font
+					(size 1.27 1.27)
+				)
+				(hide yes)
+			)
+		)
+		(property "Manufacturer_Part_Number" "RMCA0603FT150R-HP"
 			(at 184.15 69.85 0)
 			(effects
@@
 			)
 		)
-		(property "Description_1" "RES 10K OHM 1% 1/8W 0603"
+		(property "Description_1" "RES 0603 10 KOHM 1% 0.125W AUTO"
 			(at 223.52 213.36 0)
 			(effects
@@
 			)
 		)
-		(property "Manufacturer_Part_Number" "RNCP0603FTD10K0"
+		(property "Manufacturer_Part_Number" "RMCA0603FT10K0-HP"
 			(at 223.52 213.36 0)
 			(effects
@@
 			)
 		)
-		(property "Description_1" "RES 10K OHM 1% 1/8W 0603"
+		(property "Description_1" "RES 0603 10 KOHM 1% 0.125W AUTO"
 			(at 280.67 172.72 0)
 			(effects
@@
 			)
 		)
-		(property "Manufacturer_Part_Number" "RNCP0603FTD10K0"
+		(property "Manufacturer_Part_Number" "RMCA0603FT10K0-HP"
 			(at 280.67 172.72 0)
 			(effects
@@
 			)
 		)
-		(property "Description_1" "RES 10K OHM 1% 1/8W 0603"
+		(property "Description_1" "RES 0603 10 KOHM 1% 0.125W AUTO"
 			(at 165.1 110.49 0)
 			(effects
@@
 			)
 		)
-		(property "Manufacturer_Part_Number" "RNCP0603FTD10K0"
+		(property "Manufacturer_Part_Number" "RMCA0603FT10K0-HP"
 			(at 165.1 110.49 0)
 			(effects
@@
 			)
 		)
-		(property "Description_1" ""
+		(property "Description_1" "RES 0603 4.7 KOHM 1% 0.125W AUTO"
+			(at 156.21 90.17 0)
+			(effects
+				(font
+					(size 1.27 1.27)
+				)
+				(hide yes)
+			)
+		)
+		(property "Manufacturer_Name" "Stackpole Electronics Inc"
+			(at 156.21 90.17 0)
+			(effects
+				(font
+					(size 1.27 1.27)
+				)
+				(hide yes)
+			)
+		)
+		(property "Manufacturer_Part_Number" "RMCA0603FT4K70-HP"
 			(at 156.21 90.17 0)
 			(effects
@@
 			)
 		)
-		(property "Description_1" "RES 10K OHM 1% 1/8W 0603"
+		(property "Description_1" "RES 0603 10 KOHM 1% 0.125W AUTO"
 			(at 275.59 171.45 0)
 			(effects
@@
 			)
 		)
-		(property "Manufacturer_Part_Number" "RNCP0603FTD10K0"
+		(property "Manufacturer_Part_Number" "RMCA0603FT10K0-HP"
 			(at 275.59 171.45 0)
 			(effects
@@
 			)
 		)
-		(property "Description_1" ""
+		(property "Description_1" "RES 0603 4.7 KOHM 1% 0.125W AUTO"
+			(at 160.02 90.17 0)
+			(effects
+				(font
+					(size 1.27 1.27)
+				)
+				(hide yes)
+			)
+		)
+		(property "Manufacturer_Name" "Stackpole Electronics Inc"
+			(at 160.02 90.17 0)
+			(effects
+				(font
+					(size 1.27 1.27)
+				)
+				(hide yes)
+			)
+		)
+		(property "Manufacturer_Part_Number" "RMCA0603FT4K70-HP"
 			(at 160.02 90.17 0)
 			(effects
@@
 			)
 		)
-		(property "Description_1" "RES 10K OHM 1% 1/8W 0603"
+		(property "Description_1" "RES 0603 10 KOHM 1% 0.125W AUTO"
 			(at 142.24 173.99 0)
 			(effects
@@
 			)
 		)
-		(property "Manufacturer_Part_Number" "RNCP0603FTD10K0"
+		(property "Manufacturer_Part_Number" "RMCA0603FT10K0-HP"
 			(at 142.24 173.99 0)
 			(effects
@@
 			)
 		)
-		(property "Description_1" "RES 10K OHM 1% 1/8W 0603"
+		(property "Description_1" "RES 0603 10 KOHM 1% 0.125W AUTO"
 			(at 361.95 212.09 0)
 			(effects
@@
 			)
 		)
-		(property "Manufacturer_Part_Number" "RNCP0603FTD10K0"
+		(property "Manufacturer_Part_Number" "RMCA0603FT10K0-HP"
 			(at 361.95 212.09 0)
 			(effects
@@
 			)
 		)
-		(property "Description_1" "RES 10K OHM 1% 1/8W 0603"
+		(property "Description_1" "RES 0603 10 KOHM 1% 0.125W AUTO"
 			(at 137.16 172.72 0)
 			(effects
@@
 			)
 		)
-		(property "Manufacturer_Part_Number" "RNCP0603FTD10K0"
+		(property "Manufacturer_Part_Number" "RMCA0603FT10K0-HP"
 			(at 137.16 172.72 0)
 			(effects

Commit message: modified BOM to match PCBWay format
Parts:
- D10: Description_1 (none) -> DIODE STANDARD 50V 150MA SOD323; Manufacturer_Name (none) -> Vishay General Semiconductor - Diodes Division; Manufacturer_Part_Number (none) -> 1N4151WS-G3-08
- Q1: Description_1 (none) -> MOSFET P-CH 20V 1.8A SOT23-3; Manufacturer_Name (none) -> onsemi; Manufacturer_Part_Number (none) -> NTR4101PT1H
- TP140, TP141, TP148, TP149, TP163, TP164, TP165, TP168, TP169, TP5, TP6, TP7, TP8: now not fitted
- U12, U4: Description_1 (none) -> TVS DIODE 5VWM 17.5VC SC706; Manufacturer_Name (none) -> Semtech Corporation; Manufacturer_Part_Number (none) -> RCLAMP0504FBTCT
- U24: Description_1 (none) -> IC RTC CLK/CALENDAR I2C 8SON; Manufacturer_Name (none) -> Micro Crystal AG; Manufacturer_Part_Number (none) -> RV-3028-C7 32.768KHZ 1PPM-TA-QC
- U3, U37: Description_1 (none) -> IC ACCELERATOR I2C HOTSWAP 8MSOP; Manufacturer_Name (none) -> Analog Devices Inc.; Manufacturer_Part_Number (none) -> LTC4300A-1IMS8#TRPBF
- U30: Description_1 (none) -> IC FRAM 64KBIT I2C 1MHZ 8DFN; Manufacturer_Name (none) -> Infineon Technologies; Manufacturer_Part_Number (none) -> FM24CL64B-DGTR

Commit message: finished putting together BOM, needs review
Parts:
- C115: Description / Value (none) -> CAP CER 100UF 6.3V X5R 1210; Description_1 CAP CER 100UF 6.3V X5R 1210 -> (none)
- C116, C117: Description / Value (none) -> CAP CER 0.1UF 16V X7R 0603; Description_1 CAP CER 0.1UF 16V X7R 0603 -> (none)
- C131, C3: Description / Value (none) -> CAP CER 10NF 16V X7R 0603; Description_1 CAP CER 10NF 16V X7R 0603 -> (none)
- D10: Description / Value (none) -> DIODE STANDARD 50V 150MA SOD323; Description_1 DIODE STANDARD 50V 150MA SOD323 -> (none)
- Q1: Description / Value (none) -> MOSFET P-CH 20V 1.8A SOT23-3; Description_1 MOSFET P-CH 20V 1.8A SOT23-3 -> (none)
- R1, R49, R5, R51, R66, R7, R78, R79, R8, R92, R93: Description / Value (none) -> RES 0603 10 KOHM 1% 0.125W AUTO; Description_1 RES 0603 10 KOHM 1% 0.125W AUTO -> (none)
- R67: Description / Value (none) -> RES 0603 150 OHM 1% 0.125W AUTO; Description_1 RES 0603 150 OHM 1% 0.125W AUTO -> (none)
- R68, R80: Description / Value (none) -> RES 0603 4.7 KOHM 1% 0.125W AUTO; Description_1 RES 0603 4.7 KOHM 1% 0.125W AUTO -> (none)
- U12, U4: Description / Value (none) -> TVS DIODE 5VWM 17.5VC SC706; Description_1 TVS DIODE 5VWM 17.5VC SC706 -> (none)
- U24: Description / Value (none) -> IC RTC CLK/CALENDAR I2C 8SON; Description_1 IC RTC CLK/CALENDAR I2C 8SON -> (none)
- U3, U37: Description / Value (none) -> IC ACCELERATOR I2C HOTSWAP 8MSOP; Description_1 IC ACCELERATOR I2C HOTSWAP 8MSOP -> (none)
- U30: Description / Value (none) -> IC FRAM 64KBIT I2C 1MHZ 8DFN; Description_1 IC FRAM 64KBIT I2C 1MHZ 8DFN -> (none)
