File: kicad/oresat-c3-sch-opd-and-i2c.kicad_sch (KiCad schematic)
At the start: 41 parts, among them Q1 NTR4101P, U12 RCLAMP0504FB, U24 RV-3028-C7, U3 LTC4300A-1, U30 FM24CL64B-DGTR, U37 LTC4300A-1, U4 RCLAMP0504FB

Commit message: - Fixed part number for FRAM, CAN transceiver, emmc, and BJT - Change LED and connected resistors to DNP - Verified remainder of components
Parts:
- D12, R78: now not fitted
- U30: value FM24CL64B-DGTR -> FM24CL64B-GTR; Manufacturer_Part_Number FM24CL64B-DGTR -> FM24CL64B-GTR
Changed lines of the file:
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@@
 			)
 		)
-		(property "Value" "FM24CL64B-DGTR"
+		(property "Value" "FM24CL64B-GTR"
 			(at 240.6141 77.47 0)
 			(effects
@@
 			)
 		)
-		(property "Manufacturer_Part_Number" "FM24CL64B-DGTR"
+		(property "Manufacturer_Part_Number" "FM24CL64B-GTR"
 			(at 242.57 86.36 0)
 			(effects
@@
 		(in_bom yes)
 		(on_board yes)
-		(dnp no)
+		(dnp yes)
 		(property "Reference" "R78"
 			(at 166.37 167.64 0)
@@
 		(in_bom yes)
 		(on_board yes)
-		(dnp no)
+		(dnp yes)
 		(fields_autoplaced yes)
 		(property "Reference" "D12"

Commit message: Finished rerouting CAN
Parts:
- TP140, TP5: value ~ -> (none)
