File: kicad/oresat-c3-sch-osd3358-sip-e-f.kicad_sch (KiCad schematic)
At the start: 5 parts, among them U1 OSD3358-512M-BSM

Commit message: Added Oresat symbol lib. Removed any L-band related components from pcb and schematic
Parts:
- renumbered TP86 to TP19, TP87 to TP20, TP88 to TP21, TP89 to TP22
Changed lines of the file:
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@@
   (symbol (lib_id "power:GND") (at 250.19 125.73 0) (unit 1)
     (in_bom yes) (on_board yes) (dnp no)
-    (property "Reference" "#GND0172" (at 250.19 132.08 0)
+    (property "Reference" "#PWR0163" (at 250.19 132.08 0)
       (effects (font (size 1.27 1.27)) hide)
     )
@@
     (instances
       (project "oresat-c3"
-        (path "/65d12cdd-c326-4033-9053-c59fa4e0b25e/0c1da208-2d1c-4d05-9cc7-59584e50a6ac"
-          (reference "#GND0172") (unit 1)
-        )
         (path "/65d12cdd-c326-4033-9053-c59fa4e0b25e/ce2d6150-524f-4c6f-aba3-da83a5df548c"
           (reference "#PWR0163") (unit 1)
@@
   (symbol (lib_id "power:GND") (at 184.15 125.73 0) (unit 1)
     (in_bom yes) (on_board yes) (dnp no)
-    (property "Reference" "#GND0173" (at 184.15 132.08 0)
+    (property "Reference" "#PWR0162" (at 184.15 132.08 0)
       (effects (font (size 1.27 1.27)) hide)
     )
@@
     (instances
       (project "oresat-c3"
-        (path "/65d12cdd-c326-4033-9053-c59fa4e0b25e/0c1da208-2d1c-4d05-9cc7-59584e50a6ac"
-          (reference "#GND0173") (unit 1)
-        )
         (path "/65d12cdd-c326-4033-9053-c59fa4e0b25e/ce2d6150-524f-4c6f-aba3-da83a5df548c"
           (reference "#PWR0162") (unit 1)
@@
     (instances
       (project "oresat-c3"
-        (path "/65d12cdd-c326-4033-9053-c59fa4e0b25e/0c1da208-2d1c-4d05-9cc7-59584e50a6ac"
-          (reference "U1") (unit 6)
-        )
         (path "/65d12cdd-c326-4033-9053-c59fa4e0b25e/ce2d6150-524f-4c6f-aba3-da83a5df548c"
           (reference "U1") (unit 6)
@@
   (symbol (lib_id "oresat-misc:Test-Point-1mm-round") (at 187.96 162.56 0) (unit 1)
     (in_bom yes) (on_board yes) (dnp no)
-    (property "Reference" "TP86" (at 181.61 162.56 0)
+    (property "Reference" "TP19" (at 181.61 162.56 0)
       (effects (font (size 1.27 1.27)) (justify left))
     )
@@
     (instances
       (project "oresat-c3"
-        (path "/65d12cdd-c326-4033-9053-c59fa4e0b25e/0c1da208-2d1c-4d05-9cc7-59584e50a6ac"
-          (reference "TP86") (unit 1)
-        )
         (path "/65d12cdd-c326-4033-9053-c59fa4e0b25e/ce2d6150-524f-4c6f-aba3-da83a5df548c"
           (reference "TP19") (unit 1)
@@
   (symbol (lib_id "oresat-misc:Test-Point-1mm-round") (at 187.96 167.64 0) (unit 1)
     (in_bom yes) (on_board yes) (dnp no)
-    (property "Reference" "TP87" (at 181.61 167.64 0)
+    (property "Reference" "TP20" (at 181.61 167.64 0)
       (effects (font (size 1.27 1.27)) (justify left))
     )
@@
     (instances
       (project "oresat-c3"
-        (path "/65d12cdd-c326-4033-9053-c59fa4e0b25e/0c1da208-2d1c-4d05-9cc7-59584e50a6ac"
-          (reference "TP87") (unit 1)
-        )
         (path "/65d12cdd-c326-4033-9053-c59fa4e0b25e/ce2d6150-524f-4c6f-aba3-da83a5df548c"
           (reference "TP20") (unit 1)
@@
   (symbol (lib_id "oresat-misc:Test-Point-1mm-round") (at 187.96 177.8 0) (unit 1)
     (in_bom yes) (on_board yes) (dnp no)
-    (property "Reference" "TP89" (at 181.61 177.8 0)
+    (property "Reference" "TP22" (at 181.61 177.8 0)
       (effects (font (size 1.27 1.27)) (justify left))
     )
@@
     (instances
       (project "oresat-c3"
-        (path "/65d12cdd-c326-4033-9053-c59fa4e0b25e/0c1da208-2d1c-4d05-9cc7-59584e50a6ac"
-          (reference "TP89") (unit 1)
-        )
         (path "/65d12cdd-c326-4033-9053-c59fa4e0b25e/ce2d6150-524f-4c6f-aba3-da83a5df548c"
           (reference "TP22") (unit 1)
@@
   (symbol (lib_id "oresat-misc:Test-Point-1mm-round") (at 187.96 172.72 0) (unit 1)
     (in_bom yes) (on_board yes) (dnp no)
-    (property "Reference" "TP88" (at 181.61 172.72 0)
+    (property "Reference" "TP21" (at 181.61 172.72 0)
       (effects (font (size 1.27 1.27)) (justify left))
     )
@@
     (instances
       (project "oresat-c3"
-        (path "/65d12cdd-c326-4033-9053-c59fa4e0b25e/0c1da208-2d1c-4d05-9cc7-59584e50a6ac"
-          (reference "TP88") (unit 1)
-        )
         (path "/65d12cdd-c326-4033-9053-c59fa4e0b25e/ce2d6150-524f-4c6f-aba3-da83a5df548c"
           (reference "TP21") (unit 1)
@@
     (instances
       (project "oresat-c3"
-        (path "/65d12cdd-c326-4033-9053-c59fa4e0b25e/0c1da208-2d1c-4d05-9cc7-59584e50a6ac"
-          (reference "U1") (unit 5)
-        )
         (path "/65d12cdd-c326-4033-9053-c59fa4e0b25e/ce2d6150-524f-4c6f-aba3-da83a5df548c"
           (reference "U1") (unit 5)
