File: kicad/oresat-c3-sch-osd3358-sip-e-f.kicad_sch (KiCad schematic)
At the start: 5 parts, among them U1 OSD3358-512M-BSM

Commit message: modified BOM to match PCBWay format
Parts:
- TP19, TP20, TP21, TP22: now not fitted
Changed lines of the file:
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@@
 		(in_bom yes)
 		(on_board yes)
-		(dnp no)
+		(dnp yes)
 		(property "Reference" "TP19"
 			(at 181.61 162.56 0)
@@
 		(in_bom yes)
 		(on_board yes)
-		(dnp no)
+		(dnp yes)
 		(property "Reference" "TP20"
 			(at 181.61 167.64 0)
@@
 		(in_bom yes)
 		(on_board yes)
-		(dnp no)
+		(dnp yes)
 		(property "Reference" "TP22"
 			(at 181.61 177.8 0)
@@
 		(in_bom yes)
 		(on_board yes)
-		(dnp no)
+		(dnp yes)
 		(property "Reference" "TP21"
 			(at 181.61 172.72 0)

Commit message: finished putting together BOM, needs review
Parts:
- U1: value OSD3358-512M-BSM -> OSD3358-512M-ISM; Description / Value (none) -> IC MODULE CORTEX-A8 1GHZ 512MB; Manufacturer_Name (none) -> Octavo Systems LLC; Manufacturer_Part_Number (none) -> OSD3358-512M-ISM
Changed lines of the file:
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@@
 			)
 		)
-		(property "Value" "OSD3358-512M-BSM"
+		(property "Value" "OSD3358-512M-ISM"
 			(at 218.44 154.94 0)
 			(effects
@@
 			)
 		)
-		(property "Datasheet" ""
+		(property "Datasheet" "https://mm.digikey.com/Volume0/opasdata/d220001/medias/docus/778/OSd335x-Software-PwrMgmt.pdf"
 			(at 218.44 182.88 0)
 			(effects
@@
 		)
 		(property "Total Price" ""
+			(at 218.44 182.88 0)
+			(effects
+				(font
+					(size 1.27 1.27)
+				)
+				(hide yes)
+			)
+		)
+		(property "Manufacturer_Part_Number" "OSD3358-512M-ISM"
+			(at 218.44 182.88 0)
+			(effects
+				(font
+					(size 1.27 1.27)
+				)
+				(hide yes)
+			)
+		)
+		(property "Manufacturer_Name" "Octavo Systems LLC"
+			(at 218.44 182.88 0)
+			(effects
+				(font
+					(size 1.27 1.27)
+				)
+				(hide yes)
+			)
+		)
+		(property "Description / Value" "IC MODULE CORTEX-A8 1GHZ 512MB"
 			(at 218.44 182.88 0)
 			(effects
@@
 			)
 		)
-		(property "Value" "OSD3358-512M-BSM"
+		(property "Value" "OSD3358-512M-ISM"
 			(at 217.17 54.61 0)
 			(effects
@@
 			)
 		)
-		(property "Datasheet" ""
+		(property "Datasheet" "https://mm.digikey.com/Volume0/opasdata/d220001/medias/docus/778/OSd335x-Software-PwrMgmt.pdf"
 			(at 217.17 87.63 0)
 			(effects
@@
 			(at 217.17 87.63 0)
 			(effects
+				(font
+					(size 1.27 1.27)
+				)
+				(hide yes)
+			)
+		)
+		(property "Manufacturer_Part_Number" "OSD3358-512M-ISM"
+			(at 217.17 87.63 0)
+			(effects
+				(font
+					(size 1.27 1.27)
+				)
+				(hide yes)
+			)
+		)
+		(property "Manufacturer_Name" "Octavo Systems LLC"
+			(at 217.17 87.63 0)
+			(effects
+				(font
+					(size 1.27 1.27)
+				)
+				(hide yes)
+			)
+		)
+		(property "Description / Value" "IC MODULE CORTEX-A8 1GHZ 512MB"
+			(at 217.17 87.63 0)
+			(effects

Commit message: Fixed some BOM issues. Board has been ordered, generated production files
Parts:
- U1: MPN OSD3358-512M-BSM -> OSD3358-512M-ISM
Changed lines of the file:
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@@
 			)
 		)
-		(property "MPN" "OSD3358-512M-BSM"
+		(property "MPN" "OSD3358-512M-ISM"
 			(at 218.44 83.82 0)
 			(effects
@@
 			)
 		)
-		(property "MPN" "OSD3358-512M-BSM"
+		(property "MPN" "OSD3358-512M-ISM"
 			(at 217.17 -11.43 0)
 			(effects
