File: kicad/oresat-c3-sch-osd3358-usb-xtal.kicad_sch (KiCad schematic)
At the start: 36 parts, among them U1 OSD3358-512M-BSM, U11 RCLAMP0504FB, Y1 ECS-240-12-30BQ-AEN-TR, Y2 ABS07-32.768KHZ-T

Commit message: Added CAN bus termination resistors
Connections:
- net OPD_CURRENT: no longer names the net of U1.B6 (AIN2)
Changed lines of the file:
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@@
-		)
-	)
-	(global_label "OPD_CURRENT"
-		(shape input)
-		(at 271.78 127 0)
-		(fields_autoplaced yes)
-		(effects
-			(font
-				(size 1.27 1.27)
-			)
-			(justify left)
-		)
-		(property "Intersheetrefs" "${INTERSHEET_REFS}"
-			(at 288.1115 127 0)
-			(effects
-				(font
-					(size 1.27 1.27)
-				)
-				(justify left)
-			)
 		)
 	)

Commit message: Added extra decoupling capacitor to MRAM. Also grounded all unused pins and mounting holes
Connections:
- no-connect marks 1 -> 7
Changed lines of the file:
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@@
+	)
+	(no_connect
+		(at 271.78 132.08)
+	)
+	(no_connect
+		(at 271.78 134.62)
+	)
+	(no_connect
+		(at 271.78 124.46)
 	)
 	(no_connect
 		(at 191.77 210.82)
 	)
+	(no_connect
+		(at 271.78 121.92)
+	)
+	(no_connect
+		(at 271.78 129.54)
+	)
+	(no_connect
+		(at 271.78 127)
+	)
 	(polyline

Commit message: added automotive grade capacitors to the BOM
Parts:
- C26, C27: Description_1 (none) -> CAP CER 10PF 16V X7R 0603; Manufacturer_Name (none) -> KEMET; Manufacturer_Part_Number (none) -> C0603C100K4RACAUTO
- C28, C29: Description_1 (none) -> CAP CER 18PF 50V C0G/NP0 0603; Manufacturer_Name (none) -> Murata Electronics; Manufacturer_Part_Number (none) -> GCM1885C1H180JA16D
- C30, C32: Description_1 (none) -> CAP CER 0.1UF 16V X7R 0603; Manufacturer_Name (none) -> Murata Electronics; Manufacturer_Part_Number (none) -> GCJ188R71C104KA01D
- C31: Description_1 (none) -> CAP CER 1000PF 50V X7R 0603; Manufacturer_Name (none) -> Murata Electronics; Manufacturer_Part_Number (none) -> GCM188R71H102KA37D
- R46: now fitted
- R75, R76, R77: Description_1 (none) -> RES 10K OHM 1% 1/8W 0603; Manufacturer_Name (none) -> Stackpole Electronics Inc; Manufacturer_Part_Number (none) -> RNCP0603FTD10K0

Commit message: added automotive grade resistors to BOM
Parts:
- R47: Description_1 (none) -> RES 0603 1 MOHM 1% 0.125W AUTO; Manufacturer_Name (none) -> Stackpole Electronics Inc; Manufacturer_Part_Number (none) -> RMCA0603FT1M00-HP
- R75, R76, R77: Description_1 RES 10K OHM 1% 1/8W 0603 -> RES 0603 10 KOHM 1% 0.125W AUTO; Manufacturer_Part_Number RNCP0603FTD10K0 -> RMCA0603FT10K0-HP
Changed lines of the file:
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@@
 			)
 		)
-		(property "Description_1" "RES 10K OHM 1% 1/8W 0603"
+		(property "Description_1" "RES 0603 10 KOHM 1% 0.125W AUTO"
 			(at 166.37 138.43 0)
 			(effects
@@
 			)
 		)
-		(property "Manufacturer_Part_Number" "RNCP0603FTD10K0"
+		(property "Manufacturer_Part_Number" "RMCA0603FT10K0-HP"
 			(at 166.37 138.43 0)
 			(effects
@@
 			)
 		)
-		(property "Description_1" "RES 10K OHM 1% 1/8W 0603"
+		(property "Description_1" "RES 0603 10 KOHM 1% 0.125W AUTO"
 			(at 171.45 138.43 0)
 			(effects
@@
 			)
 		)
-		(property "Manufacturer_Part_Number" "RNCP0603FTD10K0"
+		(property "Manufacturer_Part_Number" "RMCA0603FT10K0-HP"
 			(at 171.45 138.43 0)
 			(effects
@@
 			)
 		)
-		(property "Description_1" ""
+		(property "Description_1" "RES 0603 1 MOHM 1% 0.125W AUTO"
+			(at 180.34 81.28 0)
+			(effects
+				(font
+					(size 1.27 1.27)
+				)
+				(hide yes)
+			)
+		)
+		(property "Manufacturer_Name" "Stackpole Electronics Inc"
+			(at 180.34 81.28 0)
+			(effects
+				(font
+					(size 1.27 1.27)
+				)
+				(hide yes)
+			)
+		)
+		(property "Manufacturer_Part_Number" "RMCA0603FT1M00-HP"
 			(at 180.34 81.28 0)
 			(effects
@@
 			)
 		)
-		(property "Description_1" "RES 10K OHM 1% 1/8W 0603"
+		(property "Description_1" "RES 0603 10 KOHM 1% 0.125W AUTO"
 			(at 158.75 148.59 0)
 			(effects
@@
 			)
 		)
-		(property "Manufacturer_Part_Number" "RNCP0603FTD10K0"
+		(property "Manufacturer_Part_Number" "RMCA0603FT10K0-HP"
 			(at 158.75 148.59 0)
 			(effects

Commit message: modified BOM to match PCBWay format
Parts:
- TP100, TP104, TP137, TP138, TP139, TP59, TP67, TP69, TP70, TP71, TP72, TP91, TP92, TP93, TP94, TP95, TP96, TP97, TP98, TP99: now not fitted
- U11: Description_1 (none) -> TVS DIODE 5VWM 17.5VC SC706; Manufacturer_Name (none) -> Semtech Corporation; Manufacturer_Part_Number (none) -> RCLAMP0504FBTCT
- Y1: Description_1 (none) -> CRYSTAL 24.0000MHZ 12PF SMD; Manufacturer_Name (none) -> ECS Inc.; Manufacturer_Part_Number (none) -> ECS-240-12-30BQ-AEN-TR
- Y2: Description_1 (none) -> CRYSTAL 32.7680KHZ 12.5PF SMD; Manufacturer_Name (none) -> Abracon LLC; Manufacturer_Part_Number (none) -> ABS07-32.768KHZ-T
Changed lines of the file:
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@@
 			)
 		)
+		(property "Description_1" "CRYSTAL 24.0000MHZ 12PF SMD"
+			(at 166.37 81.28 90)
+			(effects
+				(font
+					(size 1.27 1.27)
+				)
+				(hide yes)
+			)
+		)
+		(property "Manufacturer_Name" "ECS Inc."
+			(at 166.37 81.28 90)
+			(effects
+				(font
+					(size 1.27 1.27)
+				)
+				(hide yes)
+			)
+		)
+		(property "Manufacturer_Part_Number" "ECS-240-12-30BQ-AEN-TR"
+			(at 166.37 81.28 90)
+			(effects
+				(font
+					(size 1.27 1.27)
+				)
+				(hide yes)
+			)
+		)
 		(pin "1"
 		)
@@
 		(in_bom yes)
 		(on_board yes)
-		(dnp no)
+		(dnp yes)
 		(property "Reference" "TP70"
 			(at 270.51 149.86 0)
@@
 		(in_bom yes)
 		(on_board yes)
-		(dnp no)
+		(dnp yes)
 		(property "Reference" "TP94"
 			(at 186.69 142.24 0)
@@
 		(in_bom yes)
 		(on_board yes)
-		(dnp no)
+		(dnp yes)
 		(property "Reference" "TP91"
 			(at 186.69 134.62 0)
@@
 			)
 		)
+		(property "Description_1" "CRYSTAL 32.7680KHZ 12.5PF SMD"
+			(at 167.64 111.76 90)
+			(effects
+				(font
+					(size 1.27 1.27)
+				)
+				(hide yes)
+			)
+		)
+		(property "Manufacturer_Name" "Abracon LLC"
+			(at 167.64 111.76 90)
+			(effects
+				(font
+					(size 1.27 1.27)
+				)
+				(hide yes)
+			)
+		)
+		(property "Manufacturer_Part_Number" "ABS07-32.768KHZ-T"
+			(at 167.64 111.76 90)
+			(effects
+				(font
+					(size 1.27 1.27)
+				)
+				(hide yes)
+			)
+		)
 		(pin "1"
 		)
@@
 		(in_bom yes)
 		(on_board yes)
-		(dnp no)
+		(dnp yes)
 		(property "Reference" "TP92"
 			(at 186.69 137.16 0)
@@
 		(in_bom yes)
 		(on_board yes)
-		(dnp no)
+		(dnp yes)
 		(property "Reference" "TP72"
 			(at 270.51 172.72 0)
@@
 		(in_bom yes)
 		(on_board yes)
-		(dnp no)
+		(dnp yes)
 		(property "Reference" "TP98"
 			(at 270.51 165.1 0)
@@
 		(in_bom yes)
 		(on_board yes)
-		(dnp no)
+		(dnp yes)
 		(property "Reference" "TP96"
 			(at 186.69 149.86 0)
@@
 		(in_bom yes)
 		(on_board yes)
-		(dnp no)
+		(dnp yes)
 		(property "Reference" "TP104"
 			(at 186.69 147.32 0)
@@
 			)
 		)
+		(property "Description_1" "TVS DIODE 5VWM 17.5VC SC706"
+			(at 200.66 207.01 0)
+			(effects
+				(font
+					(size 1.27 1.27)
+				)
+				(hide yes)
+			)
+		)
+		(property "Manufacturer_Name" "Semtech Corporation"
+			(at 200.66 207.01 0)
+			(effects
+				(font
+					(size 1.27 1.27)
+				)
+				(hide yes)
+			)
+		)
+		(property "Manufacturer_Part_Number" "RCLAMP0504FBTCT"
+			(at 200.66 207.01 0)
+			(effects
+				(font
+					(size 1.27 1.27)
+				)
+				(hide yes)
+			)
+		)
 		(pin "1"
 		)
@@
 		(in_bom yes)
 		(on_board yes)
-		(dnp no)
+		(dnp yes)
 		(property "Reference" "TP100"
 			(at 271.78 160.02 0)
@@
 		(in_bom yes)
 		(on_board yes)
-		(dnp no)
+		(dnp yes)
 		(property "Reference" "TP137"
 			(at 180.34 167.64 0)
@@
 		(in_bom yes)
 		(on_board yes)
-		(dnp no)
+		(dnp yes)
 		(property "Reference" "TP69"
 			(at 270.51 144.78 0)
@@
 		(in_bom yes)
 		(on_board yes)
-		(dnp no)
+		(dnp yes)
 		(property "Reference" "TP138"
 			(at 180.34 170.18 0)
@@
 		(in_bom yes)
 		(on_board yes)
-		(dnp no)
+		(dnp yes)
 		(property "Reference" "TP99"
 			(at 270.51 162.56 0)
@@
 		(in_bom yes)
 		(on_board yes)
-		(dnp no)
+		(dnp yes)
 		(property "Reference" "TP95"
 			(at 186.69 144.78 0)
@@
 		(in_bom yes)
 		(on_board yes)
-		(dnp no)
+		(dnp yes)
 		(property "Reference" "TP93"
 			(at 186.69 139.7 0)
@@
 		(in_bom yes)
 		(on_board yes)
-		(dnp no)
+		(dnp yes)
 		(property "Reference" "TP97"
 			(at 270.51 167.64 0)
@@
 		(in_bom yes)
 		(on_board yes)
-		(dnp no)
+		(dnp yes)
 		(property "Reference" "TP59"
 			(at 264.16 68.58 0)
@@
 		(in_bom yes)
 		(on_board yes)
-		(dnp no)
+		(dnp yes)
 		(property "Reference" "TP71"
 			(at 270.51 170.18 0)
@@
 		(in_bom yes)
 		(on_board yes)
-		(dnp no)
+		(dnp yes)
 		(property "Reference" "TP67"
 			(at 270.51 137.16 0)
@@
 		(in_bom yes)
 		(on_board yes)
-		(dnp no)
+		(dnp yes)
 		(property "Reference" "TP139"
 			(at 180.34 172.72 0)

Commit message: finished putting together BOM, needs review
Parts:
- C26, C27: Description / Value (none) -> CAP CER 10PF 16V X7R 0603; Description_1 CAP CER 10PF 16V X7R 0603 -> (none)
- C28, C29: Description / Value (none) -> CAP CER 18PF 50V C0G/NP0 0603; Description_1 CAP CER 18PF 50V C0G/NP0 0603 -> (none)
- C30, C32: Description / Value (none) -> CAP CER 0.1UF 16V X7R 0603; Description_1 CAP CER 0.1UF 16V X7R 0603 -> (none)
- C31: Description / Value (none) -> CAP CER 1000PF 50V X7R 0603; Description_1 CAP CER 1000PF 50V X7R 0603 -> (none)
- R46: now not fitted
- R47: Description / Value (none) -> RES 0603 1 MOHM 1% 0.125W AUTO; Description_1 RES 0603 1 MOHM 1% 0.125W AUTO -> (none)
- R75, R76, R77: Description / Value (none) -> RES 0603 10 KOHM 1% 0.125W AUTO; Description_1 RES 0603 10 KOHM 1% 0.125W AUTO -> (none)
- U1: value OSD3358-512M-BSM -> OSD3358-512M-ISM; Description / Value (none) -> IC MODULE CORTEX-A8 1GHZ 512MB; Manufacturer_Name (none) -> Octavo Systems LLC; Manufacturer_Part_Number (none) -> OSD3358-512M-ISM
- U11: Description / Value (none) -> TVS DIODE 5VWM 17.5VC SC706; Description_1 TVS DIODE 5VWM 17.5VC SC706 -> (none)
- Y1: Description / Value (none) -> CRYSTAL 24.0000MHZ 12PF SMD; Description_1 CRYSTAL 24.0000MHZ 12PF SMD -> (none)
- Y2: Description / Value (none) -> CRYSTAL 32.7680KHZ 12.5PF SMD; Description_1 CRYSTAL 32.7680KHZ 12.5PF SMD -> (none)
Changed lines of the file:
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@@
 			)
 		)
-		(property "Description_1" "CRYSTAL 24.0000MHZ 12PF SMD"
+		(property "Manufacturer_Name" "ECS Inc."
 			(at 166.37 81.28 90)
 			(effects
@@
 			)
 		)
-		(property "Manufacturer_Name" "ECS Inc."
+		(property "Manufacturer_Part_Number" "ECS-240-12-30BQ-AEN-TR"
 			(at 166.37 81.28 90)
 			(effects
@@
 			)
 		)
-		(property "Manufacturer_Part_Number" "ECS-240-12-30BQ-AEN-TR"
+		(property "Description / Value" "CRYSTAL 24.0000MHZ 12PF SMD"
 			(at 166.37 81.28 90)
 			(effects
@@
 			)
 		)
-		(property "Description_1" "CRYSTAL 32.7680KHZ 12.5PF SMD"
+		(property "Manufacturer_Name" "Abracon LLC"
 			(at 167.64 111.76 90)
 			(effects
@@
 			)
 		)
-		(property "Manufacturer_Name" "Abracon LLC"
+		(property "Manufacturer_Part_Number" "ABS07-32.768KHZ-T"
 			(at 167.64 111.76 90)
 			(effects
@@
 			)
 		)
-		(property "Manufacturer_Part_Number" "ABS07-32.768KHZ-T"
+		(property "Description / Value" "CRYSTAL 32.7680KHZ 12.5PF SMD"
 			(at 167.64 111.76 90)
 			(effects
@@
 			)
 		)
-		(property "Description_1" "CAP CER 10PF 16V X7R 0603"
+		(property "Manufacturer_Name" "KEMET"
 			(at 153.67 88.9 90)
 			(effects
@@
 			)
 		)
-		(property "Manufacturer_Name" "KEMET"
+		(property "Manufacturer_Part_Number" "C0603C100K4RACAUTO"
 			(at 153.67 88.9 90)
 			(effects
@@
 			)
 		)
-		(property "Manufacturer_Part_Number" "C0603C100K4RACAUTO"
+		(property "Description / Value" "CAP CER 10PF 16V X7R 0603"
 			(at 153.67 88.9 90)
 			(effects
@@
 			)
 		)
-		(property "Description_1" "RES 0603 10 KOHM 1% 0.125W AUTO"
+		(property "Manufacturer_Name" "Stackpole Electronics Inc"
 			(at 166.37 138.43 0)
 			(effects
@@
 			)
 		)
-		(property "Manufacturer_Name" "Stackpole Electronics Inc"
+		(property "Manufacturer_Part_Number" "RMCA0603FT10K0-HP"
 			(at 166.37 138.43 0)
 			(effects
@@
 			)
 		)
-		(property "Manufacturer_Part_Number" "RMCA0603FT10K0-HP"
+		(property "Description / Value" "RES 0603 10 KOHM 1% 0.125W AUTO"
 			(at 166.37 138.43 0)
 			(effects
@@
 		(in_bom yes)
 		(on_board yes)
-		(dnp no)
+		(dnp yes)
 		(property "Reference" "R46"
 			(at 181.61 110.4899 0)
@@
 			)
 		)
-		(property "Description_1" ""
-			(at 179.07 111.76 0)
-			(effects
-				(font
-					(size 1.27 1.27)
-				)
-				(hide yes)
-			)
-		)
 		(pin "1"
 		)
@@
 			)
 		)
-		(property "Description_1" "TVS DIODE 5VWM 17.5VC SC706"
+		(property "Manufacturer_Name" "Semtech Corporation"
 			(at 200.66 207.01 0)
 			(effects
@@
 			)
 		)
-		(property "Manufacturer_Name" "Semtech Corporation"
+		(property "Manufacturer_Part_Number" "RCLAMP0504FBTCT"
 			(at 200.66 207.01 0)
 			(effects
@@
 			)
 		)
-		(property "Manufacturer_Part_Number" "RCLAMP0504FBTCT"
+		(property "Description / Value" "TVS DIODE 5VWM 17.5VC SC706"
 			(at 200.66 207.01 0)
 			(effects
@@
 			)
 		)
-		(property "Description_1" "CAP CER 0.1UF 16V X7R 0603"
+		(property "Manufacturer_Name" "Murata Electronics"
 			(at 215.9 196.85 0)
 			(effects
@@
 			)
 		)
-		(property "Manufacturer_Name" "Murata Electronics"
+		(property "Manufacturer_Part_Number" "GCJ188R71C104KA01D"
 			(at 215.9 196.85 0)
 			(effects
@@
 			)
 		)
-		(property "Manufacturer_Part_Number" "GCJ188R71C104KA01D"
+		(property "Description / Value" "CAP CER 0.1UF 16V X7R 0603"
 			(at 215.9 196.85 0)
 			(effects
@@
 			)
 		)
-		(property "Description_1" "CAP CER 18PF 50V C0G/NP0 0603"
+		(property "Manufacturer_Name" "Murata Electronics"
 			(at 160.02 119.38 90)
 			(effects
@@
 			)
 		)
-		(property "Manufacturer_Name" "Murata Electronics"
+		(property "Manufacturer_Part_Number" "GCM1885C1H180JA16D"
 			(at 160.02 119.38 90)
 			(effects
@@
 			)
 		)
-		(property "Manufacturer_Part_Number" "GCM1885C1H180JA16D"
+		(property "Description / Value" "CAP CER 18PF 50V C0G/NP0 0603"
 			(at 160.02 119.38 90)
 			(effects
@@
 			)
 		)
-		(property "Value" "OSD3358-512M-BSM"
+		(property "Value" "OSD3358-512M-ISM"
 			(at 226.06 55.88 0)
 			(effects
@@
 			)
 		)
-		(property "Datasheet" ""
+		(property "Datasheet" "https://mm.digikey.com/Volume0/opasdata/d220001/medias/docus/778/OSd335x-Software-PwrMgmt.pdf"
 			(at 226.06 116.84 0)
 			(effects
@@
 			)
 		)
+		(property "Manufacturer_Part_Number" "OSD3358-512M-ISM"
+			(at 226.06 116.84 0)
+			(effects
+				(font
+					(size 1.27 1.27)
+				)
+				(hide yes)
+			)
+		)
+		(property "Manufacturer_Name" "Octavo Systems LLC"
+			(at 226.06 116.84 0)
+			(effects
+				(font
+					(size 1.27 1.27)
+				)
+				(hide yes)
+			)
+		)
+		(property "Description / Value" "IC MODULE CORTEX-A8 1GHZ 512MB"
+			(at 226.06 116.84 0)
+			(effects
+				(font
+					(size 1.27 1.27)
+				)
+				(hide yes)
+			)
+		)
 		(pin "C10"
 		)
@@
 			)
 		)
-		(property "Description_1" "CAP CER 18PF 50V C0G/NP0 0603"
+		(property "Manufacturer_Name" "Murata Electronics"
 			(at 160.02 104.14 90)
 			(effects
@@
 			)
 		)
-		(property "Manufacturer_Name" "Murata Electronics"
+		(property "Manufacturer_Part_Number" "GCM1885C1H180JA16D"
 			(at 160.02 104.14 90)
 			(effects
@@
 			)
 		)
-		(property "Manufacturer_Part_Number" "GCM1885C1H180JA16D"
+		(property "Description / Value" "CAP CER 18PF 50V C0G/NP0 0603"
 			(at 160.02 104.14 90)
 			(effects
@@
 			)
 		)
-		(property "Description_1" "CAP CER 1000PF 50V X7R 0603"
+		(property "Manufacturer_Name" "Murata Electronics"
 			(at 257.81 91.44 0)
 			(effects
@@
 			)
 		)
-		(property "Manufacturer_Name" "Murata Electronics"
+		(property "Manufacturer_Part_Number" "GCM188R71H102KA37D"
 			(at 257.81 91.44 0)
 			(effects
@@
 			)
 		)
-		(property "Manufacturer_Part_Number" "GCM188R71H102KA37D"
+		(property "Description / Value" "CAP CER 1000PF 50V X7R 0603"
 			(at 257.81 91.44 0)
 			(effects
@@
 			)
 		)
-		(property "Description_1" "CAP CER 0.1UF 16V X7R 0603"
+		(property "Manufacturer_Name" "Murata Electronics"
 			(at 265.43 91.44 0)
 			(effects
@@
 			)
 		)
-		(property "Manufacturer_Name" "Murata Electronics"
+		(property "Manufacturer_Part_Number" "GCJ188R71C104KA01D"
 			(at 265.43 91.44 0)
 			(effects
@@
 			)
 		)
-		(property "Manufacturer_Part_Number" "GCJ188R71C104KA01D"
+		(property "Description / Value" "CAP CER 0.1UF 16V X7R 0603"
 			(at 265.43 91.44 0)
 			(effects
@@
 			)
 		)
-		(property "Description_1" "RES 0603 10 KOHM 1% 0.125W AUTO"
+		(property "Manufacturer_Name" "Stackpole Electronics Inc"
 			(at 171.45 138.43 0)
 			(effects
@@
 			)
 		)
-		(property "Manufacturer_Name" "Stackpole Electronics Inc"
+		(property "Manufacturer_Part_Number" "RMCA0603FT10K0-HP"
 			(at 171.45 138.43 0)
 			(effects
@@
 			)
 		)
-		(property "Manufacturer_Part_Number" "RMCA0603FT10K0-HP"
+		(property "Description / Value" "RES 0603 10 KOHM 1% 0.125W AUTO"
 			(at 171.45 138.43 0)
 			(effects
@@
 			)
 		)
-		(property "Description_1" "CAP CER 10PF 16V X7R 0603"
+		(property "Manufacturer_Name" "KEMET"
 			(at 153.67 73.66 90)
 			(effects
@@
 			)
 		)
-		(property "Manufacturer_Name" "KEMET"
+		(property "Manufacturer_Part_Number" "C0603C100K4RACAUTO"
 			(at 153.67 73.66 90)
 			(effects
@@
 			)
 		)
-		(property "Manufacturer_Part_Number" "C0603C100K4RACAUTO"
+		(property "Description / Value" "CAP CER 10PF 16V X7R 0603"
 			(at 153.67 73.66 90)
 			(effects
@@
 			)
 		)
-		(property "Description_1" "RES 0603 1 MOHM 1% 0.125W AUTO"
+		(property "Manufacturer_Name" "Stackpole Electronics Inc"
 			(at 180.34 81.28 0)
 			(effects
@@
 			)
 		)
-		(property "Manufacturer_Name" "Stackpole Electronics Inc"
+		(property "Manufacturer_Part_Number" "RMCA0603FT1M00-HP"
 			(at 180.34 81.28 0)
 			(effects
@@
 			)
 		)
-		(property "Manufacturer_Part_Number" "RMCA0603FT1M00-HP"
+		(property "Description / Value" "RES 0603 1 MOHM 1% 0.125W AUTO"
 			(at 180.34 81.28 0)
 			(effects
@@
 			)
 		)
-		(property "Description_1" "RES 0603 10 KOHM 1% 0.125W AUTO"
+		(property "Manufacturer_Name" "Stackpole Electronics Inc"
 			(at 158.75 148.59 0)
 			(effects
@@
 			)
 		)
-		(property "Manufacturer_Name" "Stackpole Electronics Inc"
+		(property "Manufacturer_Part_Number" "RMCA0603FT10K0-HP"
 			(at 158.75 148.59 0)
 			(effects
@@
 			)
 		)
-		(property "Manufacturer_Part_Number" "RMCA0603FT10K0-HP"
+		(property "Description / Value" "RES 0603 10 KOHM 1% 0.125W AUTO"
 			(at 158.75 148.59 0)
 			(effects

Commit message: Fixed some BOM issues. Board has been ordered, generated production files
Parts:
- U1: MPN OSD3358-512M-BSM -> OSD3358-512M-ISM
Changed lines of the file:
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@@
 			)
 		)
-		(property "MPN" "OSD3358-512M-BSM"
+		(property "MPN" "OSD3358-512M-ISM"
 			(at 226.06 17.78 0)
 			(effects
