File: kicad/oresat-c3.kicad_sch (KiCad schematic)
At the start: 0 parts

Commit message: Finished removing components and rerouting. Still need to place voltage and GND planes
Other:
- removed sheet Deployers
- removed sheet L Band
- removed sheet Power
- removed sheet UHF Band
Changed lines of the file:
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@@
     (effects (font (size 1.27 1.27)) (justify left bottom))
-  )
-  (sheet (at 247.65 109.22) (size 34.29 6.35)
-    (stroke (width 0.1524) (type solid))
-    (fill (color 0 0 0 0.0000))
-    (property "Sheetname" "UHF Band" (at 248.92 114.3 0)
-      (effects (font (size 2.54 2.54) bold) (justify left bottom))
-    )
-    (property "Sheetfile" "oresat-c3-sch-uhf-band.kicad_sch" (at 247.65 117.4246 0)
-      (effects (font (size 1.27 1.27)) (justify left top))
-    )
-    (instances
-      (project "oresat-c3"
-        (path "/65d12cdd-c326-4033-9053-c59fa4e0b25e" (page "9"))
-      )
-    )
   )
   (sheet (at 189.23 92.71) (size 39.37 6.35)
@@
     )
   )
-  (sheet (at 247.65 92.71) (size 34.29 6.35)
+  (sheet (at 241.3 107.95) (size 34.29 6.35)
     (stroke (width 0.1524) (type solid))
     (fill (color 0 0 0 0.0000))
-    (property "Sheetname" "L Band" (at 248.92 97.79 0)
+    (property "Sheetname" "Watchdog" (at 242.57 113.03 0)
       (effects (font (size 2.54 2.54) bold) (justify left bottom))
     )
-    (property "Sheetfile" "oresat-c3-sch-l-band.kicad_sch" (at 247.65 100.9146 0)
+    (property "Sheetfile" "oresat-c3-sch-watchdog.kicad_sch" (at 241.3 114.8846 0)
       (effects (font (size 1.27 1.27)) (justify left top))
     )
-    (instances
-      (project "oresat-c3"
-        (path "/65d12cdd-c326-4033-9053-c59fa4e0b25e" (page "8"))
-      )
-    )
-  )
-  (sheet (at 139.7 109.22) (size 34.29 6.35)
-    (stroke (width 0.1524) (type solid))
-    (fill (color 0 0 0 0.0000))
-    (property "Sheetname" "Power" (at 140.97 114.3 0)
-      (effects (font (size 2.54 2.54) bold) (justify left bottom))
-    )
-    (property "Sheetfile" "oresat-c3-sch-power.kicad_sch" (at 139.7 117.4246 0)
-      (effects (font (size 1.27 1.27)) (justify left top))
-    )
-    (instances
-      (project "oresat-c3"
-        (path "/65d12cdd-c326-4033-9053-c59fa4e0b25e" (page "2"))
-      )
-    )
-  )
-  (sheet (at 247.65 139.7) (size 34.29 6.35)
-    (stroke (width 0.1524) (type solid))
-    (fill (color 0 0 0 0.0000))
-    (property "Sheetname" "Watchdog" (at 248.92 144.78 0)
-      (effects (font (size 2.54 2.54) bold) (justify left bottom))
-    )
-    (property "Sheetfile" "oresat-c3-sch-watchdog.kicad_sch" (at 247.65 146.6346 0)
-      (effects (font (size 1.27 1.27)) (justify left top))
-    )
-    (property "Field2" "" (at 247.65 139.7 0)
+    (property "Field2" "" (at 241.3 107.95 0)
       (effects (font (size 1.27 1.27)) hide)
     )
@@
     )
   )
-  (sheet (at 247.65 124.46) (size 52.07 6.35)
+  (sheet (at 241.3 92.71) (size 52.07 6.35)
     (stroke (width 0.1524) (type solid))
     (fill (color 0 0 0 0.0000))
-    (property "Sheetname" "OPD and I2C Peripherals" (at 248.92 129.54 0)
+    (property "Sheetname" "OPD and I2C Peripherals" (at 242.57 97.79 0)
       (effects (font (size 2.54 2.54) bold) (justify left bottom))
     )
-    (property "Sheetfile" "oresat-c3-sch-opd-and-i2c.kicad_sch" (at 247.65 132.6646 0)
+    (property "Sheetfile" "oresat-c3-sch-opd-and-i2c.kicad_sch" (at 241.3 100.9146 0)
       (effects (font (size 1.27 1.27)) (justify left top))
     )
@@
       )
     )
-  )
-  (sheet (at 247.65 153.67) (size 34.29 6.35)
-    (stroke (width 0.1524) (type solid))
-    (fill (color 0 0 0 0.0000))
-    (property "Sheetname" "Deployers" (at 248.92 158.75 0)
-      (effects (font (size 2.54 2.54) bold) (justify left bottom))
-    )
-    (property "Sheetfile" "oresat-c3-sch-deployers.kicad_sch" (at 247.65 160.02 0)
-      (effects (font (size 1.27 1.27)) (justify left top))
-    )
-    (instances
-      (project "oresat-c3"
-        (path "/65d12cdd-c326-4033-9053-c59fa4e0b25e" (page "12"))
-      )
-    )
