File: kicad/oresat-c3.kicad_sch (KiCad schematic)
At the start: 0 parts

Commit message: Removed watchdog
Other:
- removed sheet Watchdog
Changed lines of the file:
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@@
-	)
-	(sheet
-		(at 241.3 107.95)
-		(size 34.29 6.35)
-		(stroke
-			(width 0.1524)
-			(type solid)
-		)
-		(fill
-			(color 0 0 0 0.0000)
-		)
-		(property "Sheetname" "Watchdog"
-			(at 242.57 113.03 0)
-			(effects
-				(font
-					(size 2.54 2.54)
-					(bold yes)
-				)
-				(justify left bottom)
-			)
-		)
-		(property "Sheetfile" "oresat-c3-sch-watchdog.kicad_sch"
-			(at 241.3 114.8846 0)
-			(effects
-				(font
-					(size 1.27 1.27)
-				)
-				(justify left top)
-			)
-		)
-		(property "Field2" ""
-			(at 241.3 107.95 0)
-			(effects
-				(font
-					(size 1.27 1.27)
-				)
-				(hide yes)
-			)
-		)
-		(instances
-			(project "oresat-c3"
-				(path "/65d12cdd-c326-4033-9053-c59fa4e0b25e"
-					(page "10")
-				)
-			)
-		)
 	)
 	(sheet

Commit message: Added MRAM chip to board
Other:
- added sheet MRAM and SPI Peripherals (mram-and-spi.kicad_sch)
Changed lines of the file:
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@@
+	)
+	(sheet
+		(at 241.3 109.22)
+		(size 54.864 6.35)
+		(stroke
+			(width 0.1524)
+			(type solid)
+		)
+		(fill
+			(color 0 0 0 0.0000)
+		)
+		(property "Sheetname" "MRAM and SPI Peripherals"
+			(at 242.57 114.046 0)
+			(effects
+				(font
+					(size 2.54 2.54)
+					(thickness 0.508)
+					(bold yes)
+				)
+				(justify left bottom)
+			)
+		)
+		(property "Sheetfile" "mram-and-spi.kicad_sch"
+			(at 241.3 116.1546 0)
+			(effects
+				(font
+					(size 1.27 1.27)
+				)
+				(justify left top)
+			)
+		)
+		(instances
+			(project "oresat-c3"
+				(path "/65d12cdd-c326-4033-9053-c59fa4e0b25e"
+					(page "9")
+				)
+			)
+		)
 	)
 	(sheet
