File: kicad/_autosave-oresat-c3.kicad_pcb (KiCad board)
At the start: 4 copper layers, 90.2 x 95.9 mm, 235 parts, among them J1 Conn_02x26_Odd_Even, J2 Conn_02x26_Odd_Even, J5 DM3BT-DSF-PEJS, J6 Conn_01x02, J7 2-1734592-0, Q1 NTR4101P, Q6 MMBT2907, U1 OSD3358-512M-BSM, U10 SN74AUC1G07DCKR, U11 RCLAMP0504FB, U12 RCLAMP0504FB, U13 MAX892LEUA+T, U14 TLVH431, U24 RV-3028-C7, U28 TLV1704-SEP, U30 FM24CL64B-DGTR, U37 LTC4300A-1, U39 TCAN330, U8 TCAN330, U9 EMMC+RESET+5.1-COMPATIBLE-BA, Y1 ECS-240-12-30BQ-AEN-TR, Y2 ABS07-32.768KHZ-T

Commit message: Fixed most DRC checks
Routing:
- net GND: track 14.9 -> 16.2 mm, vias 196 -> 195
- net UART0_RX: vias 2 -> 1
- net 5V: vias 6 -> 4
