File: kicad/oresat-c3-sch-osd3358-sysboot.kicad_sch (KiCad schematic)
At the start: 23 parts, among them J6 Conn_01x02, U1 OSD3358-512M-BSM, U8 TCAN330

Commit message: Added Oresat symbol lib. Removed any L-band related components from pcb and schematic
Parts:
- renumbered C18 to C56, TP23 to TP32, TP24 to TP49, U8 to U39
Connections:
- net LBAND_LO_SCLK: no longer names the net of U1.H15 (MII1_TXD0)
- net LBAND_LO_SDATA: no longer names the net of U1.H14 (MII1_TXD1)
- net LBAND_LO_nLOCKED: no longer names the net of U1.J14 (RMII1_REF_CLK)
- net LBAND_LO_nSEN: no longer names the net of U1.H16 (MII1_TX_CLK)
Changed lines of the file:
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@@
-    (stroke (width 0) (type default))
-  )
-  (wire (pts (xy 101.6 134.62) (xy 116.84 134.62))
     (stroke (width 0) (type default))
   )
@@
     (stroke (width 0) (type default))
   )
-  (wire (pts (xy 101.6 129.54) (xy 116.84 129.54))
-    (stroke (width 0) (type default))
-  )
   (wire (pts (xy 107.95 157.48) (xy 116.84 157.48))
     (stroke (width 0) (type default))
@@
     (stroke (width 0) (type default))
   )
-  (wire (pts (xy 102.87 172.72) (xy 116.84 172.72))
-    (stroke (width 0) (type default))
-  )
   (polyline (pts (xy 297.18 142.24) (xy 300.99 142.24))
     (stroke (width 0) (type default))
@@
   )
   (wire (pts (xy 116.84 175.26) (xy 107.95 175.26))
-    (stroke (width 0) (type default))
-  )
-  (wire (pts (xy 101.6 132.08) (xy 116.84 132.08))
     (stroke (width 0) (type default))
   )
@@
     (effects (font (size 1.27 1.27)) (justify left bottom))
   )
-  (text "LL" (at 113.03 129.54 0)
-    (effects (font (size 1.27 1.27)) (justify left bottom))
-  )
   (label "CAN0_TX" (at 102.87 139.7 0) (fields_autoplaced)
     (effects (font (size 1.27 1.27)) (justify left bottom))
@@
   (label "CAN0_RX" (at 102.87 137.16 0) (fields_autoplaced)
     (effects (font (size 1.27 1.27)) (justify left bottom))
-  )
-  (global_label "LBAND_LO_nSEN" (shape output) (at 101.6 129.54 180) (fields_autoplaced)
-    (effects (font (size 1.27 1.27)) (justify right))
-    (property "Intersheetrefs" "${INTERSHEET_REFS}" (at 83.5752 129.54 0)
-      (effects (font (size 1.27 1.27)) (justify right))
-    )
   )
   (global_label "CAN2_L" (shape input) (at 152.4 92.71 0) (fields_autoplaced)
@@
     (property "Intersheetrefs" "${INTERSHEET_REFS}" (at 162.2795 92.71 0)
       (effects (font (size 1.27 1.27)) (justify left))
-    )
-  )
-  (global_label "LBAND_LO_SDATA" (shape output) (at 101.6 134.62 180) (fields_autoplaced)
-    (effects (font (size 1.27 1.27)) (justify right))
-    (property "Intersheetrefs" "${INTERSHEET_REFS}" (at 82.7889 134.62 0)
-      (effects (font (size 1.27 1.27)) (justify right))
-    )
-  )
-  (global_label "LBAND_LO_nLOCKED" (shape input) (at 102.87 172.72 180) (fields_autoplaced)
-    (effects (font (size 1.27 1.27)) (justify right))
-    (property "Intersheetrefs" "${INTERSHEET_REFS}" (at 81.2166 172.72 0)
-      (effects (font (size 1.27 1.27)) (justify right))
-    )
-  )
-  (global_label "LBAND_LO_SCLK" (shape output) (at 101.6 132.08 180) (fields_autoplaced)
-    (effects (font (size 1.27 1.27)) (justify right))
-    (property "Intersheetrefs" "${INTERSHEET_REFS}" (at 83.6356 132.08 0)
-      (effects (font (size 1.27 1.27)) (justify right))
     )
   )
@@
   (symbol (lib_id "oresat-power:3.3V") (at 132.08 69.85 0) (unit 1)
     (in_bom yes) (on_board yes) (dnp no) (fields_autoplaced)
-    (property "Reference" "#3V0105" (at 132.08 73.66 0)
+    (property "Reference" "#3V06" (at 132.08 73.66 0)
       (effects (font (size 1.27 1.27)) hide)
     )
@@
     (instances
       (project "oresat-c3"
-        (path "/65d12cdd-c326-4033-9053-c59fa4e0b25e/f3d147ad-4cea-4d77-ae60-95882b03454e"
-          (reference "#3V0105") (unit 1)
-        )
         (path "/65d12cdd-c326-4033-9053-c59fa4e0b25e/0c732c1e-ab0d-41ac-9d77-9d7763333b6f"
           (reference "#3V06") (unit 1)
@@
   (symbol (lib_id "Interface_CAN_LIN:TCAN330") (at 132.08 90.17 0) (unit 1)
     (in_bom yes) (on_board yes) (dnp no) (fields_autoplaced)
-    (property "Reference" "U8" (at 134.0994 77.47 0)
+    (property "Reference" "U39" (at 134.0994 77.47 0)
       (effects (font (size 1.27 1.27)) (justify left))
     )
@@
     (instances
       (project "oresat-c3"
-        (path "/65d12cdd-c326-4033-9053-c59fa4e0b25e/f3d147ad-4cea-4d77-ae60-95882b03454e"
-          (reference "U8") (unit 1)
-        )
         (path "/65d12cdd-c326-4033-9053-c59fa4e0b25e/0c732c1e-ab0d-41ac-9d77-9d7763333b6f"
           (reference "U39") (unit 1)
@@
   (symbol (lib_id "oresat-misc:Test-Point-1mm-round") (at 116.84 92.71 0) (unit 1)
     (in_bom yes) (on_board yes) (dnp no)
-    (property "Reference" "TP23" (at 110.49 92.71 0)
+    (property "Reference" "TP32" (at 110.49 92.71 0)
       (effects (font (size 1.27 1.27)) (justify left))
     )
@@
     (instances
       (project "oresat-c3"
-        (path "/65d12cdd-c326-4033-9053-c59fa4e0b25e/f3d147ad-4cea-4d77-ae60-95882b03454e"
-          (reference "TP23") (unit 1)
-        )
         (path "/65d12cdd-c326-4033-9053-c59fa4e0b25e/0c732c1e-ab0d-41ac-9d77-9d7763333b6f"
           (reference "TP32") (unit 1)
@@
   (symbol (lib_id "Device:C_Small") (at 116.84 74.93 0) (unit 1)
     (in_bom yes) (on_board yes) (dnp no) (fields_autoplaced)
-    (property "Reference" "C18" (at 119.38 73.6662 0)
+    (property "Reference" "C56" (at 119.38 73.6662 0)
       (effects (font (size 1.27 1.27)) (justify left))
     )
@@
     (instances
       (project "oresat-c3"
-        (path "/65d12cdd-c326-4033-9053-c59fa4e0b25e/f3d147ad-4cea-4d77-ae60-95882b03454e"
-          (reference "C18") (unit 1)
-        )
         (path "/65d12cdd-c326-4033-9053-c59fa4e0b25e/0c732c1e-ab0d-41ac-9d77-9d7763333b6f"
           (reference "C56") (unit 1)
@@
   (symbol (lib_id "oresat-misc:Test-Point-1mm-round") (at 116.84 95.25 0) (unit 1)
     (in_bom yes) (on_board yes) (dnp no)
-    (property "Reference" "TP24" (at 110.49 95.25 0)
+    (property "Reference" "TP49" (at 110.49 95.25 0)
       (effects (font (size 1.27 1.27)) (justify left))
     )
@@
     (instances
       (project "oresat-c3"
-        (path "/65d12cdd-c326-4033-9053-c59fa4e0b25e/f3d147ad-4cea-4d77-ae60-95882b03454e"
-          (reference "TP24") (unit 1)
-        )
         (path "/65d12cdd-c326-4033-9053-c59fa4e0b25e/0c732c1e-ab0d-41ac-9d77-9d7763333b6f"
           (reference "TP49") (unit 1)
@@
   (symbol (lib_id "power:GND") (at 132.08 101.6 0) (unit 1)
     (in_bom yes) (on_board yes) (dnp no)
-    (property "Reference" "#PWR0159" (at 132.08 107.95 0)
+    (property "Reference" "#PWR014" (at 132.08 107.95 0)
       (effects (font (size 1.27 1.27)) hide)
     )
@@
     (instances
       (project "oresat-c3"
-        (path "/65d12cdd-c326-4033-9053-c59fa4e0b25e/f3d147ad-4cea-4d77-ae60-95882b03454e"
-          (reference "#PWR0159") (unit 1)
-        )
         (path "/65d12cdd-c326-4033-9053-c59fa4e0b25e/0c732c1e-ab0d-41ac-9d77-9d7763333b6f"
           (reference "#PWR014") (unit 1)
@@
   (symbol (lib_id "power:GND") (at 116.84 78.74 0) (unit 1)
     (in_bom yes) (on_board yes) (dnp no)
-    (property "Reference" "#PWR0156" (at 116.84 85.09 0)
+    (property "Reference" "#PWR013" (at 116.84 85.09 0)
       (effects (font (size 1.27 1.27)) hide)
     )
@@
     (instances
       (project "oresat-c3"
-        (path "/65d12cdd-c326-4033-9053-c59fa4e0b25e/f3d147ad-4cea-4d77-ae60-95882b03454e"
-          (reference "#PWR0156") (unit 1)
-        )
         (path "/65d12cdd-c326-4033-9053-c59fa4e0b25e/0c732c1e-ab0d-41ac-9d77-9d7763333b6f"
           (reference "#PWR013") (unit 1)

Commit message: Removed power switching circuitry
Connections:
- net RADIO_ENABLE: no longer names the net of U1.F3 (LCD_VSYNC)
Changed lines of the file:
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@@
-    )
-  )
-  (global_label "RADIO_ENABLE" (shape output) (at 186.69 175.26 0) (fields_autoplaced)
-    (effects (font (size 1.27 1.27)) (justify left))
-    (property "Intersheetrefs" "${INTERSHEET_REFS}" (at 203.1425 175.26 0)
-      (effects (font (size 1.27 1.27)) (justify left))
     )
   )

Commit message: Finished removing components and rerouting. Still need to place voltage and GND planes
Connections:
- net CAN2_H renamed CAN2_H+
- net CAN2_L renamed CAN2_L-
Changed lines of the file:
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@@
     (effects (font (size 1.27 1.27)) (justify left bottom))
   )
-  (global_label "CAN2_L" (shape input) (at 152.4 92.71 0) (fields_autoplaced)
+  (global_label "CAN2_L-" (shape input) (at 152.4 92.71 0) (fields_autoplaced)
     (effects (font (size 1.27 1.27)) (justify left))
-    (property "Intersheetrefs" "${INTERSHEET_REFS}" (at 162.2795 92.71 0)
+    (property "Intersheetrefs" "${INTERSHEET_REFS}" (at 163.8519 92.71 0)
       (effects (font (size 1.27 1.27)) (justify left))
     )
@@
     )
   )
-  (global_label "CAN2_H" (shape input) (at 152.4 87.63 0) (fields_autoplaced)
+  (global_label "CAN2_H+" (shape input) (at 152.4 87.63 0) (fields_autoplaced)
     (effects (font (size 1.27 1.27)) (justify left))
-    (property "Intersheetrefs" "${INTERSHEET_REFS}" (at 162.5819 87.63 0)
+    (property "Intersheetrefs" "${INTERSHEET_REFS}" (at 164.1543 87.63 0)
       (effects (font (size 1.27 1.27)) (justify left))
     )

Commit message: Fixed some issues, still need to clear DRC
Connections:
- no-connect marks 8 -> 13
Changed lines of the file:
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@@
   (no_connect (at 248.92 172.72))
   (no_connect (at 246.38 172.72))
+  (no_connect (at 116.84 172.72))
+  (no_connect (at 116.84 132.08))
   (no_connect (at 254 172.72))
+  (no_connect (at 186.69 175.26))
+  (no_connect (at 116.84 134.62))
+  (no_connect (at 116.84 129.54))
   (wire (pts (xy 228.6 120.65) (xy 228.6 127))
     (stroke (width 0) (type default))
