File: kicad/oresat-c3-sch-osd3358-sysboot.kicad_sch (KiCad schematic)
At the start: 27 parts, among them J4 Conn_01x05, J6 Conn_01x02, U1 OSD3358-512M-BSM, U39 TCAN330

Commit message: added automotive grade capacitors to the BOM
Parts:
- C56: Description_1 (none) -> CAP CER 0.1UF 16V X7R 0603; Manufacturer_Name (none) -> Murata Electronics; Manufacturer_Part_Number (none) -> GCJ188R71C104KA01D
- R72, R73, R74: Description_1 (none) -> RES ARRAY 8 RES 47K OHM 2512; Manufacturer_Name (none) -> Panasonic Electronic Components; Manufacturer_Part_Number (none) -> EXB-A10P473J
Changed lines of the file:
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@@
 			)
 		)
+		(property "Description_1" "RES ARRAY 8 RES 47K OHM 2512"
+			(at 256.54 185.42 90)
+			(effects
+				(font
+					(size 1.27 1.27)
+				)
+				(hide yes)
+			)
+		)
+		(property "Manufacturer_Name" "Panasonic Electronic Components"
+			(at 256.54 185.42 90)
+			(effects
+				(font
+					(size 1.27 1.27)
+				)
+				(hide yes)
+			)
+		)
+		(property "Manufacturer_Part_Number" "EXB-A10P473J"
+			(at 256.54 185.42 90)
+			(effects
+				(font
+					(size 1.27 1.27)
+				)
+				(hide yes)
+			)
+		)
 		(pin "1"
 		)
@@
 			)
 		)
+		(property "Description_1" ""
+			(at 148.59 90.17 0)
+			(effects
+				(font
+					(size 1.27 1.27)
+				)
+				(hide yes)
+			)
+		)
 		(pin "1"
 		)
@@
 			)
 		)
+		(property "Description_1" "CAP CER 0.1UF 16V X7R 0603"
+			(at 116.84 74.93 0)
+			(effects
+				(font
+					(size 1.27 1.27)
+				)
+				(hide yes)
+			)
+		)
+		(property "Manufacturer_Name" "Murata Electronics"
+			(at 116.84 74.93 0)
+			(effects
+				(font
+					(size 1.27 1.27)
+				)
+				(hide yes)
+			)
+		)
+		(property "Manufacturer_Part_Number" "GCJ188R71C104KA01D"
+			(at 116.84 74.93 0)
+			(effects
+				(font
+					(size 1.27 1.27)
+				)
+				(hide yes)
+			)
+		)
 		(pin "1"
 		)
@@
 			)
 		)
+		(property "Description_1" "RES ARRAY 8 RES 47K OHM 2512"
+			(at 231.14 185.42 90)
+			(effects
+				(font
+					(size 1.27 1.27)
+				)
+				(hide yes)
+			)
+		)
+		(property "Manufacturer_Name" "Panasonic Electronic Components"
+			(at 231.14 185.42 90)
+			(effects
+				(font
+					(size 1.27 1.27)
+				)
+				(hide yes)
+			)
+		)
+		(property "Manufacturer_Part_Number" "EXB-A10P473J"
+			(at 231.14 185.42 90)
+			(effects
+				(font
+					(size 1.27 1.27)
+				)
+				(hide yes)
+			)
+		)
 		(pin "1"
 		)
@@
 			(effects
 				(font
+					(size 1.27 1.27)
+				)
+				(hide yes)
+			)
+		)
+		(property "Description_1" "RES ARRAY 8 RES 47K OHM 2512"
+			(at 213.36 107.95 90)
+			(effects
+				(font
+					(size 1.27 1.27)
+				)
+				(hide yes)
+			)
+		)
+		(property "Manufacturer_Name" "Panasonic Electronic Components"
+			(at 213.36 107.95 90)
+			(effects
+				(font
+					(size 1.27 1.27)
+				)
+				(hide yes)
+			)
+		)
+		(property "Manufacturer_Part_Number" "EXB-A10P473J"
+			(at 213.36 107.95 90)
+			(effects
+				(font

Commit message: added automotive grade resistors to BOM
Parts:
- J4: Description_1 (none) -> CONN HEADER R/A 5POS 2.54MM; Manufacturer_Name (none) -> Samtec Inc.; Manufacturer_Part_Number (none) -> TSW-105-25-F-S-RA
- J6: Description_1 (none) -> CONN HEADER SMD R/A 2POS 2.54MM; Manufacturer_Name (none) -> Harwin Inc.; Manufacturer_Part_Number (none) -> M20-8890245
- R3: Description_1 (none) -> RES 0603 120 OHM 1% 0.125W AUTO; Manufacturer_Name (none) -> Stackpole Electronics Inc; Manufacturer_Part_Number (none) -> RMCA0603FT120R-HP
Changed lines of the file:
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@@
 			)
 		)
-		(property "Description_1" ""
+		(property "Description_1" "RES 0603 120 OHM 1% 0.125W AUTO"
+			(at 148.59 90.17 0)
+			(effects
+				(font
+					(size 1.27 1.27)
+				)
+				(hide yes)
+			)
+		)
+		(property "Manufacturer_Name" "Stackpole Electronics Inc"
+			(at 148.59 90.17 0)
+			(effects
+				(font
+					(size 1.27 1.27)
+				)
+				(hide yes)
+			)
+		)
+		(property "Manufacturer_Part_Number" "RMCA0603FT120R-HP"
 			(at 148.59 90.17 0)
 			(effects
@@
 			)
 		)
+		(property "Description_1" "CONN HEADER SMD R/A 2POS 2.54MM"
+			(at 264.16 134.62 0)
+			(effects
+				(font
+					(size 1.27 1.27)
+				)
+				(hide yes)
+			)
+		)
+		(property "Manufacturer_Name" "Harwin Inc."
+			(at 264.16 134.62 0)
+			(effects
+				(font
+					(size 1.27 1.27)
+				)
+				(hide yes)
+			)
+		)
+		(property "Manufacturer_Part_Number" "M20-8890245"
+			(at 264.16 134.62 0)
+			(effects
+				(font
+					(size 1.27 1.27)
+				)
+				(hide yes)
+			)
+		)
 		(pin "1"
 		)
@@
 			(at 313.69 177.8 0)
 			(effects
+				(font
+					(size 1.27 1.27)
+				)
+				(hide yes)
+			)
+		)
+		(property "Description_1" "CONN HEADER R/A 5POS 2.54MM"
+			(at 313.69 177.8 0)
+			(effects
+				(font
+					(size 1.27 1.27)
+				)
+				(hide yes)
+			)
+		)
+		(property "Manufacturer_Name" "Samtec Inc."
+			(at 313.69 177.8 0)
+			(effects
+				(font
+					(size 1.27 1.27)
+				)
+				(hide yes)
+			)
+		)
+		(property "Manufacturer_Part_Number" "TSW-105-25-F-S-RA"
+			(at 313.69 177.8 0)
+			(effects

Commit message: modified BOM to match PCBWay format
Parts:
- TP10, TP113, TP114, TP115, TP116, TP117, TP118, TP119, TP120, TP121, TP123, TP125, TP134, TP136, TP32, TP49, TP9, TP90: now not fitted
- U39: Description_1 (none) -> IC TRANSCEIVER 1/1 8SOIC; Manufacturer_Name (none) -> Texas Instruments; Manufacturer_Part_Number (none) -> TCAN330D
Changed lines of the file:
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@@
 		(in_bom yes)
 		(on_board yes)
-		(dnp no)
+		(dnp yes)
 		(property "Reference" "TP119"
 			(at 99.06 162.56 90)
@@
 		(in_bom yes)
 		(on_board yes)
-		(dnp no)
+		(dnp yes)
 		(property "Reference" "TP136"
 			(at 99.06 177.8 90)
@@
 		(in_bom yes)
 		(on_board yes)
-		(dnp no)
+		(dnp yes)
 		(property "Reference" "TP117"
 			(at 99.06 157.48 90)
@@
 		(in_bom yes)
 		(on_board yes)
-		(dnp no)
+		(dnp yes)
 		(property "Reference" "TP113"
 			(at 99.06 144.78 90)
@@
 		(in_bom yes)
 		(on_board yes)
-		(dnp no)
+		(dnp yes)
 		(property "Reference" "TP118"
 			(at 99.06 160.02 90)
@@
 		(in_bom yes)
 		(on_board yes)
-		(dnp no)
+		(dnp yes)
 		(property "Reference" "TP120"
 			(at 99.06 165.1 90)
@@
 		(in_bom yes)
 		(on_board yes)
-		(dnp no)
+		(dnp yes)
 		(property "Reference" "TP116"
 			(at 99.06 154.94 90)
@@
 			)
 		)
+		(property "Description_1" "IC TRANSCEIVER 1/1 8SOIC"
+			(at 132.08 90.17 0)
+			(effects
+				(font
+					(size 1.27 1.27)
+				)
+				(hide yes)
+			)
+		)
+		(property "Manufacturer_Name" "Texas Instruments"
+			(at 132.08 90.17 0)
+			(effects
+				(font
+					(size 1.27 1.27)
+				)
+				(hide yes)
+			)
+		)
+		(property "Manufacturer_Part_Number" "TCAN330D"
+			(at 132.08 90.17 0)
+			(effects
+				(font
+					(size 1.27 1.27)
+				)
+				(hide yes)
+			)
+		)
 		(pin "1"
 		)
@@
 		(in_bom yes)
 		(on_board yes)
-		(dnp no)
+		(dnp yes)
 		(property "Reference" "TP115"
 			(at 99.06 152.4 90)
@@
 		(in_bom yes)
 		(on_board yes)
-		(dnp no)
+		(dnp yes)
 		(property "Reference" "TP32"
 			(at 110.49 92.71 0)
@@
 		(in_bom yes)
 		(on_board yes)
-		(dnp no)
+		(dnp yes)
 		(property "Reference" "TP121"
 			(at 99.06 167.64 90)
@@
 		(in_bom yes)
 		(on_board yes)
-		(dnp no)
+		(dnp yes)
 		(property "Reference" "TP123"
 			(at 195.58 172.72 90)
@@
 		(in_bom yes)
 		(on_board yes)
-		(dnp no)
+		(dnp yes)
 		(property "Reference" "TP49"
 			(at 110.49 95.25 0)
@@
 		(in_bom yes)
 		(on_board yes)
-		(dnp no)
+		(dnp yes)
 		(property "Reference" "TP10"
 			(at 257.81 137.16 90)
@@
 		(in_bom yes)
 		(on_board yes)
-		(dnp no)
+		(dnp yes)
 		(property "Reference" "TP114"
 			(at 99.06 147.32 90)
@@
 		(in_bom yes)
 		(on_board yes)
-		(dnp no)
+		(dnp yes)
 		(property "Reference" "TP134"
 			(at 99.06 175.26 90)
@@
 		(in_bom yes)
 		(on_board yes)
-		(dnp no)
+		(dnp yes)
 		(property "Reference" "TP125"
 			(at 195.58 177.8 90)
@@
 		(in_bom yes)
 		(on_board yes)
-		(dnp no)
+		(dnp yes)
 		(property "Reference" "TP9"
 			(at 256.54 132.08 90)
@@
 		(in_bom yes)
 		(on_board yes)
-		(dnp no)
+		(dnp yes)
 		(property "Reference" "TP90"
 			(at 99.06 142.24 90)

Commit message: finished putting together BOM, needs review
Parts:
- C56: Description / Value (none) -> CAP CER 0.1UF 16V X7R 0603; Description_1 CAP CER 0.1UF 16V X7R 0603 -> (none)
- J4: Description / Value (none) -> CONN HEADER R/A 5POS 2.54MM; Description_1 CONN HEADER R/A 5POS 2.54MM -> (none)
- J6: Description / Value (none) -> CONN HEADER SMD R/A 2POS 2.54MM; Description_1 CONN HEADER SMD R/A 2POS 2.54MM -> (none)
- R3: Description / Value (none) -> RES 0603 120 OHM 1% 0.125W AUTO; Description_1 RES 0603 120 OHM 1% 0.125W AUTO -> (none)
- R72, R73, R74: Description / Value (none) -> RES ARRAY 8 RES 47K OHM 2512; Description_1 RES ARRAY 8 RES 47K OHM 2512 -> (none)
- U1: value OSD3358-512M-BSM -> OSD3358-512M-ISM; Description / Value (none) -> IC MODULE CORTEX-A8 1GHZ 512MB; Manufacturer_Name (none) -> Octavo Systems LLC; Manufacturer_Part_Number (none) -> OSD3358-512M-ISM
- U39: Description / Value (none) -> IC TRANSCEIVER 1/1 8SOIC; Description_1 IC TRANSCEIVER 1/1 8SOIC -> (none)
Changed lines of the file:
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@@
 			)
 		)
-		(property "Description_1" "RES ARRAY 8 RES 47K OHM 2512"
+		(property "Manufacturer_Name" "Panasonic Electronic Components"
 			(at 256.54 185.42 90)
 			(effects
@@
 			)
 		)
-		(property "Manufacturer_Name" "Panasonic Electronic Components"
+		(property "Manufacturer_Part_Number" "EXB-A10P473J"
 			(at 256.54 185.42 90)
 			(effects
@@
 			)
 		)
-		(property "Manufacturer_Part_Number" "EXB-A10P473J"
+		(property "Description / Value" "RES ARRAY 8 RES 47K OHM 2512"
 			(at 256.54 185.42 90)
 			(effects
@@
 			)
 		)
-		(property "Description_1" "RES 0603 120 OHM 1% 0.125W AUTO"
+		(property "Manufacturer_Name" "Stackpole Electronics Inc"
 			(at 148.59 90.17 0)
 			(effects
@@
 			)
 		)
-		(property "Manufacturer_Name" "Stackpole Electronics Inc"
+		(property "Manufacturer_Part_Number" "RMCA0603FT120R-HP"
 			(at 148.59 90.17 0)
 			(effects
@@
 			)
 		)
-		(property "Manufacturer_Part_Number" "RMCA0603FT120R-HP"
+		(property "Description / Value" "RES 0603 120 OHM 1% 0.125W AUTO"
 			(at 148.59 90.17 0)
 			(effects
@@
 			)
 		)
-		(property "Description_1" "IC TRANSCEIVER 1/1 8SOIC"
+		(property "Manufacturer_Name" "Texas Instruments"
 			(at 132.08 90.17 0)
 			(effects
@@
 			)
 		)
-		(property "Manufacturer_Name" "Texas Instruments"
+		(property "Manufacturer_Part_Number" "TCAN330D"
 			(at 132.08 90.17 0)
 			(effects
@@
 			)
 		)
-		(property "Manufacturer_Part_Number" "TCAN330D"
+		(property "Description / Value" "IC TRANSCEIVER 1/1 8SOIC"
 			(at 132.08 90.17 0)
 			(effects
@@
 			)
 		)
-		(property "Description_1" "CAP CER 0.1UF 16V X7R 0603"
+		(property "Manufacturer_Name" "Murata Electronics"
 			(at 116.84 74.93 0)
 			(effects
@@
 			)
 		)
-		(property "Manufacturer_Name" "Murata Electronics"
+		(property "Manufacturer_Part_Number" "GCJ188R71C104KA01D"
 			(at 116.84 74.93 0)
 			(effects
@@
 			)
 		)
-		(property "Manufacturer_Part_Number" "GCJ188R71C104KA01D"
+		(property "Description / Value" "CAP CER 0.1UF 16V X7R 0603"
 			(at 116.84 74.93 0)
 			(effects
@@
 			)
 		)
-		(property "Value" "OSD3358-512M-BSM"
+		(property "Value" "OSD3358-512M-ISM"
 			(at 147.32 121.92 0)
 			(effects
@@
 			)
 		)
-		(property "Datasheet" ""
+		(property "Datasheet" "https://mm.digikey.com/Volume0/opasdata/d220001/medias/docus/778/OSd335x-Software-PwrMgmt.pdf"
 			(at 147.32 157.48 0)
 			(effects
@@
 			)
 		)
+		(property "Manufacturer_Part_Number" "OSD3358-512M-ISM"
+			(at 147.32 157.48 0)
+			(effects
+				(font
+					(size 1.27 1.27)
+				)
+				(hide yes)
+			)
+		)
+		(property "Manufacturer_Name" "Octavo Systems LLC"
+			(at 147.32 157.48 0)
+			(effects
+				(font
+					(size 1.27 1.27)
+				)
+				(hide yes)
+			)
+		)
+		(property "Description / Value" "IC MODULE CORTEX-A8 1GHZ 512MB"
+			(at 147.32 157.48 0)
+			(effects
+				(font
+					(size 1.27 1.27)
+				)
+				(hide yes)
+			)
+		)
 		(pin "C10"
 		)
@@
 			)
 		)
-		(property "Description_1" "CONN HEADER SMD R/A 2POS 2.54MM"
+		(property "Manufacturer_Name" "Harwin Inc."
 			(at 264.16 134.62 0)
 			(effects
@@
 			)
 		)
-		(property "Manufacturer_Name" "Harwin Inc."
+		(property "Manufacturer_Part_Number" "M20-8890245"
 			(at 264.16 134.62 0)
 			(effects
@@
 			)
 		)
-		(property "Manufacturer_Part_Number" "M20-8890245"
+		(property "Description / Value" "CONN HEADER SMD R/A 2POS 2.54MM"
 			(at 264.16 134.62 0)
 			(effects
@@
 			)
 		)
-		(property "Description_1" "CONN HEADER R/A 5POS 2.54MM"
+		(property "Manufacturer_Name" "Samtec Inc."
 			(at 313.69 177.8 0)
 			(effects
@@
 			)
 		)
-		(property "Manufacturer_Name" "Samtec Inc."
+		(property "Manufacturer_Part_Number" "TSW-105-25-F-S-RA"
 			(at 313.69 177.8 0)
 			(effects
@@
 			)
 		)
-		(property "Manufacturer_Part_Number" "TSW-105-25-F-S-RA"
+		(property "Description / Value" "CONN HEADER R/A 5POS 2.54MM"
 			(at 313.69 177.8 0)
 			(effects
@@
 			)
 		)
-		(property "Description_1" "RES ARRAY 8 RES 47K OHM 2512"
+		(property "Manufacturer_Name" "Panasonic Electronic Components"
 			(at 231.14 185.42 90)
 			(effects
@@
 			)
 		)
-		(property "Manufacturer_Name" "Panasonic Electronic Components"
+		(property "Manufacturer_Part_Number" "EXB-A10P473J"
 			(at 231.14 185.42 90)
 			(effects
@@
 			)
 		)
-		(property "Manufacturer_Part_Number" "EXB-A10P473J"
+		(property "Description / Value" "RES ARRAY 8 RES 47K OHM 2512"
 			(at 231.14 185.42 90)
 			(effects
@@
 			)
 		)
-		(property "Description_1" "RES ARRAY 8 RES 47K OHM 2512"
+		(property "Manufacturer_Name" "Panasonic Electronic Components"
 			(at 213.36 107.95 90)
 			(effects
@@
 			)
 		)
-		(property "Manufacturer_Name" "Panasonic Electronic Components"
+		(property "Manufacturer_Part_Number" "EXB-A10P473J"
 			(at 213.36 107.95 90)
 			(effects
@@
 			)
 		)
-		(property "Manufacturer_Part_Number" "EXB-A10P473J"
+		(property "Description / Value" "RES ARRAY 8 RES 47K OHM 2512"
 			(at 213.36 107.95 90)
 			(effects

Commit message: - Fixed part number for FRAM, CAN transceiver, emmc, and BJT - Change LED and connected resistors to DNP - Verified remainder of components
Parts:
- U39: value TCAN330 -> TCAN330GDCNR; Manufacturer_Part_Number TCAN330D -> TCAN330GDCNR
Changed lines of the file:
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@@
 			)
 		)
-		(property "Value" "TCAN330"
+		(property "Value" "TCAN330GDCNR"
 			(at 134.0994 80.01 0)
 			(effects
@@
 			)
 		)
-		(property "Manufacturer_Part_Number" "TCAN330D"
+		(property "Manufacturer_Part_Number" "TCAN330GDCNR"
 			(at 132.08 90.17 0)
 			(effects

Commit message: Fixed some BOM issues. Board has been ordered, generated production files
Parts:
- U1: MPN OSD3358-512M-BSM -> OSD3358-512M-ISM
Changed lines of the file:
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@@
 			)
 		)
-		(property "MPN" "OSD3358-512M-BSM"
+		(property "MPN" "OSD3358-512M-ISM"
 			(at 147.32 58.42 0)
 			(effects
