File: kicad/oresat-c3-sch-osd3358-power.kicad_sch (KiCad schematic)
At the start: 39 parts, among them Q6 MMBT2907, U1 OSD3358-512M-BSM, U10 SN74AUC1G07DCKR, U14 TLVH431

Commit message: Removed power switching circuitry
Other:
- note added: "REMEMBER TO CONNECT 5V HERE"
Changed lines of the file:
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@@
     (effects (font (size 1.27 1.27)) (justify left bottom))
+  )
+  (text "REMEMBER TO CONNECT 5V HERE" (at 128.27 43.18 0)
+    (effects (font (size 2 2)) (justify left bottom))
   )
   (text "RTC_KALDO_ENN is grounded thru a\n10K so that the internal RTC LDO \nis enabled and CAP_VDD_RTC does not\nneed to be connected to VDD_CORE."

Commit message: Fixed power plane issues
Connections:
- net 3.3V: no longer R54.1, TP81.1, U1.F6 (SYS_VDD1_3P3V@1), U1.F7 (SYS_VDD1_3P3V@2), U1.G6 (SYS_VDD1_3P3V@3), U1.G7 (SYS_VDD1_3P3V@4)
- new net +3.3VADC: R54.1, TP81.1, U1.F6 (SYS_VDD1_3P3V@1), U1.F7 (SYS_VDD1_3P3V@2), U1.G6 (SYS_VDD1_3P3V@3), U1.G7 (SYS_VDD1_3P3V@4)
Other:
- note added: "NOTE: WE ARE NOT USING THE OCTAVO SIP TO POWER OUR BOARD, WE ARE POWERING FROM THE CSKB. THIS CONNECTION IS DEFERRED."
Changed lines of the file:
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@@
     (effects (font (size 1.27 1.27)) (justify left bottom))
+  )
+  (text "NOTE: WE ARE NOT USING THE OCTAVO SIP TO POWER OUR BOARD,\nWE ARE POWERING FROM THE CSKB. THIS CONNECTION IS DEFERRED."
+    (at 308.61 77.47 0)
+    (effects (font (size 2 2) (thickness 0.4) bold) (justify left bottom))
   )
   (text "ZH" (at 181.61 193.04 0)
@@
     )
   )
-  (symbol (lib_id "oresat-power:3.3V") (at 298.45 69.85 0) (unit 1)
-    (in_bom yes) (on_board yes) (dnp no) (fields_autoplaced)
-    (property "Reference" "#3V0113" (at 298.45 73.66 0)
-      (effects (font (size 1.27 1.27)) hide)
-    )
-    (property "Value" "3.3V" (at 298.45 64.77 0)
+  (symbol (lib_id "power:+3.3VADC") (at 298.45 69.85 0) (unit 1)
+    (in_bom yes) (on_board yes) (dnp no) (fields_autoplaced)
+    (property "Reference" "#PWR02" (at 302.26 71.12 0)
+      (effects (font (size 1.27 1.27)) hide)
+    )
+    (property "Value" "+3.3VADC" (at 298.45 64.77 0)
       (effects (font (size 1.27 1.27)))
     )
@@
       (project "oresat-c3"
         (path "/65d12cdd-c326-4033-9053-c59fa4e0b25e/0c1da208-2d1c-4d05-9cc7-59584e50a6ac"
-          (reference "#3V0113") (unit 1)
-        )
-      )
+          (reference "#PWR02") (unit 1)
+        )
+      )

Commit message: Fixed most DRC checks
Connections:
- net 3.3V: now also R54.1, TP81.1
- removed net +3.3VADC: R54.1, TP81.1, U1.F6 (SYS_VDD1_3P3V@1), U1.F7 (SYS_VDD1_3P3V@2), U1.G6 (SYS_VDD1_3P3V@3), U1.G7 (SYS_VDD1_3P3V@4)
Other:
- moved on the sheet: TP81
Changed lines of the file:
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@@
   (junction (at 265.43 157.48) (diameter 0) (color 0 0 0 0)
   )
-  (junction (at 265.43 71.12) (diameter 0) (color 0 0 0 0)
-  )
   (junction (at 166.37 62.23) (diameter 0) (color 0 0 0 0)
   )
@@
   (junction (at 285.75 149.86) (diameter 0) (color 0 0 0 0)
   )
-  (junction (at 265.43 73.66) (diameter 0) (color 0 0 0 0)
-  )
   (junction (at 265.43 172.72) (diameter 0) (color 0 0 0 0)
   )
@@
   (junction (at 186.69 53.34) (diameter 0) (color 0 0 0 0)
   )
-  (junction (at 265.43 76.2) (diameter 0) (color 0 0 0 0)
-  )
   (junction (at 265.43 55.88) (diameter 0) (color 0 0 0 0)
   )
@@
     (stroke (width 0) (type default))
   )
-  (wire (pts (xy 265.43 78.74) (xy 265.43 76.2))
-    (stroke (width 0) (type default))
-  )
   (wire (pts (xy 298.45 132.08) (xy 298.45 137.16))
     (stroke (width 0) (type default))
@@
     (stroke (width 0) (type default))
   )
-  (wire (pts (xy 265.43 73.66) (xy 265.43 71.12))
-    (stroke (width 0) (type default))
-  )
   (wire (pts (xy 186.69 88.9) (xy 189.23 88.9))
     (stroke (width 0) (type default))
@@
     (stroke (width 0) (type default))
   )
-  (wire (pts (xy 265.43 76.2) (xy 265.43 73.66))
-    (stroke (width 0) (type default))
-  )
   (wire (pts (xy 265.43 55.88) (xy 265.43 53.34))
     (stroke (width 0) (type default))
@@
     (stroke (width 0) (type default))
   )
-  (wire (pts (xy 265.43 71.12) (xy 298.45 71.12))
+  (wire (pts (xy 287.02 71.12) (xy 298.45 71.12))
     (stroke (width 0) (type default))
   )
@@
   )
   (wire (pts (xy 265.43 104.14) (xy 265.43 101.6))
-    (stroke (width 0) (type default))
-  )
-  (wire (pts (xy 260.35 71.12) (xy 265.43 71.12))
     (stroke (width 0) (type default))
   )
@@
     (effects (font (size 1.27 1.27)) (justify left bottom))
   )
-  (text "SYS_VDD1_3P3V" (at 269.24 73.66 0)
+  (text "SYS_VDD1_3P3V" (at 257.81 82.55 0)
     (effects (font (size 1.27 1.27)) (justify left bottom))
   )
@@
     )
   )
-  (symbol (lib_id "power:+3.3VADC") (at 298.45 69.85 0) (unit 1)
-    (in_bom yes) (on_board yes) (dnp no) (fields_autoplaced)
-    (property "Reference" "#PWR02" (at 302.26 71.12 0)
-      (effects (font (size 1.27 1.27)) hide)
-    )
-    (property "Value" "+3.3VADC" (at 298.45 64.77 0)
-      (effects (font (size 1.27 1.27)))
-    )
-    (property "Footprint" "" (at 298.45 69.85 0)
-      (effects (font (size 1.27 1.27)) hide)
-    )
-    (property "Datasheet" "" (at 298.45 69.85 0)
-      (effects (font (size 1.27 1.27)) hide)
-    )
-    (pin "1")
-    (instances
-      (project "oresat-c3"
-        (path "/65d12cdd-c326-4033-9053-c59fa4e0b25e/0c1da208-2d1c-4d05-9cc7-59584e50a6ac"
-          (reference "#PWR02") (unit 1)
-        )
-      )
-    )
-  )
   (symbol (lib_id "oresat-misc:Test-Point-1mm-round") (at 186.69 149.86 180) (unit 1)
     (in_bom yes) (on_board yes) (dnp no)
@@
     )
   )
-  (symbol (lib_id "oresat-misc:Test-Point-0.75mm-th") (at 265.43 71.12 270) (unit 1)
-    (in_bom yes) (on_board yes) (dnp no)
-    (property "Reference" "TP81" (at 264.16 68.58 90)
+  (symbol (lib_id "oresat-misc:Test-Point-0.75mm-th") (at 287.02 71.12 270) (unit 1)
+    (in_bom yes) (on_board yes) (dnp no)
+    (property "Reference" "TP81" (at 285.75 68.58 90)
       (effects (font (size 1.27 1.27)) (justify left))
     )
-    (property "Value" "Test-Point" (at 267.97 71.12 0)
-      (effects (font (size 1.27 1.27)) hide)
-    )
-    (property "Footprint" "oresat-misc:TestPoint-0.75mm-th" (at 275.59 71.12 0)
-      (effects (font (size 1.27 1.27)) hide)
-    )
-    (property "Datasheet" "" (at 265.43 71.12 0)
-      (effects (font (size 1.27 1.27)) hide)
-    )
-    (property "Part Page" "" (at 265.43 71.12 0)
-      (effects (font (size 1.27 1.27)) hide)
-    )
-    (property "Price" "" (at 265.43 71.12 0)
-      (effects (font (size 1.27 1.27)) hide)
-    )
-    (property "Total Price" "" (at 265.43 71.12 0)
+    (property "Value" "Test-Point" (at 289.56 71.12 0)
+      (effects (font (size 1.27 1.27)) hide)
+    )
+    (property "Footprint" "oresat-misc:TestPoint-0.75mm-th" (at 297.18 71.12 0)
+      (effects (font (size 1.27 1.27)) hide)
+    )
+    (property "Datasheet" "" (at 287.02 71.12 0)
+      (effects (font (size 1.27 1.27)) hide)
+    )
+    (property "Part Page" "" (at 287.02 71.12 0)
+      (effects (font (size 1.27 1.27)) hide)
+    )
+    (property "Price" "" (at 287.02 71.12 0)
+      (effects (font (size 1.27 1.27)) hide)
+    )
+    (property "Total Price" "" (at 287.02 71.12 0)
       (effects (font (size 1.27 1.27)) hide)
     )
@@
         )
       )
+    )
+  )
+  (symbol (lib_id "oresat-power:3.3V") (at 298.45 69.85 0) (unit 1)
+    (in_bom yes) (on_board yes) (dnp no) (fields_autoplaced)
+    (property "Reference" "#3V09" (at 298.45 73.66 0)
+      (effects (font (size 1.27 1.27)) hide)
+    )
+    (property "Value" "3.3V" (at 298.45 64.77 0)
+      (effects (font (size 1.27 1.27)))
+    )
+    (property "Footprint" "" (at 298.45 69.85 0)
+      (effects (font (size 1.27 1.27)) hide)
+    )
+    (property "Datasheet" "" (at 298.45 69.85 0)
+      (effects (font (size 1.27 1.27)) hide)
+    )
+    (pin "1")
+    (instances
+      (project "oresat-c3"
+        (path "/65d12cdd-c326-4033-9053-c59fa4e0b25e/0c1da208-2d1c-4d05-9cc7-59584e50a6ac"
+          (reference "#3V09") (unit 1)
+        )
+      )

Commit message: Fixed some issues, still need to clear DRC
Connections:
- no-connect marks 0 -> 4
Other:
- note added: "Providing DC to AC input?????"
Changed lines of the file:
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@@
   (junction (at 265.43 55.88) (diameter 0) (color 0 0 0 0)
   )
+  (no_connect (at 265.43 78.74))
+  (no_connect (at 260.35 71.12))
+  (no_connect (at 265.43 73.66))
+  (no_connect (at 265.43 76.2))
   (wire (pts (xy 299.72 222.25) (xy 299.72 223.52))
     (stroke (width 0) (type default))
@@
     (effects (font (size 1.27 1.27)) (justify left bottom))
   )
+  (text "Providing DC to AC input?????" (at 181.61 46.99 0)
+    (effects (font (size 1.27 1.27) bold) (justify left bottom))
+  )
   (text "All resistors are 0603 1% AEC-Q200 unless marked.\nAll capacitors are 0603 AEC-Q200 Vw >= 16V X5R or better unless marked."

Commit message: Switched 3.3V generation from CSKB to OSD3358
Connections:
- net 3.3V: now also U1.F6 (SYS_VDD1_3P3V@1), U1.F7 (SYS_VDD1_3P3V@2), U1.G6 (SYS_VDD1_3P3V@3), U1.G7 (SYS_VDD1_3P3V@4)
- no-connect marks 4 -> 0
Other:
- note removed: "NOTE: WE ARE NOT USING THE OCTAVO SIP TO POWER OUR BOARD, WE ARE POWERING FROM THE CSKB. THIS CONNECTION IS DEFERRED."
- moved on the sheet: TP81
Changed lines of the file:
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@@
   (junction (at 298.45 71.12) (diameter 0) (color 0 0 0 0)
   )
+  (junction (at 265.43 76.2) (diameter 0) (color 0 0 0 0)
+  )
   (junction (at 265.43 129.54) (diameter 0) (color 0 0 0 0)
   )
@@
   (junction (at 292.1 215.9) (diameter 0) (color 0 0 0 0)
   )
+  (junction (at 265.43 73.66) (diameter 0) (color 0 0 0 0)
+  )
   (junction (at 285.75 149.86) (diameter 0) (color 0 0 0 0)
   )
@@
   (junction (at 299.72 215.9) (diameter 0) (color 0 0 0 0)
   )
+  (junction (at 265.43 71.12) (diameter 0) (color 0 0 0 0)
+  )
   (junction (at 265.43 180.34) (diameter 0) (color 0 0 0 0)
   )
@@
   (junction (at 265.43 55.88) (diameter 0) (color 0 0 0 0)
   )
-  (no_connect (at 265.43 78.74))
-  (no_connect (at 260.35 71.12))
-  (no_connect (at 265.43 73.66))
-  (no_connect (at 265.43 76.2))
   (wire (pts (xy 299.72 222.25) (xy 299.72 223.52))
     (stroke (width 0) (type default))
@@
     (stroke (width 0) (type default))
   )
+  (wire (pts (xy 260.35 71.12) (xy 265.43 71.12))
+    (stroke (width 0) (type default))
+  )
   (wire (pts (xy 302.26 125.73) (xy 308.61 125.73))
     (stroke (width 0) (type default))
@@
     (stroke (width 0) (type default))
   )
+  (wire (pts (xy 265.43 76.2) (xy 265.43 78.74))
+    (stroke (width 0) (type default))
+  )
   (wire (pts (xy 292.1 203.2) (xy 290.83 203.2))
     (stroke (width 0) (type default))
@@
     (stroke (width 0) (type default))
   )
-  (wire (pts (xy 287.02 71.12) (xy 298.45 71.12))
+  (wire (pts (xy 265.43 71.12) (xy 298.45 71.12))
     (stroke (width 0) (type default))
   )
@@
     (stroke (width 0) (type default))
   )
+  (wire (pts (xy 265.43 73.66) (xy 265.43 76.2))
+    (stroke (width 0) (type default))
+  )
   (wire (pts (xy 182.88 220.98) (xy 182.88 222.25))
     (stroke (width 0) (type default))
@@
   )
   (wire (pts (xy 298.45 132.08) (xy 293.37 132.08))
+    (stroke (width 0) (type default))
+  )
+  (wire (pts (xy 265.43 71.12) (xy 265.43 73.66))
     (stroke (width 0) (type default))
   )
@@
   (text "Power from Backplane (Vbus\nvia Vbusp) from 5V SPS" (at 132.08 55.88 0)
     (effects (font (size 1.27 1.27)) (justify left bottom))
-  )
-  (text "NOTE: WE ARE NOT USING THE OCTAVO SIP TO POWER OUR BOARD,\nWE ARE POWERING FROM THE CSKB. THIS CONNECTION IS DEFERRED."
-    (at 308.61 77.47 0)
-    (effects (font (size 2 2) (thickness 0.4) bold) (justify left bottom))
   )
   (text "ZH" (at 181.61 193.04 0)
@@
     (effects (font (size 1.27 1.27)) (justify left bottom))
   )
-  (text "SYS_VDD1_3P3V" (at 257.81 82.55 0)
+  (text "SYS_VDD1_3P3V" (at 269.24 73.66 0)
     (effects (font (size 1.27 1.27)) (justify left bottom))
   )
@@
     )
   )
-  (symbol (lib_id "oresat-misc:Test-Point-0.75mm-th") (at 287.02 71.12 270) (unit 1)
+  (symbol (lib_id "oresat-misc:Test-Point-0.75mm-th") (at 265.43 71.12 270) (unit 1)
     (in_bom yes) (on_board yes) (dnp no)
-    (property "Reference" "TP81" (at 285.75 68.58 90)
+    (property "Reference" "TP81" (at 264.16 68.58 90)
       (effects (font (size 1.27 1.27)) (justify left))
     )
-    (property "Value" "Test-Point" (at 289.56 71.12 0)
-      (effects (font (size 1.27 1.27)) hide)
-    )
-    (property "Footprint" "oresat-misc:TestPoint-0.75mm-th" (at 297.18 71.12 0)
-      (effects (font (size 1.27 1.27)) hide)
-    )
-    (property "Datasheet" "" (at 287.02 71.12 0)
-      (effects (font (size 1.27 1.27)) hide)
-    )
-    (property "Part Page" "" (at 287.02 71.12 0)
-      (effects (font (size 1.27 1.27)) hide)
-    )
-    (property "Price" "" (at 287.02 71.12 0)
-      (effects (font (size 1.27 1.27)) hide)
-    )
-    (property "Total Price" "" (at 287.02 71.12 0)
-      (effects (font (size 1.27 1.27)) hide)
-    )
+    (property "Value" "Test-Point" (at 267.97 71.12 0)
+      (effects (font (size 1.27 1.27)) hide)
+    )
+    (property "Footprint" "oresat-misc:TestPoint-0.75mm-th" (at 275.59 71.12 0)
+      (effects (font (size 1.27 1.27)) hide)
+    )
+    (property "Datasheet" "" (at 265.43 71.12 0)
+      (effects (font (size 1.27 1.27)) hide)
+    )
+    (property "Part Page" "" (at 265.43 71.12 0)
+      (effects (font (size 1.27 1.27)) hide)
+    )
+    (property "Price" "" (at 265.43 71.12 0)
+      (effects (font (size 1.27 1.27)) hide)
+    )
+    (property "Total Price" "" (at 265.43 71.12 0)
+      (effects (font (size 1.27 1.27)) hide)
+    )
