File: kicad/oresat-c3-sch-osd3358-power.kicad_sch (KiCad schematic)
At the start: 39 parts, among them Q6 MMBT2907, U1 OSD3358-512M-BSM, U10 SN74AUC1G07DCKR, U14 TLVH431

Commit message: added automotive grade capacitors to the BOM
Parts:
- C33, C65, C78: Description_1 (none) -> CAP CER 0.1UF 16V X7R 0603; Manufacturer_Name (none) -> Murata Electronics; Manufacturer_Part_Number (none) -> GCJ188R71C104KA01D
- C34, C35, C36, C93: Description_1 (none) -> CAP CER 22UF 16V X7R 1210; Manufacturer_Name (none) -> Murata Electronics; Manufacturer_Part_Number (none) -> GCM32ER71C226KE19L
- R50, R53, R54, R57: Description_1 (none) -> RES 10K OHM 1% 1/8W 0603; Manufacturer_Name (none) -> Stackpole Electronics Inc; Manufacturer_Part_Number (none) -> RNCP0603FTD10K0

Commit message: added automotive grade resistors to BOM
Parts:
- R50, R53, R54, R57: Description_1 RES 10K OHM 1% 1/8W 0603 -> RES 0603 10 KOHM 1% 0.125W AUTO; Manufacturer_Part_Number RNCP0603FTD10K0 -> RMCA0603FT10K0-HP
- R55: Description_1 (none) -> RES 0603 499 OHM 1% 0.125W AUTO; Manufacturer_Name (none) -> Stackpole Electronics Inc; Manufacturer_Part_Number (none) -> RMCA0603FT499R-HP
- R56: Description_1 (none) -> RES 40.2K OHM 1% 1/10W 0603; Manufacturer_Name (none) -> Würth Elektronik; Manufacturer_Part_Number (none) -> 560112116003
Changed lines of the file:
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@@
 			)
 		)
-		(property "Description_1" "RES 10K OHM 1% 1/8W 0603"
+		(property "Description_1" "RES 0603 10 KOHM 1% 0.125W AUTO"
 			(at 182.88 218.44 0)
 			(effects
@@
 			)
 		)
-		(property "Manufacturer_Part_Number" "RNCP0603FTD10K0"
+		(property "Manufacturer_Part_Number" "RMCA0603FT10K0-HP"
 			(at 182.88 218.44 0)
 			(effects
@@
 			)
 		)
-		(property "Description_1" ""
+		(property "Description_1" "RES 0603 499 OHM 1% 0.125W AUTO"
+			(at 298.45 139.7 90)
+			(effects
+				(font
+					(size 1.27 1.27)
+				)
+				(hide yes)
+			)
+		)
+		(property "Manufacturer_Name" "Stackpole Electronics Inc"
+			(at 298.45 139.7 90)
+			(effects
+				(font
+					(size 1.27 1.27)
+				)
+				(hide yes)
+			)
+		)
+		(property "Manufacturer_Part_Number" "RMCA0603FT499R-HP"
 			(at 298.45 139.7 90)
 			(effects
@@
 			)
 		)
-		(property "Description_1" "RES 10K OHM 1% 1/8W 0603"
+		(property "Description_1" "RES 0603 10 KOHM 1% 0.125W AUTO"
 			(at 308.61 139.7 90)
 			(effects
@@
 			)
 		)
-		(property "Manufacturer_Part_Number" "RNCP0603FTD10K0"
+		(property "Manufacturer_Part_Number" "RMCA0603FT10K0-HP"
 			(at 308.61 139.7 90)
 			(effects
@@
 			)
 		)
-		(property "Description_1" ""
+		(property "Description_1" "RES 40.2K OHM 1% 1/10W 0603"
+			(at 308.61 114.3 90)
+			(effects
+				(font
+					(size 1.27 1.27)
+				)
+				(hide yes)
+			)
+		)
+		(property "Manufacturer_Name" "Würth Elektronik"
+			(at 308.61 114.3 90)
+			(effects
+				(font
+					(size 1.27 1.27)
+				)
+				(hide yes)
+			)
+		)
+		(property "Manufacturer_Part_Number" "560112116003"
 			(at 308.61 114.3 90)
 			(effects
@@
 			)
 		)
-		(property "Description_1" "RES 10K OHM 1% 1/8W 0603"
+		(property "Description_1" "RES 0603 10 KOHM 1% 0.125W AUTO"
 			(at 299.72 210.82 0)
 			(effects
@@
 			)
 		)
-		(property "Manufacturer_Part_Number" "RNCP0603FTD10K0"
+		(property "Manufacturer_Part_Number" "RMCA0603FT10K0-HP"
 			(at 299.72 210.82 0)
 			(effects
@@
 			)
 		)
-		(property "Description_1" "RES 10K OHM 1% 1/8W 0603"
+		(property "Description_1" "RES 0603 10 KOHM 1% 0.125W AUTO"
 			(at 298.45 76.2 0)
 			(effects
@@
 			)
 		)
-		(property "Manufacturer_Part_Number" "RNCP0603FTD10K0"
+		(property "Manufacturer_Part_Number" "RMCA0603FT10K0-HP"
 			(at 298.45 76.2 0)
 			(effects

Commit message: modified BOM to match PCBWay format
Parts:
- Q6: Description_1 (none) -> 40V 250MW 100@150MA,10V 600MA PN; Manufacturer_Name (none) -> Shenzhen Slkormicro Semicon Co., Ltd.; Manufacturer_Part_Number (none) -> MMBT2907
- TP127, TP128, TP129, TP130, TP131, TP132, TP133, TP135, TP73, TP74, TP75, TP76, TP77, TP78, TP79, TP80, TP81, TP82, TP83, TP84, TP85: now not fitted
- U10: Description_1 (none) -> IC BUFF NON-INVERT 2.7V SC-70-5; Manufacturer_Name (none) -> Texas Instruments; Manufacturer_Part_Number (none) -> SN74AUC1G07DCKR
- U14: Description_1 (none) -> IC VREF SHUNT ADJ 0.5% SOT23-3; Manufacturer_Name (none) -> Texas Instruments; Manufacturer_Part_Number (none) -> TLVH431BMDBZREP
Changed lines of the file:
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@@
 		(in_bom yes)
 		(on_board yes)
-		(dnp no)
+		(dnp yes)
 		(property "Reference" "TP84"
 			(at 267.97 144.78 90)
@@
 		(in_bom yes)
 		(on_board yes)
-		(dnp no)
+		(dnp yes)
 		(property "Reference" "TP85"
 			(at 267.97 170.18 90)
@@
 		(in_bom yes)
 		(on_board yes)
-		(dnp no)
+		(dnp yes)
 		(property "Reference" "TP75"
 			(at 167.64 203.2 0)
@@
 		(in_bom yes)
 		(on_board yes)
-		(dnp no)
+		(dnp yes)
 		(property "Reference" "TP129"
 			(at 179.07 149.86 0)
@@
 		(in_bom yes)
 		(on_board yes)
-		(dnp no)
+		(dnp yes)
 		(property "Reference" "TP135"
 			(at 292.1 218.44 0)
@@
 		(in_bom yes)
 		(on_board yes)
-		(dnp no)
+		(dnp yes)
 		(property "Reference" "TP81"
 			(at 264.16 68.58 90)
@@
 		(in_bom yes)
 		(on_board yes)
-		(dnp no)
+		(dnp yes)
 		(property "Reference" "TP132"
 			(at 179.07 172.72 0)
@@
 		(in_bom yes)
 		(on_board yes)
-		(dnp no)
+		(dnp yes)
 		(property "Reference" "TP78"
 			(at 181.61 68.58 0)
@@
 		(in_bom yes)
 		(on_board yes)
-		(dnp no)
+		(dnp yes)
 		(property "Reference" "TP79"
 			(at 167.64 209.55 0)
@@
 		(in_bom yes)
 		(on_board yes)
-		(dnp no)
+		(dnp yes)
 		(property "Reference" "TP74"
 			(at 167.64 190.5 0)
@@
 		(in_bom yes)
 		(on_board yes)
-		(dnp no)
+		(dnp yes)
 		(property "Reference" "TP130"
 			(at 179.07 157.48 0)
@@
 		(in_bom yes)
 		(on_board yes)
-		(dnp no)
+		(dnp yes)
 		(property "Reference" "TP80"
 			(at 264.16 50.8 90)
@@
 		(in_bom yes)
 		(on_board yes)
-		(dnp no)
+		(dnp yes)
 		(property "Reference" "TP73"
 			(at 167.64 182.88 0)
@@
 		(in_bom yes)
 		(on_board yes)
-		(dnp no)
+		(dnp yes)
 		(property "Reference" "TP83"
 			(at 264.16 99.06 90)
@@
 		(in_bom yes)
 		(on_board yes)
-		(dnp no)
+		(dnp yes)
 		(property "Reference" "TP128"
 			(at 179.07 137.16 0)
@@
 		(in_bom yes)
 		(on_board yes)
-		(dnp no)
+		(dnp yes)
 		(property "Reference" "TP82"
 			(at 264.16 86.36 90)
@@
 		(in_bom yes)
 		(on_board yes)
-		(dnp no)
+		(dnp yes)
 		(property "Reference" "TP127"
 			(at 179.07 127 0)
@@
 			)
 		)
+		(property "Description_1" "IC VREF SHUNT ADJ 0.5% SOT23-3"
+			(at 298.45 124.46 90)
+			(effects
+				(font
+					(size 1.27 1.27)
+				)
+				(hide yes)
+			)
+		)
+		(property "Manufacturer_Name" "Texas Instruments"
+			(at 298.45 124.46 90)
+			(effects
+				(font
+					(size 1.27 1.27)
+				)
+				(hide yes)
+			)
+		)
+		(property "Manufacturer_Part_Number" "TLVH431BMDBZREP"
+			(at 298.45 124.46 90)
+			(effects
+				(font
+					(size 1.27 1.27)
+				)
+				(hide yes)
+			)
+		)
 		(pin "1"
 		)
@@
 			)
 		)
+		(property "Description_1" "40V 250MW 100@150MA,10V 600MA PN"
+			(at 288.29 132.08 0)
+			(effects
+				(font
+					(size 1.27 1.27)
+				)
+				(hide yes)
+			)
+		)
+		(property "Manufacturer_Name" "Shenzhen Slkormicro Semicon Co., Ltd."
+			(at 288.29 132.08 0)
+			(effects
+				(font
+					(size 1.27 1.27)
+				)
+				(hide yes)
+			)
+		)
+		(property "Manufacturer_Part_Number" "MMBT2907"
+			(at 288.29 132.08 0)
+			(effects
+				(font
+					(size 1.27 1.27)
+				)
+				(hide yes)
+			)
+		)
 		(pin "1"
 		)
@@
 		(in_bom yes)
 		(on_board yes)
-		(dnp no)
+		(dnp yes)
 		(property "Reference" "TP76"
 			(at 180.34 96.52 0)
@@
 		(in_bom yes)
 		(on_board yes)
-		(dnp no)
+		(dnp yes)
 		(property "Reference" "TP77"
 			(at 180.34 93.98 0)
@@
 		(in_bom yes)
 		(on_board yes)
-		(dnp no)
+		(dnp yes)
 		(property "Reference" "TP133"
 			(at 273.05 200.66 0)
@@
 			)
 		)
+		(property "Description_1" "IC BUFF NON-INVERT 2.7V SC-70-5"
+			(at 285.75 203.2 0)
+			(effects
+				(font
+					(size 1.27 1.27)
+				)
+				(hide yes)
+			)
+		)
+		(property "Manufacturer_Name" "Texas Instruments"
+			(at 285.75 203.2 0)
+			(effects
+				(font
+					(size 1.27 1.27)
+				)
+				(hide yes)
+			)
+		)
+		(property "Manufacturer_Part_Number" "SN74AUC1G07DCKR"
+			(at 285.75 203.2 0)
+			(effects
+				(font
+					(size 1.27 1.27)
+				)
+				(hide yes)
+			)
+		)
 		(pin "1"
 		)
@@
 		(in_bom yes)
 		(on_board yes)
-		(dnp no)
+		(dnp yes)
 		(property "Reference" "TP131"
 			(at 179.07 165.1 0)

Commit message: finished putting together BOM, needs review
Parts:
- C33, C65, C78: Description / Value (none) -> CAP CER 0.1UF 16V X7R 0603; Description_1 CAP CER 0.1UF 16V X7R 0603 -> (none)
- C34, C35, C36, C93: Description / Value (none) -> CAP CER 22UF 16V X7R 1210; Description_1 CAP CER 22UF 16V X7R 1210 -> (none)
- Q6: Description / Value (none) -> 40V 250MW 100@150MA,10V 600MA PN; Description_1 40V 250MW 100@150MA,10V 600MA PN -> (none)
- R50, R53, R54, R57: Description / Value (none) -> RES 0603 10 KOHM 1% 0.125W AUTO; Description_1 RES 0603 10 KOHM 1% 0.125W AUTO -> (none)
- R55: Description / Value (none) -> RES 0603 499 OHM 1% 0.125W AUTO; Description_1 RES 0603 499 OHM 1% 0.125W AUTO -> (none)
- R56: Description / Value (none) -> RES 40.2K OHM 1% 1/10W 0603; Description_1 RES 40.2K OHM 1% 1/10W 0603 -> (none)
- U1: value OSD3358-512M-BSM -> OSD3358-512M-ISM; Description / Value (none) -> IC MODULE CORTEX-A8 1GHZ 512MB; Manufacturer_Name (none) -> Octavo Systems LLC; Manufacturer_Part_Number (none) -> OSD3358-512M-ISM
- U10: Description / Value (none) -> IC BUFF NON-INVERT 2.7V SC-70-5; Description_1 IC BUFF NON-INVERT 2.7V SC-70-5 -> (none)
- U14: Description / Value (none) -> IC VREF SHUNT ADJ 0.5% SOT23-3; Description_1 IC VREF SHUNT ADJ 0.5% SOT23-3 -> (none)
Changed lines of the file:
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@@
 			)
 		)
-		(property "Description_1" "CAP CER 22UF 16V X7R 1210"
+		(property "Manufacturer_Name" "Murata Electronics"
 			(at 162.56 58.42 0)
 			(effects
@@
 			)
 		)
-		(property "Manufacturer_Name" "Murata Electronics"
+		(property "Manufacturer_Part_Number" "GCM32ER71C226KE19L"
 			(at 162.56 58.42 0)
 			(effects
@@
 			)
 		)
-		(property "Manufacturer_Part_Number" "GCM32ER71C226KE19L"
+		(property "Description / Value" "CAP CER 22UF 16V X7R 1210"
 			(at 162.56 58.42 0)
 			(effects
@@
 			)
 		)
-		(property "Description_1" "RES 0603 10 KOHM 1% 0.125W AUTO"
+		(property "Manufacturer_Name" "Stackpole Electronics Inc"
 			(at 182.88 218.44 0)
 			(effects
@@
 			)
 		)
-		(property "Manufacturer_Name" "Stackpole Electronics Inc"
+		(property "Manufacturer_Part_Number" "RMCA0603FT10K0-HP"
 			(at 182.88 218.44 0)
 			(effects
@@
 			)
 		)
-		(property "Manufacturer_Part_Number" "RMCA0603FT10K0-HP"
+		(property "Description / Value" "RES 0603 10 KOHM 1% 0.125W AUTO"
 			(at 182.88 218.44 0)
 			(effects
@@
 			)
 		)
-		(property "Description_1" "CAP CER 0.1UF 16V X7R 0603"
+		(property "Manufacturer_Name" "Murata Electronics"
 			(at 299.72 219.71 0)
 			(effects
@@
 			)
 		)
-		(property "Manufacturer_Name" "Murata Electronics"
+		(property "Manufacturer_Part_Number" "GCJ188R71C104KA01D"
 			(at 299.72 219.71 0)
 			(effects
@@
 			)
 		)
-		(property "Manufacturer_Part_Number" "GCJ188R71C104KA01D"
+		(property "Description / Value" "CAP CER 0.1UF 16V X7R 0603"
 			(at 299.72 219.71 0)
 			(effects
@@
 			)
 		)
-		(property "Description_1" "CAP CER 0.1UF 16V X7R 0603"
+		(property "Manufacturer_Name" "Murata Electronics"
 			(at 289.56 190.5 0)
 			(effects
@@
 			)
 		)
-		(property "Manufacturer_Name" "Murata Electronics"
+		(property "Manufacturer_Part_Number" "GCJ188R71C104KA01D"
 			(at 289.56 190.5 0)
 			(effects
@@
 			)
 		)
-		(property "Manufacturer_Part_Number" "GCJ188R71C104KA01D"
+		(property "Description / Value" "CAP CER 0.1UF 16V X7R 0603"
 			(at 289.56 190.5 0)
 			(effects
@@
 			)
 		)
-		(property "Description_1" "RES 0603 499 OHM 1% 0.125W AUTO"
+		(property "Manufacturer_Name" "Stackpole Electronics Inc"
 			(at 298.45 139.7 90)
 			(effects
@@
 			)
 		)
-		(property "Manufacturer_Name" "Stackpole Electronics Inc"
+		(property "Manufacturer_Part_Number" "RMCA0603FT499R-HP"
 			(at 298.45 139.7 90)
 			(effects
@@
 			)
 		)
-		(property "Manufacturer_Part_Number" "RMCA0603FT499R-HP"
+		(property "Description / Value" "RES 0603 499 OHM 1% 0.125W AUTO"
 			(at 298.45 139.7 90)
 			(effects
@@
 			)
 		)
-		(property "Description_1" "RES 0603 10 KOHM 1% 0.125W AUTO"
+		(property "Manufacturer_Name" "Stackpole Electronics Inc"
 			(at 308.61 139.7 90)
 			(effects
@@
 			)
 		)
-		(property "Manufacturer_Name" "Stackpole Electronics Inc"
+		(property "Manufacturer_Part_Number" "RMCA0603FT10K0-HP"
 			(at 308.61 139.7 90)
 			(effects
@@
 			)
 		)
-		(property "Manufacturer_Part_Number" "RMCA0603FT10K0-HP"
+		(property "Description / Value" "RES 0603 10 KOHM 1% 0.125W AUTO"
 			(at 308.61 139.7 90)
 			(effects
@@
 			)
 		)
-		(property "Description_1" "CAP CER 0.1UF 16V X7R 0603"
+		(property "Manufacturer_Name" "Murata Electronics"
 			(at 177.165 58.42 0)
 			(effects
@@
 			)
 		)
-		(property "Manufacturer_Name" "Murata Electronics"
+		(property "Manufacturer_Part_Number" "GCJ188R71C104KA01D"
 			(at 177.165 58.42 0)
 			(effects
@@
 			)
 		)
-		(property "Manufacturer_Part_Number" "GCJ188R71C104KA01D"
+		(property "Description / Value" "CAP CER 0.1UF 16V X7R 0603"
 			(at 177.165 58.42 0)
 			(effects
@@
 			)
 		)
-		(property "Description_1" "RES 40.2K OHM 1% 1/10W 0603"
+		(property "Manufacturer_Name" "Würth Elektronik"
 			(at 308.61 114.3 90)
 			(effects
@@
 			)
 		)
-		(property "Manufacturer_Name" "Würth Elektronik"
+		(property "Manufacturer_Part_Number" "560112116003"
 			(at 308.61 114.3 90)
 			(effects
@@
 			)
 		)
-		(property "Manufacturer_Part_Number" "560112116003"
+		(property "Description / Value" "RES 40.2K OHM 1% 1/10W 0603"
 			(at 308.61 114.3 90)
 			(effects
@@
 			)
 		)
-		(property "Value" "OSD3358-512M-BSM"
+		(property "Value" "OSD3358-512M-ISM"
 			(at 224.79 45.72 0)
 			(effects
@@
 			)
 		)
-		(property "Datasheet" ""
+		(property "Datasheet" "https://mm.digikey.com/Volume0/opasdata/d220001/medias/docus/778/OSd335x-Software-PwrMgmt.pdf"
 			(at 224.79 132.08 0)
 			(effects
@@
 			)
 		)
+		(property "Manufacturer_Part_Number" "OSD3358-512M-ISM"
+			(at 224.79 132.08 0)
+			(effects
+				(font
+					(size 1.27 1.27)
+				)
+				(hide yes)
+			)
+		)
+		(property "Manufacturer_Name" "Octavo Systems LLC"
+			(at 224.79 132.08 0)
+			(effects
+				(font
+					(size 1.27 1.27)
+				)
+				(hide yes)
+			)
+		)
+		(property "Description / Value" "IC MODULE CORTEX-A8 1GHZ 512MB"
+			(at 224.79 132.08 0)
+			(effects
+				(font
+					(size 1.27 1.27)
+				)
+				(hide yes)
+			)
+		)
 		(pin "C10"
 		)
@@
 			)
 		)
-		(property "Description_1" "CAP CER 22UF 16V X7R 1210"
+		(property "Manufacturer_Name" "Murata Electronics"
 			(at 285.75 58.42 0)
 			(effects
@@
 			)
 		)
-		(property "Manufacturer_Name" "Murata Electronics"
+		(property "Manufacturer_Part_Number" "GCM32ER71C226KE19L"
 			(at 285.75 58.42 0)
 			(effects
@@
 			)
 		)
-		(property "Manufacturer_Part_Number" "GCM32ER71C226KE19L"
+		(property "Description / Value" "CAP CER 22UF 16V X7R 1210"
 			(at 285.75 58.42 0)
 			(effects
@@
 			)
 		)
-		(property "Description_1" "IC VREF SHUNT ADJ 0.5% SOT23-3"
+		(property "Manufacturer_Name" "Texas Instruments"
 			(at 298.45 124.46 90)
 			(effects
@@
 			)
 		)
-		(property "Manufacturer_Name" "Texas Instruments"
+		(property "Manufacturer_Part_Number" "TLVH431BMDBZREP"
 			(at 298.45 124.46 90)
 			(effects
@@
 			)
 		)
-		(property "Manufacturer_Part_Number" "TLVH431BMDBZREP"
+		(property "Description / Value" "IC VREF SHUNT ADJ 0.5% SOT23-3"
 			(at 298.45 124.46 90)
 			(effects
@@
 			)
 		)
-		(property "Description_1" "40V 250MW 100@150MA,10V 600MA PN"
+		(property "Manufacturer_Name" "Shenzhen Slkormicro Semicon Co., Ltd."
 			(at 288.29 132.08 0)
 			(effects
@@
 			)
 		)
-		(property "Manufacturer_Name" "Shenzhen Slkormicro Semicon Co., Ltd."
+		(property "Manufacturer_Part_Number" "MMBT2907"
 			(at 288.29 132.08 0)
 			(effects
@@
 			)
 		)
-		(property "Manufacturer_Part_Number" "MMBT2907"
+		(property "Description / Value" "40V 250MW 100@150MA,10V 600MA PN"
 			(at 288.29 132.08 0)
 			(effects
@@
 			)
 		)
-		(property "Description_1" "RES 0603 10 KOHM 1% 0.125W AUTO"
+		(property "Manufacturer_Name" "Stackpole Electronics Inc"
 			(at 299.72 210.82 0)
 			(effects
@@
 			)
 		)
-		(property "Manufacturer_Name" "Stackpole Electronics Inc"
+		(property "Manufacturer_Part_Number" "RMCA0603FT10K0-HP"
 			(at 299.72 210.82 0)
 			(effects
@@
 			)
 		)
-		(property "Manufacturer_Part_Number" "RMCA0603FT10K0-HP"
+		(property "Description / Value" "RES 0603 10 KOHM 1% 0.125W AUTO"
 			(at 299.72 210.82 0)
 			(effects
@@
 			)
 		)
-		(property "Description_1" "RES 0603 10 KOHM 1% 0.125W AUTO"
+		(property "Manufacturer_Name" "Stackpole Electronics Inc"
 			(at 298.45 76.2 0)
 			(effects
@@
 			)
 		)
-		(property "Manufacturer_Name" "Stackpole Electronics Inc"
+		(property "Manufacturer_Part_Number" "RMCA0603FT10K0-HP"
 			(at 298.45 76.2 0)
 			(effects
@@
 			)
 		)
-		(property "Manufacturer_Part_Number" "RMCA0603FT10K0-HP"
+		(property "Description / Value" "RES 0603 10 KOHM 1% 0.125W AUTO"
 			(at 298.45 76.2 0)
 			(effects
@@
 			)
 		)
-		(property "Description_1" "IC BUFF NON-INVERT 2.7V SC-70-5"
+		(property "Manufacturer_Name" "Texas Instruments"
 			(at 285.75 203.2 0)
 			(effects
@@
 			)
 		)
-		(property "Manufacturer_Name" "Texas Instruments"
+		(property "Manufacturer_Part_Number" "SN74AUC1G07DCKR"
 			(at 285.75 203.2 0)
 			(effects
@@
 			)
 		)
-		(property "Manufacturer_Part_Number" "SN74AUC1G07DCKR"
+		(property "Description / Value" "IC BUFF NON-INVERT 2.7V SC-70-5"
 			(at 285.75 203.2 0)
 			(effects
@@
 			)
 		)
-		(property "Description_1" "CAP CER 22UF 16V X7R 1210"
+		(property "Manufacturer_Name" "Murata Electronics"
 			(at 166.37 58.42 0)
 			(effects
@@
 			)
 		)
-		(property "Manufacturer_Name" "Murata Electronics"
+		(property "Manufacturer_Part_Number" "GCM32ER71C226KE19L"
 			(at 166.37 58.42 0)
 			(effects
@@
 			)
 		)
-		(property "Manufacturer_Part_Number" "GCM32ER71C226KE19L"
+		(property "Description / Value" "CAP CER 22UF 16V X7R 1210"
 			(at 166.37 58.42 0)
 			(effects
@@
 			)
 		)
-		(property "Description_1" "CAP CER 22UF 16V X7R 1210"
+		(property "Manufacturer_Name" "Murata Electronics"
 			(at 166.37 76.2 0)
 			(effects
@@
 			)
 		)
-		(property "Manufacturer_Name" "Murata Electronics"
+		(property "Manufacturer_Part_Number" "GCM32ER71C226KE19L"
 			(at 166.37 76.2 0)
 			(effects
@@
 			)
 		)
-		(property "Manufacturer_Part_Number" "GCM32ER71C226KE19L"
+		(property "Description / Value" "CAP CER 22UF 16V X7R 1210"
 			(at 166.37 76.2 0)
 			(effects

Commit message: - Fixed part number for FRAM, CAN transceiver, emmc, and BJT - Change LED and connected resistors to DNP - Verified remainder of components
Parts:
- D8, R54: now not fitted
- Q6: Manufacturer_Part_Number MMBT2907 -> PMBT2907A,235
Changed lines of the file:
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@@
 		(in_bom yes)
 		(on_board yes)
-		(dnp no)
+		(dnp yes)
 		(fields_autoplaced yes)
 		(property "Reference" "D8"
@@
 			)
 		)
-		(property "Manufacturer_Part_Number" "MMBT2907"
+		(property "Manufacturer_Part_Number" "PMBT2907A,235"
 			(at 288.29 132.08 0)
 			(effects
@@
 		(in_bom yes)
 		(on_board yes)
-		(dnp no)
+		(dnp yes)
 		(property "Reference" "R54"
 			(at 302.26 74.93 0)

Commit message: - Increased thermal relief size for Ground pads and some 3v3 pads - Made slight improvements to routing for I2C, UART lines 	- Uart 4 moved to not cross over power plane 	- Added stitching capacitor near UART2 to reduce ground loop there (5V -> GND) 	- Added stitching capacitor near UART3 aswell 	- Adding stitching capacitor between 3.3V and 5V, might remove later - Adjusted CAN0 digital lines - Adjusted some GPIO lines for better routing (7)
Other:
- note removed: "Providing DC to AC input?????"
Changed lines of the file:
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@@
-		)
-	)
-	(text "Providing DC to AC input?????"
-		(exclude_from_sim no)
-		(at 181.61 46.99 0)
-		(effects
-			(font
-				(size 1.27 1.27)
-				(bold yes)
-			)
-			(justify left bottom)
 		)
 	)

Commit message: Fixed some BOM issues. Board has been ordered, generated production files
Parts:
- U1: MPN OSD3358-512M-BSM -> OSD3358-512M-ISM
Changed lines of the file:
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@@
 			)
 		)
-		(property "MPN" "OSD3358-512M-BSM"
+		(property "MPN" "OSD3358-512M-ISM"
 			(at 224.79 132.08 0)
 			(effects
