File: kicad/oresat-c3-sch-connectors.kicad_sch (KiCad schematic)
At the start: 29 parts, among them J1 TFM-120-01-L-D-RA, J2 2-1734592-0, J3 733000020, J4 733000020

Commit message: Added Oresat symbol lib. Removed any L-band related components from pcb and schematic
Parts:
- removed J3: 733000020, oresat-connectors:J-MOLEX-SMPM-073300-002X, symbol oresat-connectors:J-MOLEX-SMPM-73300-002X
- renumbered R50 to R48
Changed lines of the file:
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@@
-    (stroke (width 0) (type default))
-  )
-  (wire (pts (xy 196.85 176.53) (xy 201.93 176.53))
     (stroke (width 0) (type default))
   )
@@
   )
   (wire (pts (xy 91.44 177.8) (xy 116.84 177.8))
-    (stroke (width 0) (type default))
-  )
-  (wire (pts (xy 191.77 181.61) (xy 191.77 184.15))
     (stroke (width 0) (type default))
   )
@@
     (effects (font (size 1.27 1.27)) (justify left))
     (property "Intersheetrefs" "${INTERSHEET_REFS}" (at 129.0591 175.26 0)
-      (effects (font (size 1.27 1.27)) (justify left))
-    )
-  )
-  (global_label "L_BAND_RF" (shape output) (at 201.93 176.53 0) (fields_autoplaced)
-    (effects (font (size 1.27 1.27)) (justify left))
-    (property "Intersheetrefs" "${INTERSHEET_REFS}" (at 215.1168 176.53 0)
       (effects (font (size 1.27 1.27)) (justify left))
     )
@@
     )
   )
-  (symbol (lib_id "oresat-connectors:J-MOLEX-SMPM-73300-002X") (at 191.77 176.53 0) (unit 1)
-    (in_bom yes) (on_board yes) (dnp no) (fields_autoplaced)
-    (property "Reference" "J3" (at 192.2526 168.91 0)
-      (effects (font (size 1.27 1.27)))
-    )
-    (property "Value" "733000020" (at 192.2526 171.45 0)
-      (effects (font (size 1.27 1.27)))
-    )
-    (property "Footprint" "oresat-connectors:J-MOLEX-SMPM-073300-002X" (at 191.77 170.18 0)
-      (effects (font (size 1.27 1.27)) hide)
-    )
-    (property "Datasheet" "https://tools.molex.com/pdm_docs/sd/733000020_sd.pdf" (at 191.77 167.64 0)
-      (effects (font (size 1.27 1.27)) hide)
-    )
-    (pin "SHLD")
-    (pin "SIG")
-    (instances
-      (project "oresat-c3"
-        (path "/65d12cdd-c326-4033-9053-c59fa4e0b25e/b9a61b98-fba0-4063-a603-e7fc9d7070a0"
-          (reference "J3") (unit 1)
-        )
-      )
-    )
-  )
   (symbol (lib_id "oresat-misc:Test-Point-1mm-round") (at 91.44 83.82 270) (unit 1)
     (in_bom yes) (on_board yes) (dnp no)
@@
   (symbol (lib_id "Device:R_Small_US") (at 214.63 83.82 90) (unit 1)
     (in_bom yes) (on_board yes) (dnp no)
-    (property "Reference" "R50" (at 214.63 86.36 90)
+    (property "Reference" "R48" (at 214.63 86.36 90)
       (effects (font (size 1.27 1.27)))
     )
@@
     (instances
       (project "oresat-c3"
-        (path "/65d12cdd-c326-4033-9053-c59fa4e0b25e/0c1da208-2d1c-4d05-9cc7-59584e50a6ac"
-          (reference "R50") (unit 1)
-        )
         (path "/65d12cdd-c326-4033-9053-c59fa4e0b25e/b9a61b98-fba0-4063-a603-e7fc9d7070a0"
           (reference "R48") (unit 1)
@@
     (instances
       (project "oresat-c3"
-        (path "/65d12cdd-c326-4033-9053-c59fa4e0b25e/0d3a1fa4-c9ee-4335-9068-a81ae0178f3f"
-          (reference "FB1") (unit 1)
-        )
         (path "/65d12cdd-c326-4033-9053-c59fa4e0b25e/b9a61b98-fba0-4063-a603-e7fc9d7070a0"
           (reference "FB1") (unit 1)
@@
         )
       )
-    )
-  )
-  (symbol (lib_id "power:GND") (at 191.77 184.15 0) (unit 1)
-    (in_bom yes) (on_board yes) (dnp no) (fields_autoplaced)
-    (property "Reference" "#PWR0104" (at 191.77 190.5 0)
-      (effects (font (size 1.27 1.27)) hide)
-    )
-    (property "Value" "GND" (at 191.77 187.96 0)
-      (effects (font (size 1.27 1.27)))
-    )
-    (property "Footprint" "" (at 191.77 184.15 0)
-      (effects (font (size 1.27 1.27)) hide)
-    )
-    (property "Datasheet" "" (at 191.77 184.15 0)
-      (effects (font (size 1.27 1.27)) hide)
-    )
-    (pin "1")
-    (instances
-      (project "oresat-c3"
-        (path "/65d12cdd-c326-4033-9053-c59fa4e0b25e/b9a61b98-fba0-4063-a603-e7fc9d7070a0"
-          (reference "#PWR0104") (unit 1)
-        )
-      )

Commit message: Removed UF band
Parts:
- removed J4: 733000020, oresat-connectors:J-MOLEX-SMPM-073300-002X, symbol oresat-connectors:J-MOLEX-SMPM-73300-002X
Changed lines of the file:
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@@
-    (stroke (width 0) (type default))
-  )
-  (wire (pts (xy 233.68 176.53) (xy 238.76 176.53))
     (stroke (width 0) (type default))
   )
@@
   )
   (wire (pts (xy 88.9 147.32) (xy 91.44 147.32))
-    (stroke (width 0) (type default))
-  )
-  (wire (pts (xy 228.6 181.61) (xy 228.6 184.15))
     (stroke (width 0) (type default))
   )
@@
     (effects (font (size 1.27 1.27)) (justify left))
     (property "Intersheetrefs" "${INTERSHEET_REFS}" (at 229.1473 76.2 0)
-      (effects (font (size 1.27 1.27)) (justify left))
-    )
-  )
-  (global_label "UHF_BAND_RF" (shape bidirectional) (at 238.76 176.53 0) (fields_autoplaced)
-    (effects (font (size 1.27 1.27)) (justify left))
-    (property "Intersheetrefs" "${INTERSHEET_REFS}" (at 255.7796 176.53 0)
       (effects (font (size 1.27 1.27)) (justify left))
     )
@@
         (path "/65d12cdd-c326-4033-9053-c59fa4e0b25e/b9a61b98-fba0-4063-a603-e7fc9d7070a0"
           (reference "TP146") (unit 1)
-        )
-      )
-    )
-  )
-  (symbol (lib_id "oresat-connectors:J-MOLEX-SMPM-73300-002X") (at 228.6 176.53 0) (unit 1)
-    (in_bom yes) (on_board yes) (dnp no) (fields_autoplaced)
-    (property "Reference" "J4" (at 228.6 168.91 0)
-      (effects (font (size 1.27 1.27)))
-    )
-    (property "Value" "733000020" (at 228.6 171.45 0)
-      (effects (font (size 1.27 1.27)))
-    )
-    (property "Footprint" "oresat-connectors:J-MOLEX-SMPM-073300-002X" (at 228.6 170.18 0)
-      (effects (font (size 1.27 1.27)) hide)
-    )
-    (property "Datasheet" "https://tools.molex.com/pdm_docs/sd/733000020_sd.pdf" (at 228.6 167.64 0)
-      (effects (font (size 1.27 1.27)) hide)
-    )
-    (pin "SHLD")
-    (pin "SIG")
-    (instances
-      (project "oresat-c3"
-        (path "/65d12cdd-c326-4033-9053-c59fa4e0b25e/b9a61b98-fba0-4063-a603-e7fc9d7070a0"
-          (reference "J4") (unit 1)
         )
       )
@@
         )
       )
-    )
-  )
-  (symbol (lib_id "power:GND") (at 228.6 184.15 0) (unit 1)
-    (in_bom yes) (on_board yes) (dnp no) (fields_autoplaced)
-    (property "Reference" "#PWR0103" (at 228.6 190.5 0)
-      (effects (font (size 1.27 1.27)) hide)
-    )
-    (property "Value" "GND" (at 228.6 187.96 0)
-      (effects (font (size 1.27 1.27)))
-    )
-    (property "Footprint" "" (at 228.6 184.15 0)
-      (effects (font (size 1.27 1.27)) hide)
-    )
-    (property "Datasheet" "" (at 228.6 184.15 0)
-      (effects (font (size 1.27 1.27)) hide)
-    )
-    (pin "1")
-    (instances
-      (project "oresat-c3"
-        (path "/65d12cdd-c326-4033-9053-c59fa4e0b25e/b9a61b98-fba0-4063-a603-e7fc9d7070a0"
-          (reference "#PWR0103") (unit 1)
-        )
-      )

Commit message: Removed antenna deployers, fixed
Connections:
- net DEPLOY_ANTENNAS: no longer names the net of J1.10, J1.9
- net DEPLOY_HELICAL: no longer names the net of J1.7, J1.8

Commit message: Finished removing components and rerouting. Still need to place voltage and GND planes
Parts:
- removed J1: TFM-120-01-L-D-RA, oresat-connectors:J-SAMTEC-TFM-120-X1-XXX-D-RA, symbol oresat-connectors:J-SAMTEC-TFM-120-01-L-D-RA
- removed J2: 2-1734592-0, oresat-connectors:J-TE-2-1734592-0, symbol oresat-connectors:J-TE-2-1734592-0
- removed PCB1: ORESAT-CARD-V1.3-GENERIC-1RF-POS2, oresat-pcbs:ORESAT-CARD-V1.3-2RF-RIGHT, symbol oresat-pcbs:ORESAT-CARD-V1.3-2RF-RIGHT
- removed R48: 10, Resistor_SMD:R_0603_1608Metric, symbol Device:R_Small_US
- removed TP101, TP102, TP103, TP106, TP107, TP108, TP142, TP143, TP144, TP145, TP146, TP147, TP152, TP153, TP154, TP155: Test-Point, oresat-misc:TestPoint_Pad_D1.0mm, symbol oresat-misc:Test-Point-1mm-round
- added J1, J2: Conn_02x26_Odd_Even, Connector_PinSocket_2.54mm:PinSocket_2x26_P2.54mm_Vertical, symbol Connector_Generic:Conn_02x26_Odd_Even
- added J7: 2-1734592-0, oresat-connectors:J-TE-2-1734592-0, symbol oresat-connectors:J-TE-2-1734592-0
- added R2: 10, Resistor_SMD:R_0603_1608Metric, symbol Device:R_Small_US
- added TP1, TP10, TP11, TP12, TP2, TP3, TP36, TP37, TP4, TP40, TP41, TP43, TP44, TP5: Test-Point, oresat-misc:TestPoint_Pad_D1.0mm, symbol oresat-misc:Test-Point-1mm-round
Connections:
- net GND: now also J2.14 (Pin_14), J2.17 (Pin_17), J2.29 (Pin_29), J2.30 (Pin_30), J2.32 (Pin_32), J2.48 (Pin_48), J2.49 (Pin_49), J2.9 (Pin_9), J7.3 (GND), J7.6 (GND), J7.9 (GND), J7.PAD1 (PAD), J7.PAD2 (PAD)
- net OPD_PWR: now also J1.31 (Pin_31)
- net OPD_SCL: now also J1.43 (Pin_43)
- net OPD_SDA: now also J1.41 (Pin_41)
- net ORESAT_nSD: now also J1.24 (Pin_24)
- net SPARE1: now also J1.2 (Pin_2), TP3.1
- net SPARE2: now also J1.4 (Pin_4), TP4.1
- net SPARE21: now also J1.5 (Pin_5), TP2.1
- net SPARE22: now also J1.3 (Pin_3), TP1.1
- net SPARE3: now also J1.6 (Pin_6), TP5.1
- net SPARE4: now also J1.8 (Pin_8), TP10.1
- net SPARE5: now also J1.10 (Pin_10), TP11.1
- net SPARE6: now also J1.12 (Pin_12), TP12.1
- net UART0_RX: now also J1.22 (Pin_22), J7.12 (CARD-RX)
- net UART0_TX: now also J1.20 (Pin_20), J7.13 (CARD-TX)
- net USB_CLI_DM: now also J7.5 (DEVICE-D-)
- net USB_CLI_DP: now also J7.4 (DEVICE-D+)
- net VBUS: now also J2.12 (Pin_12)
- net nRESET: now also R2.2
- net at FB1.1: now also J7.1 (VBUSP), J7.2 (VBUSP)
- new net: J7.10 (NRST), R2.1
- new net: J7.17 (DEBUG-0), TP40.1
- new net: J7.18 (DEBUG-1), TP41.1
- new net: J7.19 (DEBUG-2), TP43.1
- new net: J7.20 (DEBUG-3), TP44.1
- new net: J7.7 (HOST-D+), TP36.1
- new net: J7.8 (HOST-D-), TP37.1
- new net +3.3V: J2.27 (Pin_27), J2.28 (Pin_28)
- new net +5V: J1.47 (Pin_47), J1.49 (Pin_49), J2.25 (Pin_25), J2.26 (Pin_26)
- new net CAN1H+: J1.42 (Pin_42)
- new net CAN1L-: J1.44 (Pin_44)
- new net CAN2_H+: J1.34 (Pin_34)
- new net CAN2_L-: J1.36 (Pin_36)
- no-connect marks 4 -> 71
Other:
- note added: "CSKB HEADERS"
- note added: "H1"
- note added: "H2"
- note removed: "OreSat Card Main Connector (Backplane v2)"

Commit message: Added Power and ground planes, still need to fix a few things
Connections:
- net +3.3V renamed 3.3V
- net +5V renamed 5V

Commit message: Fixed power plane issues
Parts:
- removed FID1, FID2, FID3, FID4, FID5, FID6: Fiducial, Fiducial:Fiducial_1mm_Mask2mm, symbol Mechanical:Fiducial
Other:
- note removed: "Fiducials (Front)"
- note removed: "Mechanical"
Changed lines of the file:
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@@
-    (fill (type none))
-  )
-  (rectangle (start 142.24 151.13) (end 207.01 193.04)
-    (stroke (width 0) (type default))
     (fill (type none))
   )
@@
     (effects (font (size 1.27 1.27)) (justify left bottom))
   )
-  (text "Fiducials\n(Front)" (at 154.94 187.96 0)
-    (effects (font (size 1.27 1.27)) (justify left bottom))
-  )
   (text "USB Device (Ethernet over USB)" (at 300.99 95.885 0)
     (effects (font (size 1.27 1.27)) (justify left bottom))
@@
     (effects (font (size 4 4) (thickness 0.4) bold) (justify left bottom))
   )
-  (text "Fiducials\n(Front)" (at 179.07 187.96 0)
-    (effects (font (size 1.27 1.27)) (justify left bottom))
-  )
   (text "Called C3-UART-RX" (at 130.81 88.9 0)
     (effects (font (size 1.27 1.27)) (justify left bottom))
@@
   (text "Same as C3-UART" (at 297.18 88.9 0)
     (effects (font (size 1.27 1.27)) (justify left bottom))
-  )
-  (text "Mechanical" (at 158.75 158.75 0)
-    (effects (font (size 4 4) (thickness 0.4) bold) (justify left bottom))
   )
   (text "All resistors are 0603 1% AEC-Q200 unless marked.\nAll capacitors are 0603 AEC-Q200 Vw >= 16V X5R or better unless marked."
@@
     )
   )
-  (symbol (lib_id "Mechanical:Fiducial") (at 177.8 170.18 0) (unit 1)
-    (in_bom yes) (on_board yes) (dnp no) (fields_autoplaced)
-    (property "Reference" "FID4" (at 180.34 168.91 0)
-      (effects (font (size 1.27 1.27)) (justify left))
-    )
-    (property "Value" "Fiducial" (at 180.34 171.45 0)
-      (effects (font (size 1.27 1.27)) (justify left))
-    )
-    (property "Footprint" "Fiducial:Fiducial_1mm_Mask2mm" (at 177.8 170.18 0)
-      (effects (font (size 1.27 1.27)) hide)
-    )
-    (property "Datasheet" "~" (at 177.8 170.18 0)
-      (effects (font (size 1.27 1.27)) hide)
-    )
-    (property "Part Page" "" (at 177.8 170.18 0)
-      (effects (font (size 1.27 1.27)) hide)
-    )
-    (property "Price" "" (at 177.8 170.18 0)
-      (effects (font (size 1.27 1.27)) hide)
-    )
-    (property "Total Price" "" (at 177.8 170.18 0)
-      (effects (font (size 1.27 1.27)) hide)
-    )
-    (instances
-      (project "oresat-c3"
-        (path "/65d12cdd-c326-4033-9053-c59fa4e0b25e/b9a61b98-fba0-4063-a603-e7fc9d7070a0"
-          (reference "FID4") (unit 1)
-        )
-      )
-    )
-  )
   (symbol (lib_id "oresat-power:5V") (at 165.1 85.09 0) (unit 1)
     (in_bom yes) (on_board yes) (dnp no) (fields_autoplaced)
@@
         (path "/65d12cdd-c326-4033-9053-c59fa4e0b25e/b9a61b98-fba0-4063-a603-e7fc9d7070a0"
           (reference "TP5") (unit 1)
-        )
-      )
-    )
-  )
-  (symbol (lib_id "Mechanical:Fiducial") (at 177.8 180.34 0) (unit 1)
-    (in_bom yes) (on_board yes) (dnp no) (fields_autoplaced)
-    (property "Reference" "FID6" (at 180.34 179.07 0)
-      (effects (font (size 1.27 1.27)) (justify left))
-    )
-    (property "Value" "Fiducial" (at 180.34 181.61 0)
-      (effects (font (size 1.27 1.27)) (justify left))
-    )
-    (property "Footprint" "Fiducial:Fiducial_1mm_Mask2mm" (at 177.8 180.34 0)
-      (effects (font (size 1.27 1.27)) hide)
-    )
-    (property "Datasheet" "~" (at 177.8 180.34 0)
-      (effects (font (size 1.27 1.27)) hide)
-    )
-    (property "Part Page" "" (at 177.8 180.34 0)
-      (effects (font (size 1.27 1.27)) hide)
-    )
-    (property "Price" "" (at 177.8 180.34 0)
-      (effects (font (size 1.27 1.27)) hide)
-    )
-    (property "Total Price" "" (at 177.8 180.34 0)
-      (effects (font (size 1.27 1.27)) hide)
-    )
-    (instances
-      (project "oresat-c3"
-        (path "/65d12cdd-c326-4033-9053-c59fa4e0b25e/b9a61b98-fba0-4063-a603-e7fc9d7070a0"
-          (reference "FID6") (unit 1)
         )
       )
@@
     )
   )
-  (symbol (lib_id "Mechanical:Fiducial") (at 177.8 175.26 0) (unit 1)
-    (in_bom yes) (on_board yes) (dnp no) (fields_autoplaced)
-    (property "Reference" "FID5" (at 180.34 173.99 0)
-      (effects (font (size 1.27 1.27)) (justify left))
-    )
-    (property "Value" "Fiducial" (at 180.34 176.53 0)
-      (effects (font (size 1.27 1.27)) (justify left))
-    )
-    (property "Footprint" "Fiducial:Fiducial_1mm_Mask2mm" (at 177.8 175.26 0)
-      (effects (font (size 1.27 1.27)) hide)
-    )
-    (property "Datasheet" "~" (at 177.8 175.26 0)
-      (effects (font (size 1.27 1.27)) hide)
-    )
-    (property "Part Page" "" (at 177.8 175.26 0)
-      (effects (font (size 1.27 1.27)) hide)
-    )
-    (property "Price" "" (at 177.8 175.26 0)
-      (effects (font (size 1.27 1.27)) hide)
-    )
-    (property "Total Price" "" (at 177.8 175.26 0)
-      (effects (font (size 1.27 1.27)) hide)
-    )
-    (instances
-      (project "oresat-c3"
-        (path "/65d12cdd-c326-4033-9053-c59fa4e0b25e/b9a61b98-fba0-4063-a603-e7fc9d7070a0"
-          (reference "FID5") (unit 1)
-        )
-      )
-    )
-  )
-  (symbol (lib_id "Mechanical:Fiducial") (at 156.21 180.34 0) (unit 1)
-    (in_bom yes) (on_board yes) (dnp no) (fields_autoplaced)
-    (property "Reference" "FID3" (at 158.75 179.07 0)
-      (effects (font (size 1.27 1.27)) (justify left))
-    )
-    (property "Value" "Fiducial" (at 158.75 181.61 0)
-      (effects (font (size 1.27 1.27)) (justify left))
-    )
-    (property "Footprint" "Fiducial:Fiducial_1mm_Mask2mm" (at 156.21 180.34 0)
-      (effects (font (size 1.27 1.27)) hide)
-    )
-    (property "Datasheet" "~" (at 156.21 180.34 0)
-      (effects (font (size 1.27 1.27)) hide)
-    )
-    (property "Part Page" "" (at 156.21 180.34 0)
-      (effects (font (size 1.27 1.27)) hide)
-    )
-    (property "Price" "" (at 156.21 180.34 0)
-      (effects (font (size 1.27 1.27)) hide)
-    )
-    (property "Total Price" "" (at 156.21 180.34 0)
-      (effects (font (size 1.27 1.27)) hide)
-    )
-    (instances
-      (project "oresat-c3"
-        (path "/65d12cdd-c326-4033-9053-c59fa4e0b25e/b9a61b98-fba0-4063-a603-e7fc9d7070a0"
-          (reference "FID3") (unit 1)
-        )
-      )
-    )
-  )
   (symbol (lib_id "oresat-misc:Test-Point-1mm-round") (at 128.27 64.77 270) (unit 1)
     (in_bom yes) (on_board yes) (dnp no)
@@
     )
   )
-  (symbol (lib_id "Mechanical:Fiducial") (at 156.21 170.18 0) (unit 1)
-    (in_bom yes) (on_board yes) (dnp no) (fields_autoplaced)
-    (property "Reference" "FID1" (at 158.75 168.91 0)
-      (effects (font (size 1.27 1.27)) (justify left))
-    )
-    (property "Value" "Fiducial" (at 158.75 171.45 0)
-      (effects (font (size 1.27 1.27)) (justify left))
-    )
-    (property "Footprint" "Fiducial:Fiducial_1mm_Mask2mm" (at 156.21 170.18 0)
-      (effects (font (size 1.27 1.27)) hide)
-    )
-    (property "Datasheet" "~" (at 156.21 170.18 0)
-      (effects (font (size 1.27 1.27)) hide)
-    )
-    (property "Part Page" "" (at 156.21 170.18 0)
-      (effects (font (size 1.27 1.27)) hide)
-    )
-    (property "Price" "" (at 156.21 170.18 0)
-      (effects (font (size 1.27 1.27)) hide)
-    )
-    (property "Total Price" "" (at 156.21 170.18 0)
-      (effects (font (size 1.27 1.27)) hide)
-    )
-    (instances
-      (project "oresat-c3"
-        (path "/65d12cdd-c326-4033-9053-c59fa4e0b25e/b9a61b98-fba0-4063-a603-e7fc9d7070a0"
-          (reference "FID1") (unit 1)
-        )
-      )
-    )
-  )
   (symbol (lib_id "power:GND") (at 190.5 114.3 0) (unit 1)
     (in_bom yes) (on_board yes) (dnp no) (fields_autoplaced)
@@
         )
       )
-    )
-  )
-  (symbol (lib_id "Mechanical:Fiducial") (at 156.21 175.26 0) (unit 1)
-    (in_bom yes) (on_board yes) (dnp no) (fields_autoplaced)
-    (property "Reference" "FID2" (at 158.75 173.99 0)
-      (effects (font (size 1.27 1.27)) (justify left))
-    )
-    (property "Value" "Fiducial" (at 158.75 176.53 0)
-      (effects (font (size 1.27 1.27)) (justify left))
-    )
-    (property "Footprint" "Fiducial:Fiducial_1mm_Mask2mm" (at 156.21 175.26 0)
-      (effects (font (size 1.27 1.27)) hide)
-    )
-    (property "Datasheet" "~" (at 156.21 175.26 0)
-      (effects (font (size 1.27 1.27)) hide)
-    )
-    (property "Part Page" "" (at 156.21 175.26 0)
-      (effects (font (size 1.27 1.27)) hide)
-    )
-    (property "Price" "" (at 156.21 175.26 0)
-      (effects (font (size 1.27 1.27)) hide)
-    )
-    (property "Total Price" "" (at 156.21 175.26 0)
-      (effects (font (size 1.27 1.27)) hide)
-    )
-    (instances
-      (project "oresat-c3"
-        (path "/65d12cdd-c326-4033-9053-c59fa4e0b25e/b9a61b98-fba0-4063-a603-e7fc9d7070a0"
-          (reference "FID2") (unit 1)
-        )
-      )

Commit message: Switched 3.3V generation from CSKB to OSD3358
Connections:
- net 3.3V: no longer names the net of J2.27 (Pin_27)
- net 3.3V: no longer J2.28 (Pin_28)
- no-connect marks 71 -> 73
Changed lines of the file:
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@@
   (no_connect (at 113.03 105.41))
   (no_connect (at 186.69 99.06))
+  (no_connect (at 186.69 88.9))
   (no_connect (at 113.03 87.63))
   (no_connect (at 113.03 113.03))
@@
   (no_connect (at 186.69 66.04))
   (no_connect (at 173.99 73.66))
+  (no_connect (at 173.99 88.9))
   (no_connect (at 125.73 105.41))
   (no_connect (at 113.03 90.17))
@@
     (stroke (width 0) (type default))
   )
-  (wire (pts (xy 186.69 88.9) (xy 199.39 88.9))
-    (stroke (width 0) (type default))
-  )
-  (wire (pts (xy 199.39 81.28) (xy 199.39 88.9))
-    (stroke (width 0) (type default))
-  )
   (wire (pts (xy 110.49 59.69) (xy 100.33 59.69))
     (stroke (width 0) (type default))
@@
     (stroke (width 0) (type default))
   )
-  (wire (pts (xy 158.75 88.9) (xy 158.75 82.55))
-    (stroke (width 0) (type default))
-  )
   (wire (pts (xy 125.73 67.31) (xy 128.27 67.31))
     (stroke (width 0) (type default))
@@
   )
   (wire (pts (xy 113.03 59.69) (xy 110.49 59.69))
-    (stroke (width 0) (type default))
-  )
-  (wire (pts (xy 173.99 88.9) (xy 158.75 88.9))
     (stroke (width 0) (type default))
   )
@@
     )
   )
-  (symbol (lib_id "oresat-power:3.3V") (at 199.39 81.28 0) (unit 1)
-    (in_bom yes) (on_board yes) (dnp no) (fields_autoplaced)
-    (property "Reference" "#3V07" (at 199.39 85.09 0)
-      (effects (font (size 1.27 1.27)) hide)
-    )
-    (property "Value" "3.3V" (at 199.39 76.2 0)
-      (effects (font (size 1.27 1.27)))
-    )
-    (property "Footprint" "" (at 199.39 81.28 0)
-      (effects (font (size 1.27 1.27)) hide)
-    )
-    (property "Datasheet" "" (at 199.39 81.28 0)
-      (effects (font (size 1.27 1.27)) hide)
-    )
-    (pin "1")
-    (instances
-      (project "oresat-c3"
-        (path "/65d12cdd-c326-4033-9053-c59fa4e0b25e/b9a61b98-fba0-4063-a603-e7fc9d7070a0"
-          (reference "#3V07") (unit 1)
-        )
-      )
-    )
-  )
   (symbol (lib_id "oresat-misc:Test-Point-1mm-round") (at 275.59 104.14 270) (unit 1)
     (in_bom yes) (on_board yes) (dnp no)
@@
         )
       )
-    )
-  )
-  (symbol (lib_id "oresat-power:3.3V") (at 158.75 82.55 0) (unit 1)
-    (in_bom yes) (on_board yes) (dnp no) (fields_autoplaced)
-    (property "Reference" "#3V04" (at 158.75 86.36 0)
-      (effects (font (size 1.27 1.27)) hide)
-    )
-    (property "Value" "3.3V" (at 158.75 77.47 0)
-      (effects (font (size 1.27 1.27)))
-    )
-    (property "Footprint" "" (at 158.75 82.55 0)
-      (effects (font (size 1.27 1.27)) hide)
-    )
-    (property "Datasheet" "" (at 158.75 82.55 0)
-      (effects (font (size 1.27 1.27)) hide)
-    )
-    (pin "1")
-    (instances
-      (project "oresat-c3"
-        (path "/65d12cdd-c326-4033-9053-c59fa4e0b25e/b9a61b98-fba0-4063-a603-e7fc9d7070a0"
-          (reference "#3V04") (unit 1)
-        )
-      )
