File: kicad/oresat-c3-sch-connectors.kicad_sch (KiCad schematic)
At the start: 19 parts, among them J1 Conn_02x26_Odd_Even, J2 Conn_02x26_Odd_Even, J7 2-1734592-0

Commit message: Added mounting holes
Parts:
- added H1, H2, H3, H4: MountingHole_Pad, MountingHole:MountingHole_3.2mm_M3_ISO7380_Pad, symbol Mechanical:MountingHole_Pad
Connections:
- no-connect marks 73 -> 77
Changed lines of the file:
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@@
   (no_connect (at 186.69 96.52))
   (no_connect (at 113.03 85.09))
+  (no_connect (at 285.496 188.468))
   (no_connect (at 173.99 78.74))
   (no_connect (at 173.99 101.6))
@@
   (no_connect (at 186.69 88.9))
   (no_connect (at 113.03 87.63))
+  (no_connect (at 275.336 188.722))
   (no_connect (at 113.03 113.03))
   (no_connect (at 273.05 81.28))
@@
   (no_connect (at 186.69 63.5))
   (no_connect (at 113.03 69.85))
+  (no_connect (at 265.43 188.976))
   (no_connect (at 113.03 67.31))
   (no_connect (at 113.03 102.87))
@@
   (no_connect (at 173.99 81.28))
   (no_connect (at 113.03 92.71))
+  (no_connect (at 297.688 188.976))
   (wire (pts (xy 194.31 85.09) (xy 194.31 86.36))
     (stroke (width 0) (type default))
@@
     )
   )
+  (symbol (lib_id "Mechanical:MountingHole_Pad") (at 297.688 186.436 0) (unit 1)
+    (in_bom yes) (on_board yes) (dnp no) (fields_autoplaced)
+    (property "Reference" "H4" (at 300.228 183.896 0)
+      (effects (font (size 1.27 1.27)) (justify left))
+    )
+    (property "Value" "MountingHole_Pad" (at 300.228 186.436 0)
+      (effects (font (size 1.27 1.27)) (justify left) hide)
+    )
+    (property "Footprint" "MountingHole:MountingHole_3.2mm_M3_ISO7380_Pad" (at 297.688 186.436 0)
+      (effects (font (size 1.27 1.27)) hide)
+    )
+    (property "Datasheet" "~" (at 297.688 186.436 0)
+      (effects (font (size 1.27 1.27)) hide)
+    )
+    (pin "1")
+    (instances
+      (project "oresat-c3"
+        (path "/65d12cdd-c326-4033-9053-c59fa4e0b25e/b9a61b98-fba0-4063-a603-e7fc9d7070a0"
+          (reference "H4") (unit 1)
+        )
+      )
+    )
+  )
   (symbol (lib_id "oresat-misc:Test-Point-1mm-round") (at 275.59 109.22 270) (unit 1)
     (in_bom yes) (on_board yes) (dnp no)
@@
         (path "/65d12cdd-c326-4033-9053-c59fa4e0b25e/b9a61b98-fba0-4063-a603-e7fc9d7070a0"
           (reference "TP36") (unit 1)
+        )
+      )
+    )
+  )
+  (symbol (lib_id "Mechanical:MountingHole_Pad") (at 285.496 185.928 0) (unit 1)
+    (in_bom yes) (on_board yes) (dnp no) (fields_autoplaced)
+    (property "Reference" "H3" (at 288.036 183.388 0)
+      (effects (font (size 1.27 1.27)) (justify left))
+    )
+    (property "Value" "MountingHole_Pad" (at 288.036 185.928 0)
+      (effects (font (size 1.27 1.27)) (justify left) hide)
+    )
+    (property "Footprint" "MountingHole:MountingHole_3.2mm_M3_ISO7380_Pad" (at 285.496 185.928 0)
+      (effects (font (size 1.27 1.27)) hide)
+    )
+    (property "Datasheet" "~" (at 285.496 185.928 0)
+      (effects (font (size 1.27 1.27)) hide)
+    )
+    (pin "1")
+    (instances
+      (project "oresat-c3"
+        (path "/65d12cdd-c326-4033-9053-c59fa4e0b25e/b9a61b98-fba0-4063-a603-e7fc9d7070a0"
+          (reference "H3") (unit 1)
         )
       )
@@
     )
   )
+  (symbol (lib_id "Mechanical:MountingHole_Pad") (at 275.336 186.182 0) (unit 1)
+    (in_bom yes) (on_board yes) (dnp no) (fields_autoplaced)
+    (property "Reference" "H2" (at 277.876 183.642 0)
+      (effects (font (size 1.27 1.27)) (justify left))
+    )
+    (property "Value" "MountingHole_Pad" (at 277.876 186.182 0)
+      (effects (font (size 1.27 1.27)) (justify left) hide)
+    )
+    (property "Footprint" "MountingHole:MountingHole_3.2mm_M3_ISO7380_Pad" (at 275.336 186.182 0)
+      (effects (font (size 1.27 1.27)) hide)
+    )
+    (property "Datasheet" "~" (at 275.336 186.182 0)
+      (effects (font (size 1.27 1.27)) hide)
+    )
+    (pin "1")
+    (instances
+      (project "oresat-c3"
+        (path "/65d12cdd-c326-4033-9053-c59fa4e0b25e/b9a61b98-fba0-4063-a603-e7fc9d7070a0"
+          (reference "H2") (unit 1)
+        )
+      )
+    )
+  )
   (symbol (lib_id "oresat-misc:Test-Point-1mm-round") (at 128.27 69.85 270) (unit 1)
     (in_bom yes) (on_board yes) (dnp no)
@@
         )
       )
+    )
+  )
+  (symbol (lib_id "Mechanical:MountingHole_Pad") (at 265.43 186.436 0) (unit 1)
+    (in_bom yes) (on_board yes) (dnp no) (fields_autoplaced)
+    (property "Reference" "H1" (at 267.97 183.896 0)
+      (effects (font (size 1.27 1.27)) (justify left))
+    )
+    (property "Value" "MountingHole_Pad" (at 267.97 186.436 0)
+      (effects (font (size 1.27 1.27)) (justify left) hide)
+    )
+    (property "Footprint" "MountingHole:MountingHole_3.2mm_M3_ISO7380_Pad" (at 265.43 186.436 0)
+      (effects (font (size 1.27 1.27)) hide)
+    )
+    (property "Datasheet" "~" (at 265.43 186.436 0)
+      (effects (font (size 1.27 1.27)) hide)
+    )
+    (pin "1")
+    (instances
+      (project "oresat-c3"
+        (path "/65d12cdd-c326-4033-9053-c59fa4e0b25e/b9a61b98-fba0-4063-a603-e7fc9d7070a0"
+          (reference "H1") (unit 1)
+        )
+      )
