File: kicad/oresat-c3-sch-connectors.kicad_sch (KiCad schematic)
At the start: 15 parts, among them J1 Conn_02x26_Odd_Even, J2 Conn_02x26_Odd_Even, J7 2-1734592-0

Commit message: - Routed New boot pin properly, added test points to old spots as backups - Filled some floating ground planes with vias near I2C2 Buffer - Routed UART0 to new pins properly - Fixed SD card connector, it somehow got moved - Fixed som DRC issues, still need to go through a lot - Labelled CSKB, added x to anything unconnected
Connections:
- no-connect marks 17 -> 69
Changed lines of the file:
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@@
+	)
+	(no_connect
+		(at 106.68 68.58)
 	)
 	(no_connect
@@
 	)
 	(no_connect
+		(at 189.23 86.36)
+	)
+	(no_connect
+		(at 189.23 81.28)
+	)
+	(no_connect
+		(at 129.54 109.22)
+	)
+	(no_connect
+		(at 129.54 93.98)
+	)
+	(no_connect
+		(at 189.23 73.66)
+	)
+	(no_connect
+		(at 106.68 76.2)
+	)
+	(no_connect
+		(at 189.23 71.12)
+	)
+	(no_connect
+		(at 189.23 119.38)
+	)
+	(no_connect
 		(at 289.56 64.77)
 	)
 	(no_connect
+		(at 129.54 96.52)
+	)
+	(no_connect
+		(at 189.23 76.2)
+	)
+	(no_connect
 		(at 189.23 99.06)
 	)
 	(no_connect
+		(at 212.09 66.04)
+	)
+	(no_connect
+		(at 129.54 60.96)
+	)
+	(no_connect
+		(at 212.09 58.42)
+	)
+	(no_connect
+		(at 212.09 86.36)
+	)
+	(no_connect
+		(at 212.09 60.96)
+	)
+	(no_connect
+		(at 106.68 96.52)
+	)
+	(no_connect
 		(at 289.56 74.93)
 	)
 	(no_connect
+		(at 189.23 96.52)
+	)
+	(no_connect
+		(at 212.09 104.14)
+	)
+	(no_connect
 		(at 189.23 109.22)
 	)
 	(no_connect
+		(at 189.23 58.42)
+	)
+	(no_connect
+		(at 212.09 121.92)
+	)
+	(no_connect
+		(at 189.23 121.92)
+	)
+	(no_connect
+		(at 212.09 76.2)
+	)
+	(no_connect
+		(at 106.68 81.28)
+	)
+	(no_connect
+		(at 129.54 106.68)
+	)
+	(no_connect
 		(at 212.09 101.6)
 	)
 	(no_connect
+		(at 212.09 71.12)
+	)
+	(no_connect
+		(at 212.09 106.68)
+	)
+	(no_connect
+		(at 129.54 81.28)
+	)
+	(no_connect
 		(at 289.56 72.39)
 	)
 	(no_connect
+		(at 129.54 68.58)
+	)
+	(no_connect
+		(at 129.54 111.76)
+	)
+	(no_connect
+		(at 106.68 91.44)
+	)
+	(no_connect
+		(at 189.23 106.68)
+	)
+	(no_connect
+		(at 212.09 81.28)
+	)
+	(no_connect
 		(at 212.09 91.44)
 	)
 	(no_connect
+		(at 106.68 73.66)
+	)
+	(no_connect
+		(at 129.54 83.82)
+	)
+	(no_connect
+		(at 189.23 66.04)
+	)
+	(no_connect
 		(at 189.23 114.3)
 	)
@@
 	)
 	(no_connect
+		(at 129.54 88.9)
+	)
+	(no_connect
+		(at 129.54 58.42)
+	)
+	(no_connect
 		(at 212.09 99.06)
 	)
 	(no_connect
+		(at 189.23 63.5)
+	)
+	(no_connect
 		(at 106.68 106.68)
 	)
 	(no_connect
+		(at 106.68 88.9)
+	)
+	(no_connect
+		(at 212.09 63.5)
+	)
+	(no_connect
+		(at 129.54 91.44)
+	)
+	(no_connect
 		(at 212.09 111.76)
 	)
 	(no_connect
+		(at 129.54 73.66)
+	)
+	(no_connect
 		(at 289.56 69.85)
 	)
 	(no_connect
+		(at 212.09 119.38)
+	)
+	(no_connect
+		(at 189.23 60.96)
+	)
+	(no_connect
+		(at 129.54 86.36)
+	)
+	(no_connect
+		(at 106.68 71.12)
+	)
+	(no_connect
+		(at 106.68 93.98)
+	)
+	(no_connect
+		(at 129.54 76.2)
+	)
+	(no_connect
+		(at 189.23 104.14)
+	)
+	(no_connect
+		(at 212.09 68.58)
+	)
+	(no_connect
 		(at 212.09 114.3)
 	)
@@
 		(at 189.23 111.76)
 	)
+	(no_connect
+		(at 129.54 71.12)
+	)
 	(wire

Commit message: - Removed ground from mounting holes - Moves SLIP header lower so it doesnt go off edge of PCB
Connections:
- net GND: no longer H1.1, H2.1, H3.1, H4.1
- no-connect marks 69 -> 73

Commit message: added automotive grade capacitors to the BOM
Parts:
- FB1: Description_1 (none) -> FERRITE BEAD 30 OHM 0603 1LN; Manufacturer_Name (none) -> Murata Electronics; Manufacturer_Part_Number (none) -> BLM18KG300JH1D
- J1, J2: Description_1 (none) -> CONN SOCKET 52POS 0.1 GOLD PCB; Manufacturer_Name SAMTEC -> Samtec Inc.; Manufacturer_Part_Number ESQ-126-39-G-D-001 -> ESQ-126-39-G-D
- R2: Description_1 (none) -> RES 10 OHM 1% 1/8W 0603; Manufacturer_Name (none) -> Stackpole Electronics Inc; Manufacturer_Part_Number (none) -> RNCP0603FTD10R0
Changed lines of the file:
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@@
+			)
+		)
+		(property "Description_1" "FERRITE BEAD 30 OHM 0603 1LN"
+			(at 293.37 59.69 90)
+			(effects
+				(font
+					(size 1.27 1.27)
+				)
+				(hide yes)
+			)
+		)
+		(property "Manufacturer_Name" "Murata Electronics"
+			(at 293.37 59.69 90)
+			(effects
+				(font
+					(size 1.27 1.27)
+				)
+				(hide yes)
+			)
+		)
+		(property "Manufacturer_Part_Number" "BLM18KG300JH1D"
+			(at 293.37 59.69 90)
+			(effects
+				(font
+					(size 1.27 1.27)
+				)
+				(hide yes)
 			)
 		)
@@
 			)
 		)
-		(property "Manufacturer_Name" "SAMTEC"
+		(property "Manufacturer_Name" "Samtec Inc."
 			(at 208.28 553.34 0)
 			(effects
@@
 			)
 		)
-		(property "Manufacturer_Part_Number" "ESQ-126-39-G-D-001"
+		(property "Manufacturer_Part_Number" "ESQ-126-39-G-D"
 			(at 208.28 653.34 0)
 			(effects
@@
 				)
 				(justify left top)
+				(hide yes)
+			)
+		)
+		(property "Description_1" "CONN SOCKET 52POS 0.1 GOLD PCB"
+			(at 189.23 58.42 0)
+			(effects
+				(font
+					(size 1.27 1.27)
+				)
 				(hide yes)
 			)
@@
 			)
 		)
+		(property "Description_1" "RES 10 OHM 1% 1/8W 0603"
+			(at 293.37 67.31 90)
+			(effects
+				(font
+					(size 1.27 1.27)
+				)
+				(hide yes)
+			)
+		)
+		(property "Manufacturer_Name" "Stackpole Electronics Inc"
+			(at 293.37 67.31 90)
+			(effects
+				(font
+					(size 1.27 1.27)
+				)
+				(hide yes)
+			)
+		)
+		(property "Manufacturer_Part_Number" "RNCP0603FTD10R0"
+			(at 293.37 67.31 90)
+			(effects
+				(font
+					(size 1.27 1.27)
+				)
+				(hide yes)
+			)
+		)
 		(pin "1"
 		)
@@
 			)
 		)
-		(property "Manufacturer_Name" "SAMTEC"
+		(property "Manufacturer_Name" "Samtec Inc."
 			(at 125.73 553.34 0)
 			(effects
@@
 			)
 		)
-		(property "Manufacturer_Part_Number" "ESQ-126-39-G-D-001"
+		(property "Manufacturer_Part_Number" "ESQ-126-39-G-D"
 			(at 125.73 653.34 0)
 			(effects
@@
 				(hide yes)
 			)
+		)
+		(property "Description_1" "CONN SOCKET 52POS 0.1 GOLD PCB"
+			(at 106.68 58.42 0)
+			(effects
+				(font
+					(size 1.27 1.27)
+				)
+				(hide yes)
+			)

Commit message: added automotive grade resistors to BOM
Parts:
- R2: Description_1 RES 10 OHM 1% 1/8W 0603 -> RES 0603 10 OHM 1% 0.125W AUTO; Manufacturer_Part_Number RNCP0603FTD10R0 -> RMCA0603FT10R0-HP
Changed lines of the file:
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@@
 			)
 		)
-		(property "Description_1" "RES 10 OHM 1% 1/8W 0603"
+		(property "Description_1" "RES 0603 10 OHM 1% 0.125W AUTO"
 			(at 293.37 67.31 90)
 			(effects
@@
 			)
 		)
-		(property "Manufacturer_Part_Number" "RNCP0603FTD10R0"
+		(property "Manufacturer_Part_Number" "RMCA0603FT10R0-HP"
 			(at 293.37 67.31 90)
 			(effects

Commit message: modified BOM to match PCBWay format
Parts:
- H1, H2, H3, H4, TP36, TP37, TP40, TP41, TP43, TP44: now not fitted
Changed lines of the file:
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@@
 		(in_bom yes)
 		(on_board yes)
-		(dnp no)
+		(dnp yes)
 		(fields_autoplaced yes)
 		(property "Reference" "H4"
@@
 		(in_bom yes)
 		(on_board yes)
-		(dnp no)
+		(dnp yes)
 		(property "Reference" "TP40"
 			(at 294.64 102.235 90)
@@
 		(in_bom yes)
 		(on_board yes)
-		(dnp no)
+		(dnp yes)
 		(property "Reference" "TP36"
 			(at 294.64 94.615 90)
@@
 		(in_bom yes)
 		(on_board yes)
-		(dnp no)
+		(dnp yes)
 		(fields_autoplaced yes)
 		(property "Reference" "H3"
@@
 		(in_bom yes)
 		(on_board yes)
-		(dnp no)
+		(dnp yes)
 		(property "Reference" "TP37"
 			(at 294.64 97.155 90)
@@
 		(in_bom yes)
 		(on_board yes)
-		(dnp no)
+		(dnp yes)
 		(fields_autoplaced yes)
 		(property "Reference" "H2"
@@
 		(in_bom yes)
 		(on_board yes)
-		(dnp no)
+		(dnp yes)
 		(property "Reference" "TP44"
 			(at 294.64 109.855 90)
@@
 		(in_bom yes)
 		(on_board yes)
-		(dnp no)
+		(dnp yes)
 		(property "Reference" "TP43"
 			(at 294.64 107.315 90)
@@
 		(in_bom yes)
 		(on_board yes)
-		(dnp no)
+		(dnp yes)
 		(property "Reference" "TP41"
 			(at 294.64 104.775 90)
@@
 		(in_bom yes)
 		(on_board yes)
-		(dnp no)
+		(dnp yes)
 		(fields_autoplaced yes)
 		(property "Reference" "H1"

Commit message: finished putting together BOM, needs review
Parts:
- FB1: Description / Value (none) -> FERRITE BEAD 30 OHM 0603 1LN; Description_1 FERRITE BEAD 30 OHM 0603 1LN -> (none)
- J1, J2: Description / Value (none) -> CONN SOCKET 52POS 0.1 GOLD PCB; Description_1 CONN SOCKET 52POS 0.1 GOLD PCB -> (none)
- J7: Description / Value (none) -> CONN FPC BOTTOM 20POS 0.5MM R/A; Manufacturer_Name (none) -> TE Connectivity AMP Connectors; Manufacturer_Part_Number (none) -> 2-1734592-0
- R2: Description / Value (none) -> RES 0603 10 OHM 1% 0.125W AUTO; Description_1 RES 0603 10 OHM 1% 0.125W AUTO -> (none)
Changed lines of the file:
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@@
-			)
-		)
-		(property "Description_1" "FERRITE BEAD 30 OHM 0603 1LN"
-			(at 293.37 59.69 90)
-			(effects
-				(font
-					(size 1.27 1.27)
-				)
-				(hide yes)
 			)
 		)
@@
 		)
 		(property "Manufacturer_Part_Number" "BLM18KG300JH1D"
+			(at 293.37 59.69 90)
+			(effects
+				(font
+					(size 1.27 1.27)
+				)
+				(hide yes)
+			)
+		)
+		(property "Description / Value" "FERRITE BEAD 30 OHM 0603 1LN"
 			(at 293.37 59.69 90)
 			(effects
@@
 		)
 		(property "Total Price" ""
+			(at 279.4 87.63 0)
+			(effects
+				(font
+					(size 1.27 1.27)
+				)
+				(hide yes)
+			)
+		)
+		(property "Manufacturer_Name" "TE Connectivity AMP Connectors"
+			(at 279.4 87.63 0)
+			(effects
+				(font
+					(size 1.27 1.27)
+				)
+				(hide yes)
+			)
+		)
+		(property "Manufacturer_Part_Number" "2-1734592-0"
+			(at 279.4 87.63 0)
+			(effects
+				(font
+					(size 1.27 1.27)
+				)
+				(hide yes)
+			)
+		)
+		(property "Description / Value" "CONN FPC BOTTOM 20POS 0.5MM R/A"
 			(at 279.4 87.63 0)
 			(effects
@@
 			)
 		)
-		(property "Description_1" "CONN SOCKET 52POS 0.1 GOLD PCB"
+		(property "Description / Value" "CONN SOCKET 52POS 0.1 GOLD PCB"
 			(at 189.23 58.42 0)
 			(effects
@@
 			)
 		)
-		(property "Description_1" "RES 0603 10 OHM 1% 0.125W AUTO"
-			(at 293.37 67.31 90)
-			(effects
-				(font
-					(size 1.27 1.27)
-				)
-				(hide yes)
-			)
-		)
 		(property "Manufacturer_Name" "Stackpole Electronics Inc"
 			(at 293.37 67.31 90)
@@
 		)
 		(property "Manufacturer_Part_Number" "RMCA0603FT10R0-HP"
+			(at 293.37 67.31 90)
+			(effects
+				(font
+					(size 1.27 1.27)
+				)
+				(hide yes)
+			)
+		)
+		(property "Description / Value" "RES 0603 10 OHM 1% 0.125W AUTO"
 			(at 293.37 67.31 90)
 			(effects
@@
 			)
 		)
-		(property "Description_1" "CONN SOCKET 52POS 0.1 GOLD PCB"
+		(property "Description / Value" "CONN SOCKET 52POS 0.1 GOLD PCB"
 			(at 106.68 58.42 0)
 			(effects

Commit message: - Increased thermal relief size for Ground pads and some 3v3 pads - Made slight improvements to routing for I2C, UART lines 	- Uart 4 moved to not cross over power plane 	- Added stitching capacitor near UART2 to reduce ground loop there (5V -> GND) 	- Added stitching capacitor near UART3 aswell 	- Adding stitching capacitor between 3.3V and 5V, might remove later - Adjusted CAN0 digital lines - Adjusted some GPIO lines for better routing (7)
Parts:
- added C4, C5, C6: 10n, Capacitor_SMD:C_0603_1608Metric, symbol Device:C_Small
Connections:
- net 5V: now also C4.1, C5.1, C6.1
- net GND: now also C4.2, C5.2
- new net 3.3V: C6.2
Other:
- note added: "Stitching Capacitors"

Commit message: Finished rerouting CAN
Connections:
- net CAN1+: now also J1.3; no longer J1.1
- net CAN1-: now also J1.1; no longer J1.3
