File: kicad/oresat-c3.kicad_pcb (KiCad board)
At the start: 4 copper layers, 90.2 x 95.9 mm, 227 parts, among them J1 Conn_02x26_Odd_Even, J2 Conn_02x26_Odd_Even, J5 DM3BT-DSF-PEJS, J6 Conn_01x02, J7 2-1734592-0, Q1 NTR4101P, Q6 MMBT2907, U1 OSD3358-512M-BSM, U10 SN74AUC1G07DCKR, U11 RCLAMP0504FB, U12 RCLAMP0504FB, U14 TLVH431, U24 RV-3028-C7, U28 TLV1704-SEP, U30 FM24CL64B-DGTR, U37 LTC4300A-1, U39 TCAN330, U8 TCAN330, U9 EMMC+RESET+5.1-COMPATIBLE-BA, Y1 ECS-240-12-30BQ-AEN-TR, Y2 ABS07-32.768KHZ-T

Commit message: Switched 5V on AC_Input to a plane instead of traces
Routing:
- net 5V: track 12.5 -> 0.00 mm, vias 4 -> 6
- added copper zone on F.Cu, net 5V
Changed lines of the file:
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@@
 		(net 2)
 	)
-	(segment
-		(start 100.805 102.955)
-		(end 100.805 102.555)
-		(width 0.25)
-		(layer "F.Cu")
-		(net 3)
-	)
-	(segment
-		(start 100.805 101.685)
-		(end 100.805 101.955)
-		(width 0.25)
-		(layer "F.Cu")
-		(net 3)
-	)
-	(segment
-		(start 102.525 111.4)
-		(end 102.525 114.6)
-		(width 0.3)
-		(layer "F.Cu")
-		(net 3)
-	)
-	(segment
-		(start 102.475 109.025)
-		(end 102.475 111.35)
-		(width 0.3)
-		(layer "F.Cu")
-		(net 3)
-	)
-	(segment
-		(start 102.475 109.025)
-		(end 102.475 106.2)
-		(width 0.3)
-		(layer "F.Cu")
-		(net 3)
-	)
-	(segment
-		(start 100.805 102.555)
-		(end 100.6 102.35)
-		(width 0.25)
-		(layer "F.Cu")
-		(net 3)
-	)
-	(segment
-		(start 100.6 104.02)
-		(end 100.805 104.225)
-		(width 0.25)
-		(layer "F.Cu")
-		(net 3)
-	)
-	(segment
-		(start 100.805 101.955)
-		(end 101.2 102.35)
-		(width 0.25)
-		(layer "F.Cu")
-		(net 3)
-	)
-	(segment
-		(start 100.6 103.6)
-		(end 100.6 104.02)
-		(width 0.25)
-		(layer "F.Cu")
-		(net 3)
-	)
-	(segment
-		(start 102.475 106.2)
-		(end 101.2 104.925)
-		(width 0.3)
-		(layer "F.Cu")
-		(net 3)
-	)
-	(segment
-		(start 102.475 111.35)
-		(end 102.525 111.4)
-		(width 0.3)
-		(layer "F.Cu")
-		(net 3)
-	)
 	(via
 		(at 100.6 103.6)
@@
 	)
 	(via
+		(at 100.6348 104.902)
+		(size 0.4572)
+		(drill 0.254)
+		(layers "F.Cu" "B.Cu")
+		(free yes)
+		(net 3)
+	)
+	(via
 		(at 100.6 102.35)
 		(size 0.4572)
@@
 		(net 3)
 	)
+	(via
+		(at 101.1936 103.5812)
+		(size 0.4572)
+		(drill 0.254)
+		(layers "F.Cu" "B.Cu")
+		(free yes)
+		(net 3)
+	)
 	(segment
 		(start 95.725 83.975)
@@
 			)
 		)
+	)
+	(zone
+		(net 3)
+		(net_name "5V")
+		(layer "F.Cu")
+		(hatch none 0.508)
+		(priority 24)
+		(connect_pads yes
+			(clearance 0.2)
+		)
+		(min_thickness 0.127)
+		(filled_areas_thickness no)
+		(fill yes
+			(thermal_gap 0.127)
+			(thermal_bridge_width 0.2)
+			(smoothing fillet)
+			(radius 0.2)
+		)
+		(polygon
+			(pts
+				(xy 101.59435 101.2492) (xy 101.59435 105.397466) (xy 102.3256 106.0857) (xy 103.2256 106.9857)
+				(xy 103.2256 116.16895) (xy 101.750821 116.16895) (xy 101.71835 107.294046) (xy 100.3236 106.0492)
+				(xy 100.3236 101.2492)
+			)
+		)

Commit message: Brought out some pins that need to be used for UART SLIP connection on sysboot schematic
Parts:
- added J3: Conn_01x03, Connector_PinHeader_2.54mm:PinHeader_1x03_P2.54mm_Vertical, F.Cu at (71.7, 101.1)
Routing:
- net Net-(J3-Pin_1): track 17.1 -> 25.3 mm
- net Net-(J3-Pin_2): track 23.4 -> 28.4 mm
- net 3.3V: track 134.9 -> 136.4 mm
- net Net-(R72-66): track 19.7 -> 19.0 mm

Commit message: Added via stitching
Parts:
- moved G*** 1.44 mm to (131.0, 102.0)
Routing:
- net GND: vias 190 -> 339
