File: kicad/oresat-c3.kicad_pcb (KiCad board)
At the start: 4 copper layers, 90.2 x 95.9 mm, 228 parts, among them J1 Conn_02x26_Odd_Even, J2 Conn_02x26_Odd_Even, J3 Conn_01x03, J5 DM3BT-DSF-PEJS, J6 Conn_01x02, J7 2-1734592-0, Q1 NTR4101P, Q6 MMBT2907, U1 OSD3358-512M-BSM, U10 SN74AUC1G07DCKR, U11 RCLAMP0504FB, U12 RCLAMP0504FB, U14 TLVH431, U24 RV-3028-C7, U28 TLV1704-SEP, U30 FM24CL64B-DGTR, U37 LTC4300A-1, U39 TCAN330, U8 TCAN330, U9 EMMC+RESET+5.1-COMPATIBLE-BA, Y1 ECS-240-12-30BQ-AEN-TR, Y2 ABS07-32.768KHZ-T

Commit message: Added UART TX pin for ADCS GNSS. Also fixed I2C SDA/SCL, they were swapped accidently
Connections:
- J1 pad 40: unconnected-(J1-Pin_40-Pad40) -> ADCS_UART_GNSS
- J1 pad 42: OPD_SCL -> OPD_SDA
- J1 pad 44: OPD_SDA -> OPD_SCL
- U1 pad A3: unconnected-(U1C-MCASP0_ACLKR-PadA3) -> ADCS_UART_GNSS
- U1 pad C5: unconnected-(U1C-ECAP0_IN_PWM0_OUT-PadC5) -> ADCS_UART_GNSS
Routing:
- net ADCS_UART_GNSS: track 0.00 -> 59.7 mm, vias 0 -> 1
- net OPD_SCL: track 20.9 -> 25.4 mm
- net OPD_SDA: track 22.0 -> 19.8 mm
- net I2C2_SYS_DISABLE: track 93.8 -> 92.0 mm
- net PET_WDT: track 64.9 -> 64.3 mm

Commit message: pcb changes
Other:
- board text added: "RX"
- board text added: "TX"
Changed lines of the file:
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@@
+		)
+	)
+	(gr_text "RX"
+		(at 69.2 103.6 0)
+		(layer "F.SilkS")
+		(effects
+			(font
+				(size 1 1)
+				(thickness 0.15)
+			)
+		)
+	)
+	(gr_text "TX"
+		(at 69.15 101.25 0)
+		(layer "F.SilkS")
+		(effects
+			(font
+				(size 1 1)
+				(thickness 0.15)
+			)
 		)
 	)

Commit message: Removed floating metal pours with via filling
Routing:
- net GND: vias 339 -> 350
Changed lines of the file:
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@@
+	)
+	(via
+		(at 107.7468 84.582)
+		(size 0.4572)
+		(drill 0.254)
+		(layers "F.Cu" "B.Cu")
+		(free yes)
+		(net 157)
 	)
 	(via
@@
 	)
 	(via
+		(at 103.9876 100.9904)
+		(size 0.4572)
+		(drill 0.254)
+		(layers "F.Cu" "B.Cu")
+		(free yes)
+		(net 157)
+	)
+	(via
 		(at 132.878376 49.28974)
 		(size 0.4572)
@@
 	)
 	(via
+		(at 131.3688 120.8532)
+		(size 0.4572)
+		(drill 0.254)
+		(layers "F.Cu" "B.Cu")
+		(free yes)
+		(net 157)
+	)
+	(via
 		(at 104.8 113)
 		(size 0.4572)
@@
 	)
 	(via
+		(at 100.33 67.6148)
+		(size 0.4572)
+		(drill 0.254)
+		(layers "F.Cu" "B.Cu")
+		(free yes)
+		(net 157)
+	)
+	(via
 		(at 97.65 98.5)
 		(size 0.4572)
@@
 	)
 	(via
+		(at 144.1196 72.5932)
+		(size 0.4572)
+		(drill 0.254)
+		(layers "F.Cu" "B.Cu")
+		(free yes)
+		(net 157)
+	)
+	(via
 		(at 142.878376 139.28974)
 		(size 0.4572)
@@
 	)
 	(via
+		(at 98.3488 106.3244)
+		(size 0.4572)
+		(drill 0.254)
+		(layers "F.Cu" "B.Cu")
+		(free yes)
+		(net 157)
+	)
+	(via
 		(at 137.878376 114.28974)
 		(size 0.4572)
@@
 	)
 	(via
+		(at 110.6932 90.8304)
+		(size 0.4572)
+		(drill 0.254)
+		(layers "F.Cu" "B.Cu")
+		(free yes)
+		(net 157)
+	)
+	(via
 		(at 107.878376 124.28974)
 		(size 0.4572)
@@
 	)
 	(via
+		(at 144.3736 75.9968)
+		(size 0.4572)
+		(drill 0.254)
+		(layers "F.Cu" "B.Cu")
+		(free yes)
+		(net 157)
+	)
+	(via
 		(at 111 102.85)
 		(size 0.4572)
@@
 	)
 	(via
+		(at 101.854 80.1624)
+		(size 0.4572)
+		(drill 0.254)
+		(layers "F.Cu" "B.Cu")
+		(free yes)
+		(net 157)
+	)
+	(via
 		(at 137.878376 89.28974)
 		(size 0.4572)
@@
 	)
 	(via
+		(at 126.8476 73.0504)
+		(size 0.4572)
+		(drill 0.254)
+		(layers "F.Cu" "B.Cu")
+		(free yes)
+		(net 157)
+	)
+	(via
 		(at 72.878376 54.28974)
 		(size 0.4572)
@@
 		(size 0.4572)
 		(drill 0.254)
+		(layers "F.Cu" "B.Cu")
+		(free yes)
+		(net 157)
+	)
+	(via
+		(at 98.552 109.5756)
+		(size 0.4572)
+		(drill 0.254)
