File: kicad/oresat-c3-sch-osd3358-sd-emmc.kicad_sch (KiCad schematic)
At the start: 44 parts, among them J5 DM3BT-DSF-PEJS, U1 OSD3358-512M-BSM, U8 TCAN330, U9 EMMC+RESET+5.1-COMPATIBLE-BA

Commit message: Added I2C1 bus lines
Connections:
- net I2C1_SYS_SCL: now reaches U1.A14 (SPI0_CS0)
- net I2C1_SYS_SDA: now reaches U1.B14 (SPI0_D1)
- no-connect marks 28 -> 26
Other:
- note added: "USE B14 AND A14 AS I2C1 BUS"
- note removed: "TO UHF RADIO (AX5043)"
Changed lines of the file:
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@@
 	)
 	(no_connect
-		(at 154.94 137.16)
-	)
-	(no_connect
 		(at 223.52 144.78)
 	)
@@
 	)
 	(no_connect
-		(at 154.94 139.7)
-	)
-	(no_connect
 		(at 154.94 177.8)
 	)
@@
 		)
 	)
-	(text "TO UHF RADIO\n(AX5043)"
+	(text "USE B14 AND A14 \nAS I2C1 BUS\n"
 		(exclude_from_sim no)
-		(at 123.19 137.16 0)
+		(at 119.126 136.398 0)
 		(effects
 			(font
@@
 		)
 	)
+	(global_label "I2C1_SYS_SDA"
+		(shape input)
+		(at 154.94 137.16 180)
+		(fields_autoplaced yes)
+		(effects
+			(font
+				(size 1.27 1.27)
+			)
+			(justify right)
+		)
+		(property "Intersheetrefs" "${INTERSHEET_REFS}"
+			(at 138.6501 137.16 0)
+			(effects
+				(font
+					(size 1.27 1.27)
+				)
+				(justify right)
+			)
+		)
+	)
 	(global_label "OPD_nENABLE"
 		(shape output)
@@
 			(effects
 				(font
+					(size 1.27 1.27)
+				)
+				(justify right)
+			)
+		)
+	)
+	(global_label "I2C1_SYS_SCL"
+		(shape input)
+		(at 154.94 139.7 180)
+		(fields_autoplaced yes)
+		(effects
+			(font
+				(size 1.27 1.27)
+			)
+			(justify right)
+		)
+		(property "Intersheetrefs" "${INTERSHEET_REFS}"
+			(at 138.7106 139.7 0)
+			(effects
+				(font

Commit message: Removed OPD and added LTC4300A to I2C1 bus
Connections:
- net OPD_nENABLE: no longer names the net of U1.C3 (MCASP0_AXR1)
- net OPD_nFAULT: no longer names the net of U1.B3 (MCASP0_FSR)
- no-connect marks 26 -> 28
Changed lines of the file:
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@@
 	)
 	(no_connect
+		(at 154.94 182.88)
+	)
+	(no_connect
 		(at 223.52 144.78)
 	)
@@
 	)
 	(no_connect
+		(at 154.94 185.42)
+	)
+	(no_connect
 		(at 231.14 106.68)
 	)
@@
 	)
 	(global_label "I2C1_SYS_SDA"
-		(shape input)
+		(shape bidirectional)
 		(at 154.94 137.16 180)
 		(fields_autoplaced yes)
@@
 		)
 		(property "Intersheetrefs" "${INTERSHEET_REFS}"
-			(at 138.6501 137.16 0)
-			(effects
-				(font
-					(size 1.27 1.27)
-				)
-				(justify right)
-			)
-		)
-	)
-	(global_label "OPD_nENABLE"
-		(shape output)
-		(at 154.94 185.42 180)
-		(fields_autoplaced yes)
-		(effects
-			(font
-				(size 1.27 1.27)
-			)
-			(justify right)
-		)
-		(property "Intersheetrefs" "${INTERSHEET_REFS}"
-			(at 139.0319 185.42 0)
+			(at 137.5388 137.16 0)
 			(effects
 				(font
@@
 			)
 		)
-	)
-	(global_label "OPD_nFAULT"
-		(shape input)
-		(at 154.94 182.88 180)
-		(fields_autoplaced yes)
-		(effects
-			(font
-				(size 1.27 1.27)
-			)
-			(justify right)
-		)
-		(property "Intersheetrefs" "${INTERSHEET_REFS}"
-			(at 140.5437 182.88 0)
-			(effects
-				(font
-					(size 1.27 1.27)
-				)
-				(justify right)
-			)
-		)

Commit message: Added CAN bus termination resistors
Parts:
- added R1: 120k, Resistor_SMD:R_0603_1608Metric, symbol Device:R_Small_US
Connections:
- net CAN1H+: now also R1.2
- net CAN1L-: now also R1.1
Changed lines of the file:
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@@
 	)
 	(junction
+		(at 176.53 69.85)
+		(diameter 0)
+		(color 0 0 0 0)
+	)
+	(junction
 		(at 274.32 208.28)
 		(diameter 0)
@@
 	)
 	(junction
+		(at 176.53 64.77)
+		(diameter 0)
+		(color 0 0 0 0)
+	)
+	(junction
 		(at 350.52 167.64)
 		(diameter 0)
@@
 	(wire
 		(pts
+			(xy 176.53 69.85) (xy 180.34 69.85)
+		)
+		(stroke
+			(width 0)
+			(type default)
+		)
+	)
+	(wire
+		(pts
 			(xy 281.94 165.1) (xy 317.5 165.1)
 		)
@@
 	(wire
 		(pts
-			(xy 172.72 64.77) (xy 180.34 64.77)
+			(xy 172.72 64.77) (xy 176.53 64.77)
 		)
 		(stroke
@@
 	(wire
 		(pts
-			(xy 172.72 69.85) (xy 180.34 69.85)
+			(xy 172.72 69.85) (xy 176.53 69.85)
 		)
 		(stroke
@@
 	(wire
 		(pts
+			(xy 176.53 64.77) (xy 180.34 64.77)
+		)
+		(stroke
+			(width 0)
+			(type default)
+		)
+	)
+	(wire
+		(pts
 			(xy 241.3 152.4) (xy 241.3 157.48)
 		)
@@
 					(unit 1)
 				)
+			)
+		)
+	)
+	(symbol
+		(lib_id "Device:R_Small_US")
+		(at 176.53 67.31 180)
+		(unit 1)
+		(exclude_from_sim no)
+		(in_bom yes)
+		(on_board yes)
+		(dnp no)
+		(fields_autoplaced yes)
+		(property "Reference" "R1"
+			(at 179.07 66.675 0)
+			(effects
+				(font
+					(size 1.27 1.27)
+				)
+				(justify right)
+			)
+		)
+		(property "Value" "120k"
+			(at 179.07 69.215 0)
+			(effects
+				(font
+					(size 1.27 1.27)
+				)
+				(justify right)
+			)
+		)
+		(property "Footprint" "Resistor_SMD:R_0603_1608Metric"
+			(at 176.53 67.31 0)
+			(effects
+				(font
+					(size 1.27 1.27)
+				)
+				(hide yes)
+			)
+		)
+		(property "Datasheet" "~"
+			(at 176.53 67.31 0)
+			(effects
+				(font
+					(size 1.27 1.27)
+				)
+				(hide yes)
+			)
+		)
+		(property "Description" ""
+			(at 176.53 67.31 0)
+			(effects
+				(font
+					(size 1.27 1.27)
+				)
+				(hide yes)
+			)
+		)
+		(property "Part Page" ""
+			(at 176.53 67.31 0)
+			(effects
+				(font
+					(size 1.27 1.27)
+				)
+				(hide yes)
+			)
+		)
+		(property "Price" ""
+			(at 176.53 67.31 0)
+			(effects
+				(font
+					(size 1.27 1.27)
+				)
+				(hide yes)
+			)
+		)
+		(property "Total Price" ""
+			(at 176.53 67.31 0)
+			(effects
+				(font
+					(size 1.27 1.27)
+				)
+				(hide yes)
+			)
+		)
+		(pin "1"
+		)
+		(pin "2"
+		)
+		(instances
+			(project "oresat-c3"
+				(path "/65d12cdd-c326-4033-9053-c59fa4e0b25e/f3d147ad-4cea-4d77-ae60-95882b03454e"
+					(reference "R1")
+					(unit 1)
+				)

Commit message: Added GPIO enable pins for ADCS
Connections:
- net ADCS_ENABLE_CONTROL: now reaches TP46.1, U1.P7 (GPMC_AD15)
- net ADCS_BOOT_CONTROL: now reaches TP42.1, U1.T6 (GPMC_AD14)
Changed lines of the file:
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@@
 	)
 	(junction
+		(at 229.87 203.2)
+		(diameter 0)
+		(color 0 0 0 0)
+	)
+	(junction
 		(at 350.52 167.64)
 		(diameter 0)
@@
 	)
 	(junction
+		(at 229.87 200.66)
+		(diameter 0)
+		(color 0 0 0 0)
+	)
+	(junction
 		(at 269.24 157.48)
 		(diameter 0)
@@
 	(wire
 		(pts
+			(xy 236.22 203.2) (xy 229.87 203.2)
+		)
+		(stroke
+			(width 0)
+			(type default)
+		)
+	)
+	(wire
+		(pts
 			(xy 250.19 193.04) (xy 250.19 208.28)
 		)
@@
 	(wire
 		(pts
+			(xy 236.22 224.79) (xy 236.22 203.2)
+		)
+		(stroke
+			(width 0)
+			(type default)
+		)
+	)
+	(wire
+		(pts
 			(xy 114.3 132.08) (xy 86.36 132.08)
 		)
@@
 	(wire
 		(pts
+			(xy 236.22 224.79) (xy 240.03 224.79)
+		)
+		(stroke
+			(width 0)
+			(type default)
+		)
+	)
+	(wire
+		(pts
 			(xy 279.4 154.94) (xy 279.4 162.56)
 		)
@@
 	(wire
 		(pts
+			(xy 240.03 200.66) (xy 240.03 222.25)
+		)
+		(stroke
+			(width 0)
+			(type default)
+		)
+	)
+	(wire
+		(pts
 			(xy 269.24 104.14) (xy 278.13 104.14)
 		)
@@
 	(wire
 		(pts
+			(xy 240.03 200.66) (xy 229.87 200.66)
+		)
+		(stroke
+			(width 0)
+			(type default)
+		)
+	)
+	(wire
+		(pts
 			(xy 238.76 160.02) (xy 266.7 160.02)
 		)
@@
 		)
 	)
+	(global_label "ADCS_ENABLE_CONTROL"
+		(shape bidirectional)
+		(at 240.03 224.79 0)
+		(fields_autoplaced yes)
+		(effects
+			(font
+				(size 1.27 1.27)
+			)
+			(justify left)
+		)
+		(property "Intersheetrefs" "${INTERSHEET_REFS}"
+			(at 266.4422 224.79 0)
+			(effects
+				(font
+					(size 1.27 1.27)
+				)
+				(justify left)
+			)
+		)
+	)
 	(global_label "CAN1L-"
 		(shape input)
@@
 			(effects
 				(font
+					(size 1.27 1.27)
+				)
+				(justify left)
+			)
+		)
+	)
+	(global_label "ADCS_BOOT_CONTROL"
+		(shape bidirectional)
+		(at 240.03 222.25 0)
+		(fields_autoplaced yes)
+		(effects
+			(font
+				(size 1.27 1.27)
+			)
+			(justify left)
+		)
+		(property "Intersheetrefs" "${INTERSHEET_REFS}"
+			(at 264.3256 222.25 0)
+			(effects
+				(font

Commit message: Added UART TX pin for ADCS GNSS. Also fixed I2C SDA/SCL, they were swapped accidently
Connections:
- net ADCS_UART_GNSS: now reaches U1.A3 (MCASP0_ACLKR)
- net ADCS_UART_GNSS: now also U1.C5 (ECAP0_IN_PWM0_OUT)
- no-connect marks 28 -> 26
Changed lines of the file:
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@@
 	)
 	(junction
+		(at 125.73 200.66)
+		(diameter 0)
+		(color 0 0 0 0)
+	)
+	(junction
 		(at 350.52 160.02)
 		(diameter 0)
@@
 	)
 	(no_connect
-		(at 162.56 200.66)
-	)
-	(no_connect
 		(at 154.94 187.96)
 	)
@@
 	)
 	(no_connect
-		(at 154.94 180.34)
-	)
-	(no_connect
 		(at 231.14 134.62)
 	)
@@
 	(wire
 		(pts
+			(xy 118.11 200.66) (xy 125.73 200.66)
+		)
+		(stroke
+			(width 0)
+			(type default)
+		)
+	)
+	(wire
+		(pts
 			(xy 127 119.38) (xy 162.56 119.38)
 		)
@@
 	(wire
 		(pts
+			(xy 125.73 180.34) (xy 125.73 200.66)
+		)
+		(stroke
+			(width 0)
+			(type default)
+		)
+	)
+	(wire
+		(pts
 			(xy 355.6 167.64) (xy 350.52 167.64)
 		)
@@
 	(wire
 		(pts
+			(xy 125.73 200.66) (xy 162.56 200.66)
+		)
+		(stroke
+			(width 0)
+			(type default)
+		)
+	)
+	(wire
+		(pts
 			(xy 289.56 177.8) (xy 317.5 177.8)
 		)
@@
 	(wire
 		(pts
-			(xy 154.94 180.34) (xy 162.56 180.34)
-		)
-		(stroke
-			(width 0)
-			(type default)
-		)
-	)
-	(wire
-		(pts
 			(xy 223.52 165.1) (xy 281.94 165.1)
 		)
@@
 	(wire
 		(pts
+			(xy 125.73 180.34) (xy 162.56 180.34)
+		)
+		(stroke
+			(width 0)
+			(type default)
+		)
+	)
+	(wire
+		(pts
 			(xy 55.88 152.4) (xy 55.88 153.67)
 		)
@@
 			(effects
 				(font
+					(size 1.27 1.27)
+				)
+				(justify right)
+			)
+		)
+	)
+	(global_label "ADCS_UART_GNSS"
+		(shape output)
+		(at 118.11 200.66 180)
+		(fields_autoplaced yes)
+		(effects
+			(font
+				(size 1.27 1.27)
+			)
+			(justify right)
+		)
+		(property "Intersheetrefs" "${INTERSHEET_REFS}"
+			(at 98.6753 200.66 0)
+			(effects
+				(font

Commit message: Added MRAM chip to board
Connections:
- net MRAM_SPI_CLK: now reaches U1.A1 (MCASP0_ACLKX)
- net MRAM_SPI_MISO: now reaches U1.A2 (MCASP0_FSX)
- net MRAM_SPI_CS: now reaches U1.B1 (MCASP0_AHCLKR)
- net MRAM_SPI_MOSI: now reaches U1.B2 (MCASP0_AXR0)
- no-connect marks 26 -> 22
Other:
- note added: "SPI INTERFACE FOR KUBOS"
Changed lines of the file:
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@@
 	)
 	(no_connect
-		(at 154.94 175.26)
-	)
-	(no_connect
 		(at 78.74 119.38)
 	)
@@
 	)
 	(no_connect
-		(at 154.94 170.18)
-	)
-	(no_connect
-		(at 154.94 177.8)
-	)
-	(no_connect
 		(at 154.94 185.42)
 	)
@@
 		(at 231.14 129.54)
 	)
-	(no_connect
-		(at 154.94 172.72)
-	)
 	(wire
 		(pts
@@
 	(wire
 		(pts
-			(xy 154.94 177.8) (xy 162.56 177.8)
+			(xy 88.9 137.16) (xy 88.9 119.38)
 		)
 		(stroke
@@
 	(wire
 		(pts
-			(xy 88.9 137.16) (xy 88.9 119.38)
+			(xy 146.05 104.14) (xy 154.94 104.14)
 		)
 		(stroke
@@
 	(wire
 		(pts
-			(xy 146.05 104.14) (xy 154.94 104.14)
+			(xy 287.02 180.34) (xy 317.5 180.34)
 		)
 		(stroke
@@
 	(wire
 		(pts
-			(xy 287.02 180.34) (xy 317.5 180.34)
+			(xy 176.53 69.85) (xy 180.34 69.85)
 		)
 		(stroke
@@
 	(wire
 		(pts
-			(xy 176.53 69.85) (xy 180.34 69.85)
+			(xy 281.94 165.1) (xy 317.5 165.1)
 		)
 		(stroke
@@
 	(wire
 		(pts
-			(xy 281.94 165.1) (xy 317.5 165.1)
+			(xy 153.67 177.8) (xy 162.56 177.8)
 		)
 		(stroke
@@
 	(wire
 		(pts
+			(xy 153.67 172.72) (xy 162.56 172.72)
+		)
+		(stroke
+			(width 0)
+			(type default)
+		)
+	)
+	(wire
+		(pts
 			(xy 274.32 119.38) (xy 278.13 119.38)
 		)
@@
 	(wire
 		(pts
-			(xy 154.94 175.26) (xy 162.56 175.26)
-		)
-		(stroke
-			(width 0)
-			(type default)
-		)
-	)
-	(wire
-		(pts
 			(xy 375.92 160.02) (xy 383.54 160.02)
 		)
@@
 		)
 	)
+	(wire
+		(pts
+			(xy 153.67 170.18) (xy 162.56 170.18)
+		)
+		(stroke
+			(width 0)
+			(type default)
+		)
+	)
 	(polyline
 		(pts
@@
 		)
 	)
+	(polyline
+		(pts
+			(xy 135.89 179.832) (xy 138.43 179.832)
+		)
+		(stroke
+			(width 0)
+			(type default)
+		)
+	)
 	(wire
 		(pts
@@
 	(wire
 		(pts
-			(xy 154.94 170.18) (xy 162.56 170.18)
-		)
-		(stroke
-			(width 0)
-			(type default)
-		)
-	)
-	(wire
-		(pts
 			(xy 83.82 119.38) (xy 83.82 129.54)
 		)
@@
 	(wire
 		(pts
+			(xy 153.67 175.26) (xy 162.56 175.26)
+		)
+		(stroke
+			(width 0)
+			(type default)
+		)
+	)
+	(wire
+		(pts
 			(xy 114.3 152.4) (xy 162.56 152.4)
 		)
@@
 		)
 	)
+	(polyline
+		(pts
+			(xy 138.43 167.132) (xy 135.89 167.132)
+		)
+		(stroke
+			(width 0)
+			(type default)
+		)
+	)
 	(wire
 		(pts
@@
 		)
 	)
+	(polyline
+		(pts
+			(xy 135.89 167.132) (xy 135.89 179.832)
+		)
+		(stroke
+			(width 0)
+			(type default)
+		)
+	)
 	(wire
 		(pts
@@
 	(wire
 		(pts
-			(xy 154.94 172.72) (xy 162.56 172.72)
-		)
-		(stroke
-			(width 0)
-			(type default)
-		)
-	)
-	(wire
-		(pts
 			(xy 67.31 113.03) (xy 67.31 114.3)
 		)
@@
 		)
 	)
+	(text "SPI INTERFACE\nFOR KUBOS"
+		(exclude_from_sim no)
+		(at 118.872 175.26 0)
+		(effects
+			(font
+				(size 1.27 1.27)
+			)
+			(justify left bottom)
+		)
+	)
 	(text "HH"
 		(exclude_from_sim no)
@@
 		)
 	)
+	(global_label "MRAM_SPI_CLK"
+		(shape output)
+		(at 153.67 170.18 180)
+		(fields_autoplaced yes)
+		(effects
+			(font
+				(size 1.27 1.27)
+			)
+			(justify right)
+		)
+		(property "Intersheetrefs" "${INTERSHEET_REFS}"
+			(at 136.8358 170.18 0)
+			(effects
+				(font
+					(size 1.27 1.27)
+				)
+				(justify right)
+			)
+		)
+	)
 	(global_label "I2C2_SYS_DISABLE"
 		(shape input)
@@
 		)
 	)
+	(global_label "MRAM_SPI_CS"
+		(shape output)
+		(at 153.67 177.8 180)
+		(fields_autoplaced yes)
+		(effects
+			(font
+				(size 1.27 1.27)
+			)
+			(justify right)
+		)
+		(property "Intersheetrefs" "${INTERSHEET_REFS}"
+			(at 137.9244 177.8 0)
+			(effects
+				(font
+					(size 1.27 1.27)
+				)
+				(justify right)
+			)
+		)
+	)
+	(global_label "MRAM_SPI_MOSI"
+		(shape output)
+		(at 153.67 175.26 180)
+		(fields_autoplaced yes)
+		(effects
+			(font
+				(size 1.27 1.27)
+			)
+			(justify right)
+		)
+		(property "Intersheetrefs" "${INTERSHEET_REFS}"
+			(at 135.8077 175.26 0)
+			(effects
+				(font
+					(size 1.27 1.27)
+				)
+				(justify right)
+			)
+		)
+	)
 	(global_label "I2C1_SYS_SCL"
 		(shape input)
@@
 			)
 		)
+	)
+	(global_label "MRAM_SPI_MISO"
+		(shape input)
+		(at 153.67 172.72 180)
+		(fields_autoplaced yes)
+		(effects
+			(font
+				(size 1.27 1.27)
+			)
+			(justify right)
+		)
+		(property "Intersheetrefs" "${INTERSHEET_REFS}"
+			(at 135.8077 172.72 0)
+			(effects
+				(font
+					(size 1.27 1.27)
+				)
+				(justify right)
+			)
+		)

Commit message: Added extra decoupling capacitor to MRAM. Also grounded all unused pins and mounting holes
Connections:
- no-connect marks 22 -> 24
Changed lines of the file:
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@@
+	)
+	(no_connect
+		(at 162.56 109.22)
 	)
 	(no_connect
@@
 	)
 	(no_connect
+		(at 162.56 106.68)
+	)
+	(no_connect

Commit message: Fixed skew on CAN lines
Connections:
- net CAN1H+ renamed CAN1+
- net CAN1L- renamed CAN1-
Changed lines of the file:
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@@
 		)
 	)
-	(global_label "CAN1L-"
+	(global_label "CAN1-"
 		(shape input)
 		(at 180.34 69.85 0)
@@
 		)
 		(property "Intersheetrefs" "${INTERSHEET_REFS}"
-			(at 190.8243 69.85 0)
+			(at 189.7962 69.85 0)
 			(effects
 				(font
@@
 		)
 	)
-	(global_label "CAN1H+"
+	(global_label "CAN1+"
 		(shape input)
 		(at 180.34 64.77 0)
@@
 		)
 		(property "Intersheetrefs" "${INTERSHEET_REFS}"
-			(at 191.1267 64.77 0)
+			(at 189.7962 64.77 0)
 			(effects
 				(font
