File: kicad/oresat-c3-sch-osd3358-sd-emmc.kicad_sch (KiCad schematic)
At the start: 45 parts, among them J5 DM3BT-DSF-PEJS, U1 OSD3358-512M-BSM, U8 TCAN330, U9 EMMC+RESET+5.1-COMPATIBLE-BA

Commit message: - Locked CSKB Headers on PCB - Removed CAN1 from schematic - Removed ADCS boot enable from schematic - Removed unnecessary grounds from PCB
Parts:
- removed TP42: Test-Point, oresat-misc:TestPoint_Pad_D1.0mm, symbol oresat-misc:Test-Point-1mm-round
Connections:
- net ADCS_BOOT_CONTROL: no longer names the net of U1.T6 (GPMC_AD14)
Changed lines of the file:
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@@
 	)
 	(junction
-		(at 229.87 200.66)
-		(diameter 0)
-		(color 0 0 0 0)
-	)
-	(junction
 		(at 269.24 157.48)
 		(diameter 0)
@@
 	(wire
 		(pts
-			(xy 240.03 200.66) (xy 240.03 222.25)
-		)
-		(stroke
-			(width 0)
-			(type default)
-		)
-	)
-	(wire
-		(pts
 			(xy 269.24 104.14) (xy 278.13 104.14)
 		)
@@
 	(wire
 		(pts
-			(xy 240.03 200.66) (xy 229.87 200.66)
-		)
-		(stroke
-			(width 0)
-			(type default)
-		)
-	)
-	(wire
-		(pts
 			(xy 238.76 160.02) (xy 266.7 160.02)
 		)
@@
 	(wire
 		(pts
-			(xy 223.52 200.66) (xy 229.87 200.66)
-		)
-		(stroke
-			(width 0)
-			(type default)
-		)
-	)
-	(wire
-		(pts
 			(xy 270.51 193.04) (xy 274.32 193.04)
 		)
@@
 		)
 	)
-	(global_label "ADCS_BOOT_CONTROL"
-		(shape bidirectional)
-		(at 240.03 222.25 0)
-		(fields_autoplaced yes)
-		(effects
-			(font
-				(size 1.27 1.27)
-			)
-			(justify left)
-		)
-		(property "Intersheetrefs" "${INTERSHEET_REFS}"
-			(at 264.3256 222.25 0)
-			(effects
-				(font
-					(size 1.27 1.27)
-				)
-				(justify left)
-			)
-		)
-	)
 	(global_label "UART0_TX"
 		(shape input)
@@
 					(unit 1)
 				)
-			)
-		)
-	)
-	(symbol
-		(lib_id "oresat-misc:Test-Point-1mm-round")
-		(at 229.87 200.66 90)
-		(unit 1)
-		(exclude_from_sim no)
-		(in_bom yes)
-		(on_board yes)
-		(dnp no)
-		(property "Reference" "TP42"
-			(at 236.22 200.66 90)
-			(effects
-				(font
-					(size 1.27 1.27)
-				)
-				(justify left)
-			)
-		)
-		(property "Value" "Test-Point"
-			(at 227.33 200.66 0)
-			(effects
-				(font
-					(size 1.27 1.27)
-				)
-				(hide yes)
-			)
-		)
-		(property "Footprint" "oresat-misc:TestPoint_Pad_D1.0mm"
-			(at 219.71 200.66 0)
-			(effects
-				(font
-					(size 1.27 1.27)
-				)
-				(hide yes)
-			)
-		)
-		(property "Datasheet" ""
-			(at 229.87 200.66 0)
-			(effects
-				(font
-					(size 1.27 1.27)
-				)
-				(hide yes)
-			)
-		)
-		(property "Description" ""
-			(at 229.87 200.66 0)
-			(effects
-				(font
-					(size 1.27 1.27)
-				)
-				(hide yes)
-			)
-		)
-		(property "Part Page" ""
-			(at 229.87 200.66 0)
-			(effects
-				(font
-					(size 1.27 1.27)
-				)
-				(hide yes)
-			)
-		)
-		(property "Price" ""
-			(at 229.87 200.66 0)
-			(effects
-				(font
-					(size 1.27 1.27)
-				)
-				(hide yes)
-			)
-		)
-		(property "Total Price" ""
-			(at 229.87 200.66 0)
-			(effects
-				(font
-					(size 1.27 1.27)
-				)
-				(hide yes)
-			)
-		)
-		(pin "1"
-		)
-		(instances
-			(project "oresat-c3"
-				(path "/65d12cdd-c326-4033-9053-c59fa4e0b25e/f3d147ad-4cea-4d77-ae60-95882b03454e"
-					(reference "TP42")
-					(unit 1)
-				)

Commit message: - Grounded FRAM Write protect permanently - Erased old CAN transceivers for unused bus - Fixed CAN termination resistor value to 120 ohm - Redid Clock skew for CAN lines - Removed UART0 from CSKB - Added second I2C buffer for I2C2 bus - Re-routed and placed all I2C bus components 	- Still need to route I2C sys disable, will do later after GPIOs since its lower prio - Added ADCS Enable pin components and routed everything
Parts:
- removed C18: 100n, Capacitor_SMD:C_0603_1608Metric, symbol Device:C_Small
- removed R1: 120k, Resistor_SMD:R_0603_1608Metric, symbol Device:R_Small_US
- removed TP23, TP24, TP26, TP27: Test-Point, oresat-misc:TestPoint_Pad_D1.0mm, symbol oresat-misc:Test-Point-1mm-round
- removed U8: TCAN330, Package_TO_SOT_SMD:SOT-23-8, symbol Interface_CAN_LIN:TCAN330
- added Q2: SI7106DN-T1-GE3, SIS862DNT1GE3, symbol SI7106DN-T1-GE3:SI7106DN-T1-GE3
- added R6: 20k, Resistor_SMD:R_0603_1608Metric, symbol Device:R_Small_US
Connections:
- net ADCS_ENABLE_CONTROL: now also Q2.10 (D_6), Q2.11 (D_7), Q2.5 (D_1), Q2.6 (D_2), Q2.7 (D_3), Q2.8 (D_4), Q2.9 (D_5); no longer TP46.1, U1.P7 (GPMC_AD15)
- net GND: now also Q2.1 (S_1), Q2.2 (S_2), Q2.3 (S_3), R6.2
- net CAN1_RXD renamed UART1_TX
- net CAN1_TXD renamed UART1_RX
- new net: Q2.4 (G), R6.1, TP46.1, U1.P7 (GPMC_AD15)
Other:
- note removed: "CAN Transceiver"
- note removed: "CAN1 RX = B11 = UART1_TXD CAN1 TX = A11 = UART1_RXD"
- note removed: "To main card connector"

Commit message: - Labelled GPIOs and UART lines to processor pins - Routed UART lines - Routed GPIO Lines - Refilled zones - Added via fencing back in - Board should be ready to be reviewed now
Parts:
- removed TP68: Test-Point, oresat-misc:TestPoint_Pad_D1.0mm, symbol oresat-misc:Test-Point-1mm-round
Connections:
- net USR1: no longer R42.1
- net GPIO8: now reaches TP38.1, U1.R12 (GPMC_A1)
- net UART2_RX: now reaches U1.A13 (SPI0_SCLK)
- net UART2_TX: now reaches U1.B13 (SPI0_D0)
- net GPIO3: now reaches U1.B3 (MCASP0_FSR)
- net GPIO1: now reaches U1.C4 (MCASP0_AHCLKX)
- net GPIO2: now reaches U1.M1 (GPMC_ADVN_ALE)
- net GPIO10: now reaches U1.N14 (GPMC_BEN1)
- net GPIO5: now reaches TP65.1, U1.N2 (GPMC_WEN)
- net GPIO6: now reaches TP64.1, U1.N3 (GPMC_BEN0_CLE)
- net UART3_RX: now reaches U1.P15 (GPMC_WAIT0)
- net UART3_TX: now reaches U1.R16 (GPMC_WPN)
- net GPIO9: now reaches U1.T12 (GPMC_A0)
- net GPIO7: now reaches U1.T6 (GPMC_AD14)
- net ADCS_UART_GNSS renamed GPIO4
- no-connect marks 24 -> 16

Commit message: OBC review session changes
Connections:
- net USR1: now also R42.1
Changed lines of the file:
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@@
-	(wire
-		(pts
-			(xy 269.24 104.14) (xy 260.35 104.14)
-		)
-		(stroke
-			(width 0)
-			(type default)
-		)
-	)
 	(wire
 		(pts
@@
 		)
 		(stroke
+			(width 0)
+			(type default)
+		)
+	)
+	(wire
+		(pts
+			(xy 269.24 104.14) (xy 278.13 104.14)
+		)
+		(stroke

Commit message: Added 2 new GPIO pins
Connections:
- net GPIO8: now also TP47.1, U1.P3 (GPMC_CSN0); no longer TP38.1, U1.R12 (GPMC_A1)
- net GPIO9: now also TP66.1, U1.N1 (GPMC_OEN_REN); no longer U1.T12 (GPMC_A0)
- new net GPIO11: U1.T12 (GPMC_A0)
- new net GPIO12: TP38.1, U1.R12 (GPMC_A1)
Changed lines of the file:
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@@
 	)
 	(junction
+		(at 229.87 215.9)
+		(diameter 0)
+		(color 0 0 0 0)
+	)
+	(junction
 		(at 276.86 243.84)
 		(diameter 0)
@@
 	)
 	(junction
+		(at 229.87 149.86)
+		(diameter 0)
+		(color 0 0 0 0)
+	)
+	(junction
 		(at 300.99 111.76)
 		(diameter 0)
@@
 	(wire
 		(pts
+			(xy 229.87 149.86) (xy 238.76 149.86)
+		)
+		(stroke
+			(width 0)
+			(type default)
+		)
+	)
+	(wire
+		(pts
 			(xy 241.3 152.4) (xy 241.3 157.48)
 		)
@@
 	(wire
 		(pts
+			(xy 229.87 215.9) (xy 237.49 215.9)
+		)
+		(stroke
+			(width 0)
+			(type default)
+		)
+	)
+	(wire
+		(pts
 			(xy 114.3 152.4) (xy 162.56 152.4)
 		)
@@
 		)
 	)
+	(global_label "GPIO9"
+		(shape output)
+		(at 237.49 215.9 0)
+		(fields_autoplaced yes)
+		(effects
+			(font
+				(size 1.27 1.27)
+			)
+			(justify left)
+		)
+		(property "Intersheetrefs" "${INTERSHEET_REFS}"
+			(at 246.16 215.9 0)
+			(effects
+				(font
+					(size 1.27 1.27)
+				)
+				(justify left)
+			)
+		)
+	)
 	(global_label "MRAM_SPI_CLK"
 		(shape output)
@@
 		)
 	)
-	(global_label "GPIO9"
+	(global_label "GPIO11"
 		(shape output)
 		(at 240.03 106.68 0)
@@
 		)
 		(property "Intersheetrefs" "${INTERSHEET_REFS}"
-			(at 248.7 106.68 0)
+			(at 249.9095 106.68 0)
+			(effects
+				(font
+					(size 1.27 1.27)
+				)
+				(justify left)
+			)
+		)
+	)
+	(global_label "GPIO8"
+		(shape output)
+		(at 238.76 149.86 0)
+		(fields_autoplaced yes)
+		(effects
+			(font
+				(size 1.27 1.27)
+			)
+			(justify left)
+		)
+		(property "Intersheetrefs" "${INTERSHEET_REFS}"
+			(at 247.43 149.86 0)
 			(effects
 				(font
@@
 		)
 	)
-	(global_label "GPIO8"
+	(global_label "GPIO12"
 		(shape output)
 		(at 240.03 109.22 0)
@@
 		)
 		(property "Intersheetrefs" "${INTERSHEET_REFS}"
-			(at 248.7 109.22 0)
+			(at 249.9095 109.22 0)
 			(effects
 				(font

Commit message: - Configured pin headers for UART5 and boot pins to be horizontal - Removed some TPs for GPIO pins
Parts:
- removed TP38, TP47, TP64, TP65, TP66: Test-Point, oresat-misc:TestPoint_Pad_D1.0mm, symbol oresat-misc:Test-Point-1mm-round

Commit message: Moved connectors around, still needs to be routed
Parts:
- added J3: Conn_01x03, symbol Connector_Generic:Conn_01x03
Connections:
- net GND: now also J3.1 (Pin_1)
- net UART0_RX: now also J3.3 (Pin_3)
- net UART0_TX: now also J3.2 (Pin_2)
Other:
- note added: "UART0 SERIAL CONNECTOR"
Changed lines of the file:
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@@
 		)
 	)
+	(text "UART0 SERIAL CONNECTOR"
+		(exclude_from_sim no)
+		(at 145.542 81.026 0)
+		(effects
+			(font
+				(size 1.27 1.27)
+			)
+			(justify left bottom)
+		)
+	)
 	(text "SPI INTERFACE\nFOR KUBOS"
 		(exclude_from_sim no)
@@
 	)
 	(junction
+		(at 153.67 104.14)
+		(diameter 0)
+		(color 0 0 0 0)
+	)
+	(junction
 		(at 276.86 236.22)
 		(diameter 0)
@@
 	)
 	(junction
+		(at 151.13 101.6)
+		(diameter 0)
+		(color 0 0 0 0)
+	)
+	(junction
 		(at 67.31 106.68)
 		(diameter 0)
@@
 	(wire
 		(pts
+			(xy 153.67 104.14) (xy 153.67 88.9)
+		)
+		(stroke
+			(width 0)
+			(type default)
+		)
+	)
+	(wire
+		(pts
 			(xy 327.66 152.4) (xy 327.66 154.94)
 		)
@@
 	(wire
 		(pts
+			(xy 153.67 88.9) (xy 156.21 88.9)
+		)
+		(stroke
+			(width 0)
+			(type default)
+		)
+	)
+	(wire
+		(pts
 			(xy 265.43 208.28) (xy 250.19 208.28)
 		)
@@
 	(wire
 		(pts
+			(xy 146.05 104.14) (xy 153.67 104.14)
+		)
+		(stroke
+			(width 0)
+			(type default)
+		)
+	)
+	(wire
+		(pts
 			(xy 287.02 180.34) (xy 317.5 180.34)
 		)
@@
 	(wire
 		(pts
-			(xy 146.05 104.14) (xy 162.56 104.14)
-		)
-		(stroke
-			(width 0)
-			(type default)
-		)
-	)
-	(wire
-		(pts
 			(xy 274.32 193.04) (xy 274.32 198.12)
 		)
@@
 	(wire
 		(pts
+			(xy 151.13 101.6) (xy 162.56 101.6)
+		)
+		(stroke
+			(width 0)
+			(type default)
+		)
+	)
+	(wire
+		(pts
 			(xy 274.32 233.68) (xy 276.86 233.68)
 		)
@@
 	(wire
 		(pts
+			(xy 153.67 104.14) (xy 162.56 104.14)
+		)
+		(stroke
+			(width 0)
+			(type default)
+		)
+	)
+	(wire
+		(pts
 			(xy 274.32 124.46) (xy 274.32 119.38)
 		)
@@
 	(wire
 		(pts
+			(xy 151.13 86.36) (xy 156.21 86.36)
+		)
+		(stroke
+			(width 0)
+			(type default)
+		)
+	)
+	(wire
+		(pts
 			(xy 125.73 180.34) (xy 125.73 200.66)
 		)
@@
 	(wire
 		(pts
+			(xy 151.13 86.36) (xy 151.13 101.6)
+		)
+		(stroke
+			(width 0)
+			(type default)
+		)
+	)
+	(wire
+		(pts
 			(xy 162.56 139.7) (xy 154.94 139.7)
 		)
@@
 	(wire
 		(pts
+			(xy 146.05 83.82) (xy 146.05 86.36)
+		)
+		(stroke
+			(width 0)
+			(type default)
+		)
+	)
+	(wire
+		(pts
 			(xy 300.99 129.54) (xy 300.99 127)
 		)
@@
 	(wire
 		(pts
+			(xy 146.05 83.82) (xy 156.21 83.82)
+		)
+		(stroke
+			(width 0)
+			(type default)
+		)
+	)
+	(wire
+		(pts
 			(xy 223.52 203.2) (xy 229.87 203.2)
 		)
@@
 	(wire
 		(pts
-			(xy 146.05 101.6) (xy 162.56 101.6)
+			(xy 146.05 101.6) (xy 151.13 101.6)
 		)
 		(stroke
@@
 	)
 	(symbol
+		(lib_id "power:GND")
+		(at 146.05 86.36 0)
+		(unit 1)
+		(exclude_from_sim no)
+		(in_bom yes)
+		(on_board yes)
+		(dnp no)
+		(property "Reference" "#PWR023"
+			(at 146.05 92.71 0)
+			(effects
+				(font
+					(size 1.27 1.27)
+				)
+				(hide yes)
+			)
+		)
+		(property "Value" "GND"
+			(at 146.05 90.17 0)
+			(effects
+				(font
+					(size 1.27 1.27)
+				)
+			)
+		)
+		(property "Footprint" ""
+			(at 146.05 86.36 0)
+			(effects
+				(font
+					(size 1.27 1.27)
+				)
+				(hide yes)
+			)
+		)
+		(property "Datasheet" ""
+			(at 146.05 86.36 0)
+			(effects
+				(font
+					(size 1.27 1.27)
+				)
+				(hide yes)
+			)
+		)
+		(property "Description" ""
+			(at 146.05 86.36 0)
+			(effects
+				(font
+					(size 1.27 1.27)
+				)
+				(hide yes)
+			)
+		)
+		(pin "1"
+		)
+		(instances
+			(project "oresat-c3"
+				(path "/65d12cdd-c326-4033-9053-c59fa4e0b25e/f3d147ad-4cea-4d77-ae60-95882b03454e"
+					(reference "#PWR023")
+					(unit 1)
+				)
+			)
+		)
+	)
+	(symbol
 		(lib_id "SI7106DN-T1-GE3:SI7106DN-T1-GE3")
 		(at 248.92 233.68 0)
@@
 					(unit 1)
 				)
+			)
+		)
+	)
+	(symbol
+		(lib_id "Connector_Generic:Conn_01x03")
+		(at 161.29 86.36 0)
+		(unit 1)
+		(exclude_from_sim no)
+		(in_bom yes)
+		(on_board yes)
+		(dnp no)
+		(fields_autoplaced yes)
+		(property "Reference" "J3"
+			(at 163.83 85.0899 0)
+			(effects
+				(font
+					(size 1.27 1.27)
+				)
+				(justify left)
+			)
+		)
+		(property "Value" "Conn_01x03"
+			(at 163.83 87.6299 0)
+			(effects
+				(font
+					(size 1.27 1.27)
+				)
+				(justify left)
+			)
+		)
+		(property "Footprint" ""
+			(at 161.29 86.36 0)
+			(effects
+				(font
+					(size 1.27 1.27)
+				)
+				(hide yes)
+			)
+		)
+		(property "Datasheet" "~"
+			(at 161.29 86.36 0)
+			(effects
+				(font
+					(size 1.27 1.27)
+				)
+				(hide yes)
+			)
+		)
+		(property "Description" "Generic connector, single row, 01x03, script generated (kicad-library-utils/schlib/autogen/connector/)"
+			(at 161.29 86.36 0)
+			(effects
+				(font
+					(size 1.27 1.27)
+				)
+				(hide yes)
+			)
+		)
+		(pin "1"
+		)
+		(pin "2"
+		)
+		(pin "3"
+		)
+		(instances
+			(project ""
+				(path "/65d12cdd-c326-4033-9053-c59fa4e0b25e/f3d147ad-4cea-4d77-ae60-95882b03454e"
+					(reference "J3")
+					(unit 1)
+				)
