File: kicad/oresat-c3-sch-osd3358-sd-emmc.kicad_sch (KiCad schematic)
At the start: 34 parts, among them J3 Conn_01x03, J5 DM3BT-DSF-PEJS, Q2 SI7106DN-T1-GE3, U1 OSD3358-512M-BSM, U9 EMMC+RESET+5.1-COMPATIBLE-BA

Commit message: - Routed New boot pin properly, added test points to old spots as backups - Filled some floating ground planes with vias near I2C2 Buffer - Routed UART0 to new pins properly - Fixed SD card connector, it somehow got moved - Fixed som DRC issues, still need to go through a lot - Labelled CSKB, added x to anything unconnected
Other:
- moved on the sheet: J3
Changed lines of the file:
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@@
 	)
 	(junction
-		(at 153.67 104.14)
-		(diameter 0)
-		(color 0 0 0 0)
-	)
-	(junction
 		(at 276.86 236.22)
 		(diameter 0)
@@
 	)
 	(junction
-		(at 151.13 101.6)
-		(diameter 0)
-		(color 0 0 0 0)
-	)
-	(junction
 		(at 67.31 106.68)
 		(diameter 0)
@@
 	(wire
 		(pts
-			(xy 153.67 104.14) (xy 153.67 88.9)
-		)
-		(stroke
-			(width 0)
-			(type default)
-		)
-	)
-	(wire
-		(pts
 			(xy 327.66 152.4) (xy 327.66 154.94)
 		)
@@
 	(wire
 		(pts
+			(xy 157.48 86.36) (xy 151.13 86.36)
+		)
+		(stroke
+			(width 0)
+			(type default)
+		)
+	)
+	(wire
+		(pts
 			(xy 276.86 233.68) (xy 276.86 236.22)
 		)
@@
 	(wire
 		(pts
-			(xy 153.67 88.9) (xy 156.21 88.9)
-		)
-		(stroke
-			(width 0)
-			(type default)
-		)
-	)
-	(wire
-		(pts
 			(xy 265.43 208.28) (xy 250.19 208.28)
 		)
@@
 	(wire
 		(pts
-			(xy 146.05 104.14) (xy 153.67 104.14)
-		)
-		(stroke
-			(width 0)
-			(type default)
-		)
-	)
-	(wire
-		(pts
 			(xy 287.02 180.34) (xy 317.5 180.34)
 		)
@@
 	(wire
 		(pts
-			(xy 151.13 101.6) (xy 162.56 101.6)
+			(xy 274.32 233.68) (xy 276.86 233.68)
 		)
 		(stroke
@@
 	(wire
 		(pts
-			(xy 274.32 233.68) (xy 276.86 233.68)
+			(xy 109.22 154.94) (xy 162.56 154.94)
 		)
 		(stroke
@@
 	(wire
 		(pts
-			(xy 109.22 154.94) (xy 162.56 154.94)
+			(xy 242.57 241.3) (xy 248.92 241.3)
 		)
 		(stroke
@@
 	(wire
 		(pts
-			(xy 242.57 241.3) (xy 248.92 241.3)
+			(xy 88.9 102.87) (xy 88.9 104.14)
 		)
 		(stroke
@@
 	(wire
 		(pts
-			(xy 88.9 102.87) (xy 88.9 104.14)
+			(xy 151.13 88.9) (xy 157.48 88.9)
 		)
 		(stroke
@@
 	(wire
 		(pts
-			(xy 153.67 104.14) (xy 162.56 104.14)
-		)
-		(stroke
-			(width 0)
-			(type default)
-		)
-	)
-	(wire
-		(pts
 			(xy 274.32 124.46) (xy 274.32 119.38)
 		)
@@
 	(wire
 		(pts
-			(xy 151.13 86.36) (xy 156.21 86.36)
-		)
-		(stroke
-			(width 0)
-			(type default)
-		)
-	)
-	(wire
-		(pts
 			(xy 125.73 180.34) (xy 125.73 200.66)
 		)
@@
 	(wire
 		(pts
-			(xy 151.13 86.36) (xy 151.13 101.6)
-		)
-		(stroke
-			(width 0)
-			(type default)
-		)
-	)
-	(wire
-		(pts
 			(xy 162.56 139.7) (xy 154.94 139.7)
 		)
@@
 	(wire
 		(pts
-			(xy 146.05 83.82) (xy 146.05 86.36)
+			(xy 132.08 83.82) (xy 132.08 86.36)
 		)
 		(stroke
@@
 	(wire
 		(pts
-			(xy 146.05 83.82) (xy 156.21 83.82)
+			(xy 132.08 83.82) (xy 157.48 83.82)
 		)
 		(stroke
@@
 	(wire
 		(pts
+			(xy 146.05 101.6) (xy 162.56 101.6)
+		)
+		(stroke
+			(width 0)
+			(type default)
+		)
+	)
+	(wire
+		(pts
 			(xy 345.44 166.37) (xy 345.44 167.64)
 		)
@@
 	(wire
 		(pts
-			(xy 146.05 101.6) (xy 151.13 101.6)
+			(xy 330.2 154.94) (xy 330.2 157.48)
 		)
 		(stroke
@@
 	(wire
 		(pts
-			(xy 330.2 154.94) (xy 330.2 157.48)
+			(xy 314.96 185.42) (xy 317.5 185.42)
 		)
 		(stroke
@@
 	(wire
 		(pts
-			(xy 314.96 185.42) (xy 317.5 185.42)
+			(xy 223.52 111.76) (xy 229.87 111.76)
 		)
 		(stroke
@@
 	(wire
 		(pts
-			(xy 223.52 111.76) (xy 229.87 111.76)
+			(xy 146.05 104.14) (xy 162.56 104.14)
 		)
 		(stroke
@@
 		)
 	)
+	(global_label "UART0_RX"
+		(shape input)
+		(at 151.13 88.9 180)
+		(fields_autoplaced yes)
+		(effects
+			(font
+				(size 1.27 1.27)
+			)
+			(justify right)
+		)
+		(property "Intersheetrefs" "${INTERSHEET_REFS}"
+			(at 138.9109 88.9 0)
+			(effects
+				(font
+					(size 1.27 1.27)
+				)
+				(justify right)
+			)
+		)
+	)
 	(global_label "UART3_RX"
 		(shape input)
@@
 		)
 	)
+	(global_label "UART0_TX"
+		(shape input)
+		(at 151.13 86.36 180)
+		(fields_autoplaced yes)
+		(effects
+			(font
+				(size 1.27 1.27)
+			)
+			(justify right)
+		)
+		(property "Intersheetrefs" "${INTERSHEET_REFS}"
+			(at 139.2133 86.36 0)
+			(effects
+				(font
+					(size 1.27 1.27)
+				)
+				(justify right)
+			)
+		)
+	)
 	(global_label "MRAM_SPI_MISO"
 		(shape input)
@@
 	(symbol
 		(lib_id "power:GND")
-		(at 146.05 86.36 0)
+		(at 132.08 86.36 0)
 		(unit 1)
 		(exclude_from_sim no)
@@
 		(dnp no)
 		(property "Reference" "#PWR023"
-			(at 146.05 92.71 0)
+			(at 132.08 92.71 0)
 			(effects
 				(font
@@
 		)
 		(property "Value" "GND"
-			(at 146.05 90.17 0)
+			(at 132.08 90.17 0)
 			(effects
 				(font
@@
 		)
 		(property "Footprint" ""
-			(at 146.05 86.36 0)
+			(at 132.08 86.36 0)
 			(effects
 				(font
@@
 		)
 		(property "Datasheet" ""
-			(at 146.05 86.36 0)
+			(at 132.08 86.36 0)
 			(effects
 				(font
@@
 		)
 		(property "Description" ""
-			(at 146.05 86.36 0)
+			(at 132.08 86.36 0)
 			(effects
 				(font
@@
 	(symbol
 		(lib_id "Connector_Generic:Conn_01x03")
-		(at 161.29 86.36 0)
+		(at 162.56 86.36 0)
 		(unit 1)
 		(exclude_from_sim no)
@@
 		(fields_autoplaced yes)
 		(property "Reference" "J3"
-			(at 163.83 85.0899 0)
+			(at 165.1 85.0899 0)
 			(effects
 				(font
@@
 		)
 		(property "Value" "Conn_01x03"
-			(at 163.83 87.6299 0)
+			(at 165.1 87.6299 0)
 			(effects
 				(font
@@
 		)
 		(property "Footprint" ""
-			(at 161.29 86.36 0)
+			(at 162.56 86.36 0)
 			(effects
 				(font
@@
 		)
 		(property "Datasheet" "~"
-			(at 161.29 86.36 0)
+			(at 162.56 86.36 0)
 			(effects
 				(font
@@
 		)
 		(property "Description" "Generic connector, single row, 01x03, script generated (kicad-library-utils/schlib/autogen/connector/)"
-			(at 161.29 86.36 0)
+			(at 162.56 86.36 0)
 			(effects
 				(font

Commit message: added automotive grade capacitors to the BOM
Parts:
- C16, C25: Description_1 (none) -> CAP CER 10UF 16V X5R 0805; Manufacturer_Name (none) -> Murata Electronics; Manufacturer_Part_Number (none) -> GRT21BR61C106KE01L
- C17: Description_1 (none) -> CAP CER 0.1UF 16V X7R 0603; Manufacturer_Name (none) -> Murata Electronics; Manufacturer_Part_Number (none) -> GCJ188R71C104KA01D
- C19, C20, C21, C22, C23, C24: Description_1 (none) -> CAP CER 1UF 16V X7R 0603; Manufacturer_Name (none) -> Murata Electronics; Manufacturer_Part_Number (none) -> GCM188R71C105KA64D
- J5: Description_1 (none) -> CONN MICRO SD CARD R/A SMD; Manufacturer_Name (none) -> Hirose Electric Co Ltd; Manufacturer_Part_Number (none) -> DM3BT-DSF-PEJS
- Q2: Description_1 (none) -> MOSFET N-CH 20V 12.5A PPAK1212-8; Manufacturer_Name Vishay -> Vishay Siliconix
- R104, R118, R26, R27, R42, R43, R44, R45, R90: Description_1 (none) -> RES 10K OHM 1% 1/8W 0603; Manufacturer_Name (none) -> Stackpole Electronics Inc; Manufacturer_Part_Number (none) -> RNCP0603FTD10K0
- R69, R70, R71: Description_1 (none) -> RES ARRAY 8 RES 47K OHM 2512; Manufacturer_Name (none) -> Panasonic Electronic Components; Manufacturer_Part_Number (none) -> EXB-A10P473J

Commit message: added automotive grade resistors to BOM
Parts:
- J3: footprint (none) -> Connector_PinHeader_2.54mm:PinHeader_1x03_P2.54mm_Horizontal; Description_1 (none) -> CONN HEADER R/A 3POS 2.54MM; Manufacturer_Name (none) -> Samtec Inc.; Manufacturer_Part_Number (none) -> TSW-103-25-F-S-RA
- R104, R118, R26, R27, R42, R43, R44, R45, R90: Description_1 RES 10K OHM 1% 1/8W 0603 -> RES 0603 10 KOHM 1% 0.125W AUTO; Manufacturer_Part_Number RNCP0603FTD10K0 -> RMCA0603FT10K0-HP
- R6: Description_1 (none) -> RES 0603 20 KOHM 1% 0.125W AUTO; Manufacturer_Name (none) -> Stackpole Electronics Inc; Manufacturer_Part_Number (none) -> RMCA0603FT20K0-HP
Changed lines of the file:
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@@
 			)
 		)
-		(property "Description_1" "RES 10K OHM 1% 1/8W 0603"
+		(property "Description_1" "RES 0603 10 KOHM 1% 0.125W AUTO"
 			(at 267.97 213.36 90)
 			(effects
@@
 			)
 		)
-		(property "Manufacturer_Part_Number" "RNCP0603FTD10K0"
+		(property "Manufacturer_Part_Number" "RMCA0603FT10K0-HP"
 			(at 267.97 213.36 90)
 			(effects
@@
 			)
 		)
-		(property "Description_1" "RES 10K OHM 1% 1/8W 0603"
+		(property "Description_1" "RES 0603 10 KOHM 1% 0.125W AUTO"
 			(at 280.67 119.38 90)
 			(effects
@@
 			)
 		)
-		(property "Manufacturer_Part_Number" "RNCP0603FTD10K0"
+		(property "Manufacturer_Part_Number" "RMCA0603FT10K0-HP"
 			(at 280.67 119.38 90)
 			(effects
@@
 			)
 		)
-		(property "Description_1" "RES 10K OHM 1% 1/8W 0603"
+		(property "Description_1" "RES 0603 10 KOHM 1% 0.125W AUTO"
 			(at 280.67 104.14 90)
 			(effects
@@
 			)
 		)
-		(property "Manufacturer_Part_Number" "RNCP0603FTD10K0"
+		(property "Manufacturer_Part_Number" "RMCA0603FT10K0-HP"
 			(at 280.67 104.14 90)
 			(effects
@@
 			)
 		)
-		(property "Description_1" "RES 10K OHM 1% 1/8W 0603"
+		(property "Description_1" "RES 0603 10 KOHM 1% 0.125W AUTO"
 			(at 267.97 198.12 90)
 			(effects
@@
 			)
 		)
-		(property "Manufacturer_Part_Number" "RNCP0603FTD10K0"
+		(property "Manufacturer_Part_Number" "RMCA0603FT10K0-HP"
 			(at 267.97 198.12 90)
 			(effects
@@
 			)
 		)
-		(property "Description_1" ""
+		(property "Description_1" "RES 0603 20 KOHM 1% 0.125W AUTO"
+			(at 242.57 246.38 90)
+			(effects
+				(font
+					(size 1.27 1.27)
+				)
+				(hide yes)
+			)
+		)
+		(property "Manufacturer_Name" "Stackpole Electronics Inc"
+			(at 242.57 246.38 90)
+			(effects
+				(font
+					(size 1.27 1.27)
+				)
+				(hide yes)
+			)
+		)
+		(property "Manufacturer_Part_Number" "RMCA0603FT20K0-HP"
 			(at 242.57 246.38 90)
 			(effects
@@
 			)
 		)
-		(property "Description_1" "RES 10K OHM 1% 1/8W 0603"
+		(property "Description_1" "RES 0603 10 KOHM 1% 0.125W AUTO"
 			(at 267.97 208.28 90)
 			(effects
@@
 			)
 		)
-		(property "Manufacturer_Part_Number" "RNCP0603FTD10K0"
+		(property "Manufacturer_Part_Number" "RMCA0603FT10K0-HP"
 			(at 267.97 208.28 90)
 			(effects
@@
 			)
 		)
-		(property "Description_1" "RES 10K OHM 1% 1/8W 0603"
+		(property "Description_1" "RES 0603 10 KOHM 1% 0.125W AUTO"
 			(at 280.67 111.76 90)
 			(effects
@@
 			)
 		)
-		(property "Manufacturer_Part_Number" "RNCP0603FTD10K0"
+		(property "Manufacturer_Part_Number" "RMCA0603FT10K0-HP"
 			(at 280.67 111.76 90)
 			(effects
@@
 			)
 		)
-		(property "Footprint" ""
+		(property "Footprint" "Connector_PinHeader_2.54mm:PinHeader_1x03_P2.54mm_Horizontal"
 			(at 162.56 86.36 0)
 			(effects
@@
 			)
 		)
+		(property "Description_1" "CONN HEADER R/A 3POS 2.54MM"
+			(at 162.56 86.36 0)
+			(effects
+				(font
+					(size 1.27 1.27)
+				)
+				(hide yes)
+			)
+		)
+		(property "Manufacturer_Name" "Samtec Inc."
+			(at 162.56 86.36 0)
+			(effects
+				(font
+					(size 1.27 1.27)
+				)
+				(hide yes)
+			)
+		)
+		(property "Manufacturer_Part_Number" "TSW-103-25-F-S-RA"
+			(at 162.56 86.36 0)
+			(effects
+				(font
+					(size 1.27 1.27)
+				)
+				(hide yes)
+			)
+		)
 		(pin "1"
 		)
@@
 			)
 		)
-		(property "Description_1" "RES 10K OHM 1% 1/8W 0603"
+		(property "Description_1" "RES 0603 10 KOHM 1% 0.125W AUTO"
 			(at 267.97 193.04 90)
 			(effects
@@
 			)
 		)
-		(property "Manufacturer_Part_Number" "RNCP0603FTD10K0"
+		(property "Manufacturer_Part_Number" "RMCA0603FT10K0-HP"
 			(at 267.97 193.04 90)
 			(effects
@@
 			)
 		)
-		(property "Description_1" "RES 10K OHM 1% 1/8W 0603"
+		(property "Description_1" "RES 0603 10 KOHM 1% 0.125W AUTO"
 			(at 280.67 127 90)
 			(effects
@@
 			)
 		)
-		(property "Manufacturer_Part_Number" "RNCP0603FTD10K0"
+		(property "Manufacturer_Part_Number" "RMCA0603FT10K0-HP"
 			(at 280.67 127 90)
 			(effects
@@
 			)
 		)
-		(property "Description_1" "RES 10K OHM 1% 1/8W 0603"
+		(property "Description_1" "RES 0603 10 KOHM 1% 0.125W AUTO"
 			(at 267.97 203.2 90)
 			(effects
@@
 			)
 		)
-		(property "Manufacturer_Part_Number" "RNCP0603FTD10K0"
+		(property "Manufacturer_Part_Number" "RMCA0603FT10K0-HP"
 			(at 267.97 203.2 90)
 			(effects

Commit message: modified BOM to match PCBWay format
Parts:
- TP39, TP46, TP48: now not fitted
Changed lines of the file:
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@@
 		(in_bom yes)
 		(on_board yes)
-		(dnp no)
+		(dnp yes)
 		(property "Reference" "TP46"
 			(at 236.22 203.2 90)
@@
 		(in_bom yes)
 		(on_board yes)
-		(dnp no)
+		(dnp yes)
 		(property "Reference" "TP48"
 			(at 236.22 157.48 0)
@@
 		(in_bom yes)
 		(on_board yes)
-		(dnp no)
+		(dnp yes)
 		(property "Reference" "TP39"
 			(at 236.22 111.76 0)

Commit message: finished putting together BOM, needs review
Parts:
- C16, C25: Description / Value (none) -> CAP CER 10UF 16V X5R 0805; Description_1 CAP CER 10UF 16V X5R 0805 -> (none)
- C17: Description / Value (none) -> CAP CER 0.1UF 16V X7R 0603; Description_1 CAP CER 0.1UF 16V X7R 0603 -> (none)
- C19, C20, C21, C22, C23, C24: Description / Value (none) -> CAP CER 1UF 16V X7R 0603; Description_1 CAP CER 1UF 16V X7R 0603 -> (none)
- J3: Description / Value (none) -> CONN HEADER R/A 3POS 2.54MM; Description_1 CONN HEADER R/A 3POS 2.54MM -> (none)
- J5: Description / Value (none) -> CONN MICRO SD CARD R/A SMD; Description_1 CONN MICRO SD CARD R/A SMD -> (none)
- Q2: Description / Value (none) -> MOSFET N-CH 20V 12.5A PPAK1212-8; Description_1 MOSFET N-CH 20V 12.5A PPAK1212-8 -> (none)
- R104, R118, R26, R27, R42, R43, R44, R45, R90: Description / Value (none) -> RES 0603 10 KOHM 1% 0.125W AUTO; Description_1 RES 0603 10 KOHM 1% 0.125W AUTO -> (none)
- R6: Description / Value (none) -> RES 0603 20 KOHM 1% 0.125W AUTO; Description_1 RES 0603 20 KOHM 1% 0.125W AUTO -> (none)
- R69, R70, R71: Description / Value (none) -> RES ARRAY 8 RES 47K OHM 2512; Description_1 RES ARRAY 8 RES 47K OHM 2512 -> (none)
- U1: value OSD3358-512M-BSM -> OSD3358-512M-ISM; Description / Value (none) -> IC MODULE CORTEX-A8 1GHZ 512MB; Manufacturer_Name (none) -> Octavo Systems LLC; Manufacturer_Part_Number (none) -> OSD3358-512M-ISM
- U9: Description / Value (none) -> IC FLASH 64GBIT EMMC 100LFBGA; Manufacturer_Name (none) -> ISSI, Integrated Silicon Solution Inc; Manufacturer_Part_Number (none) -> IS21ES08GA-JQLI-TR

Commit message: - Fixed part number for FRAM, CAN transceiver, emmc, and BJT - Change LED and connected resistors to DNP - Verified remainder of components
Parts:
- D4, D5, D6, D7, R42, R43, R44, R45: now not fitted
- U9: Manufacturer_Part_Number IS21ES08GA-JQLI-TR -> IS21ES08GA-JCLI-TR
Changed lines of the file:
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@@
 		(in_bom yes)
 		(on_board yes)
-		(dnp no)
+		(dnp yes)
 		(property "Reference" "D4"
 			(at 290.83 101.6 0)
@@
 		(in_bom yes)
 		(on_board yes)
-		(dnp no)
+		(dnp yes)
 		(property "Reference" "R44"
 			(at 278.13 116.84 90)
@@
 			)
 		)
-		(property "Manufacturer_Part_Number" "IS21ES08GA-JQLI-TR"
+		(property "Manufacturer_Part_Number" "IS21ES08GA-JCLI-TR"
 			(at 330.2 175.26 0)
 			(effects
@@
 		(in_bom yes)
 		(on_board yes)
-		(dnp no)
+		(dnp yes)
 		(property "Reference" "R42"
 			(at 278.13 101.6 90)
@@
 		(in_bom yes)
 		(on_board yes)
-		(dnp no)
+		(dnp yes)
 		(property "Reference" "D5"
 			(at 290.83 109.22 0)
@@
 		(in_bom yes)
 		(on_board yes)
-		(dnp no)
+		(dnp yes)
 		(property "Reference" "R43"
 			(at 278.13 109.22 90)
@@
 		(in_bom yes)
 		(on_board yes)
-		(dnp no)
+		(dnp yes)
 		(property "Reference" "D6"
 			(at 290.83 116.84 0)
@@
 		(in_bom yes)
 		(on_board yes)
-		(dnp no)
+		(dnp yes)
 		(property "Reference" "D7"
 			(at 290.83 124.46 0)
@@
 		(in_bom yes)
 		(on_board yes)
-		(dnp no)
+		(dnp yes)
 		(property "Reference" "R45"
 			(at 278.13 124.46 90)

Commit message: - removed C5 pin connected to GPIO4/A3 - Redid teardrops - fixed one DRC issue with a via
Connections:
- net GPIO4: no longer U1.C5 (ECAP0_IN_PWM0_OUT)
- no-connect marks 16 -> 17
Changed lines of the file:
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@@
-	)
-	(junction
-		(at 125.73 200.66)
-		(diameter 0)
-		(color 0 0 0 0)
 	)
 	(junction
@@
 	)
 	(no_connect
+		(at 162.56 200.66)
+	)
+	(no_connect
 		(at 154.94 185.42)
 	)
@@
 		)
 		(stroke
-			(width 0)
-			(type default)
-		)
-	)
-	(wire
-		(pts
-			(xy 125.73 200.66) (xy 162.56 200.66)
-		)
-		(stroke

Commit message: Fixed GPIO4 and increased trace widths, added stitching vias to reduce parasitic cap.
Connections:
- net GPIO4: now also U1.C5 (ECAP0_IN_PWM0_OUT)
- no-connect marks 17 -> 16
Changed lines of the file:
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@@
+	)
+	(junction
+		(at 125.73 200.66)
+		(diameter 0)
+		(color 0 0 0 0)
 	)
 	(junction
@@
 	)
 	(no_connect
-		(at 162.56 200.66)
-	)
-	(no_connect
 		(at 154.94 185.42)
 	)
@@
 		)
 		(stroke
+			(width 0)
+			(type default)
+		)
+	)
+	(wire
+		(pts
+			(xy 125.73 200.66) (xy 162.56 200.66)
+		)
+		(stroke
