File: kicad/mram-and-spi.kicad_sch (KiCad schematic)
At the start: 7 parts, among them U2 MR20H40CDF

Commit message: Added extra decoupling capacitor to MRAM. Also grounded all unused pins and mounting holes
Parts:
- added C2: 10u, Capacitor_SMD:C_0603_1608Metric, symbol Device:C_Small
Connections:
- net 3.3V: now also C2.1
- net GND: now also C2.2
Changed lines of the file:
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@@
+	)
+	(junction
+		(at 158.75 63.5)
+		(diameter 0)
+		(color 0 0 0 0)
 	)
 	(junction
@@
 		(pts
 			(xy 113.03 78.74) (xy 115.57 78.74)
+		)
+		(stroke
+			(width 0)
+			(type default)
+		)
+	)
+	(wire
+		(pts
+			(xy 158.75 63.5) (xy 170.18 63.5)
 		)
 		(stroke
@@
 	)
 	(symbol
+		(lib_id "Device:C_Small")
+		(at 170.18 66.04 0)
+		(unit 1)
+		(exclude_from_sim no)
+		(in_bom yes)
+		(on_board yes)
+		(dnp no)
+		(fields_autoplaced yes)
+		(property "Reference" "C2"
+			(at 172.72 64.7762 0)
+			(effects
+				(font
+					(size 1.27 1.27)
+				)
+				(justify left)
+			)
+		)
+		(property "Value" "10u"
+			(at 172.72 67.3162 0)
+			(effects
+				(font
+					(size 1.27 1.27)
+				)
+				(justify left)
+			)
+		)
+		(property "Footprint" "Capacitor_SMD:C_0603_1608Metric"
+			(at 170.18 66.04 0)
+			(effects
+				(font
+					(size 1.27 1.27)
+				)
+				(hide yes)
+			)
+		)
+		(property "Datasheet" "~"
+			(at 170.18 66.04 0)
+			(effects
+				(font
+					(size 1.27 1.27)
+				)
+				(hide yes)
+			)
+		)
+		(property "Description" "Unpolarized capacitor, small symbol"
+			(at 170.18 66.04 0)
+			(effects
+				(font
+					(size 1.27 1.27)
+				)
+				(hide yes)
+			)
+		)
+		(pin "1"
+		)
+		(pin "2"
+		)
+		(instances
+			(project "oresat-c3"
+				(path "/65d12cdd-c326-4033-9053-c59fa4e0b25e/34cfbc26-5d78-4591-9d1f-0b27f2515f88"
+					(reference "C2")
+					(unit 1)
+				)
+			)
+		)
+	)
+	(symbol
 		(lib_id "power:GND")
 		(at 158.75 68.58 0)
@@
 					(unit 1)
 				)
+			)
+		)
+	)
+	(symbol
+		(lib_id "power:GND")
+		(at 170.18 68.58 0)
+		(unit 1)
+		(exclude_from_sim no)
+		(in_bom yes)
+		(on_board yes)
+		(dnp no)
+		(property "Reference" "#PWR07"
+			(at 170.18 74.93 0)
+			(effects
+				(font
+					(size 1.27 1.27)
+				)
+				(hide yes)
+			)
+		)
+		(property "Value" "GND"
+			(at 170.18 72.39 0)
+			(effects
+				(font
+					(size 1.27 1.27)
+				)
+			)
+		)
+		(property "Footprint" ""
+			(at 170.18 68.58 0)
+			(effects
+				(font
+					(size 1.27 1.27)
+				)
+				(hide yes)
+			)
+		)
+		(property "Datasheet" ""
+			(at 170.18 68.58 0)
+			(effects
+				(font
+					(size 1.27 1.27)
+				)
+				(hide yes)
+			)
+		)
+		(property "Description" ""
+			(at 170.18 68.58 0)
+			(effects
+				(font
+					(size 1.27 1.27)
+				)
+				(hide yes)
+			)
+		)
+		(pin "1"
+		)
+		(instances
+			(project "oresat-c3"
+				(path "/65d12cdd-c326-4033-9053-c59fa4e0b25e/34cfbc26-5d78-4591-9d1f-0b27f2515f88"
+					(reference "#PWR07")
+					(unit 1)
+				)

Commit message: added automotive grade capacitors to the BOM
Parts:
- C1: Description_1 (none) -> CAP CER 0.1UF 16V X7R 0603; Manufacturer_Name (none) -> Murata Electronics; Manufacturer_Part_Number (none) -> GCJ188R71C104KA01D
- C2: Description_1 (none) -> CAP CER 10UF 16V X5R 0603; Manufacturer_Name (none) -> Murata Electronics; Manufacturer_Part_Number (none) -> GRT188R61C106KE13D
- R4: Description_1 (none) -> RES 10K OHM 1% 1/8W 0603; Manufacturer_Name (none) -> Stackpole Electronics Inc; Manufacturer_Part_Number (none) -> RNCP0603FTD10K0
Changed lines of the file:
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@@
+			)
+		)
+		(property "Description_1" "CAP CER 0.1UF 16V X7R 0603"
+			(at 158.75 66.04 0)
+			(effects
+				(font
+					(size 1.27 1.27)
+				)
+				(hide yes)
+			)
+		)
+		(property "Manufacturer_Name" "Murata Electronics"
+			(at 158.75 66.04 0)
+			(effects
+				(font
+					(size 1.27 1.27)
+				)
+				(hide yes)
+			)
+		)
+		(property "Manufacturer_Part_Number" "GCJ188R71C104KA01D"
+			(at 158.75 66.04 0)
+			(effects
+				(font
+					(size 1.27 1.27)
+				)
+				(hide yes)
 			)
 		)
@@
 			)
 		)
+		(property "Description_1" "CAP CER 10UF 16V X5R 0603"
+			(at 170.18 66.04 0)
+			(effects
+				(font
+					(size 1.27 1.27)
+				)
+				(hide yes)
+			)
+		)
+		(property "Manufacturer_Name" "Murata Electronics"
+			(at 170.18 66.04 0)
+			(effects
+				(font
+					(size 1.27 1.27)
+				)
+				(hide yes)
+			)
+		)
+		(property "Manufacturer_Part_Number" "GRT188R61C106KE13D"
+			(at 170.18 66.04 0)
+			(effects
+				(font
+					(size 1.27 1.27)
+				)
+				(hide yes)
+			)
+		)
 		(pin "1"
 		)
@@
 			(at 113.03 69.85 0)
 			(effects
+				(font
+					(size 1.27 1.27)
+				)
+				(hide yes)
+			)
+		)
+		(property "Description_1" "RES 10K OHM 1% 1/8W 0603"
+			(at 113.03 69.85 0)
+			(effects
+				(font
+					(size 1.27 1.27)
+				)
+				(hide yes)
+			)
+		)
+		(property "Manufacturer_Name" "Stackpole Electronics Inc"
+			(at 113.03 69.85 0)
+			(effects
+				(font
+					(size 1.27 1.27)
+				)
+				(hide yes)
+			)
+		)
+		(property "Manufacturer_Part_Number" "RNCP0603FTD10K0"
+			(at 113.03 69.85 0)
+			(effects

Commit message: added automotive grade resistors to BOM
Parts:
- R4: Description_1 RES 10K OHM 1% 1/8W 0603 -> RES 0603 10 KOHM 1% 0.125W AUTO; Manufacturer_Part_Number RNCP0603FTD10K0 -> RMCA0603FT10K0-HP
Changed lines of the file:
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@@
 			)
 		)
-		(property "Description_1" "RES 10K OHM 1% 1/8W 0603"
+		(property "Description_1" "RES 0603 10 KOHM 1% 0.125W AUTO"
 			(at 113.03 69.85 0)
 			(effects
@@
 			)
 		)
-		(property "Manufacturer_Part_Number" "RNCP0603FTD10K0"
+		(property "Manufacturer_Part_Number" "RMCA0603FT10K0-HP"
 			(at 113.03 69.85 0)
 			(effects

Commit message: modified BOM to match PCBWay format
Parts:
- U2: Description_1 MRAM (Magnetoresistive RAM) Memory IC 4Mb (512K x 8) SPI 50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 -> IC RAM 4MBIT SPI 50MHZ 8DFN; Manufacturer_Name (none) -> Everspin Technologies Inc.; Manufacturer_Part_Number (none) -> MR20H40CDF
Changed lines of the file:
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@@
 			)
 		)
-		(property "Description_1" "\n                        \n                            MRAM (Magnetoresistive RAM) Memory IC 4Mb (512K x 8) SPI 50 MHz 8-DFN-EP, Small Flag (5x6)\n                        \n"
+		(property "Description_1" "IC RAM 4MBIT SPI 50MHZ 8DFN"
 			(at 134.62 81.28 0)
 			(effects
@@
 				(hide yes)
 			)
+		)
+		(property "Manufacturer_Name" "Everspin Technologies Inc."
+			(at 134.62 81.28 0)
+			(effects
+				(font
+					(size 1.27 1.27)
+				)
+				(hide yes)
+			)
+		)
+		(property "Manufacturer_Part_Number" "MR20H40CDF"
+			(at 134.62 81.28 0)
+			(effects
+				(font
+					(size 1.27 1.27)
+				)
+				(hide yes)
+			)

Commit message: finished putting together BOM, needs review
Parts:
- C1: Description / Value (none) -> CAP CER 0.1UF 16V X7R 0603; Description_1 CAP CER 0.1UF 16V X7R 0603 -> (none)
- C2: Description / Value (none) -> CAP CER 10UF 16V X5R 0603; Description_1 CAP CER 10UF 16V X5R 0603 -> (none)
- R4: Description / Value (none) -> RES 0603 10 KOHM 1% 0.125W AUTO; Description_1 RES 0603 10 KOHM 1% 0.125W AUTO -> (none)
- U2: Description / Value (none) -> IC RAM 4MBIT SPI 50MHZ 8DFN; Description_1 IC RAM 4MBIT SPI 50MHZ 8DFN -> (none)
Changed lines of the file:
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@@
-			)
-		)
-		(property "Description_1" "CAP CER 0.1UF 16V X7R 0603"
-			(at 158.75 66.04 0)
-			(effects
-				(font
-					(size 1.27 1.27)
-				)
-				(hide yes)
 			)
 		)
@@
 		)
 		(property "Manufacturer_Part_Number" "GCJ188R71C104KA01D"
+			(at 158.75 66.04 0)
+			(effects
+				(font
+					(size 1.27 1.27)
+				)
+				(hide yes)
+			)
+		)
+		(property "Description / Value" "CAP CER 0.1UF 16V X7R 0603"
 			(at 158.75 66.04 0)
 			(effects
@@
 			)
 		)
-		(property "Description_1" "CAP CER 10UF 16V X5R 0603"
-			(at 170.18 66.04 0)
-			(effects
-				(font
-					(size 1.27 1.27)
-				)
-				(hide yes)
-			)
-		)
 		(property "Manufacturer_Name" "Murata Electronics"
 			(at 170.18 66.04 0)
@@
 		)
 		(property "Manufacturer_Part_Number" "GRT188R61C106KE13D"
+			(at 170.18 66.04 0)
+			(effects
+				(font
+					(size 1.27 1.27)
+				)
+				(hide yes)
+			)
+		)
+		(property "Description / Value" "CAP CER 10UF 16V X5R 0603"
 			(at 170.18 66.04 0)
 			(effects
@@
 			)
 		)
-		(property "Description_1" "IC RAM 4MBIT SPI 50MHZ 8DFN"
-			(at 134.62 81.28 0)
-			(effects
-				(font
-					(size 1.27 1.27)
-				)
-				(justify bottom)
-				(hide yes)
-			)
-		)
 		(property "MANUFACTURER" "Everspin Technologies"
 			(at 134.62 81.28 0)
@@
 		)
 		(property "Manufacturer_Part_Number" "MR20H40CDF"
+			(at 134.62 81.28 0)
+			(effects
+				(font
+					(size 1.27 1.27)
+				)
+				(hide yes)
+			)
+		)
+		(property "Description / Value" "IC RAM 4MBIT SPI 50MHZ 8DFN"
 			(at 134.62 81.28 0)
 			(effects
@@
 			)
 		)
-		(property "Description_1" "RES 0603 10 KOHM 1% 0.125W AUTO"
-			(at 113.03 69.85 0)
-			(effects
-				(font
-					(size 1.27 1.27)
-				)
-				(hide yes)
-			)
-		)
 		(property "Manufacturer_Name" "Stackpole Electronics Inc"
 			(at 113.03 69.85 0)
@@
 			(at 113.03 69.85 0)
 			(effects
+				(font
+					(size 1.27 1.27)
+				)
+				(hide yes)
+			)
+		)
+		(property "Description / Value" "RES 0603 10 KOHM 1% 0.125W AUTO"
+			(at 113.03 69.85 0)
+			(effects
